File: schematics/kicad/misc.kicad_sch (KiCad schematic)
At the start: 100 parts, among them J11 Conn_01x04_Pin, K900 1000uF, K901 1000uF, K903 1000uF, K904 1000uF, X1 0.1uF, X10 0.1uF, X11 0.1uF, X12 0.1uF, X13 0.1uF, X14 0.1uF, X15 0.1uF, X16 0.1uF, X17 0.1uF, X18 0.1uF, X19 0.1uF, X2 0.1uF, X20 0.1uF, X21 0.1uF, X22 0.1uF, X23 0.1uF, X24 0.1uF, X25 0.1uF, X26 0.1uF, X27 0.1uF, X28 0.1uF, X29 0.1uF, X3 0.1uF, X30 0.1uF, X31 0.1uF, X32 0.1uF, X33 0.1uF, X34 0.1uF, X35 0.1uF, X36 0.1uF, X37 0.1uF, X38 0.1uF, X39 0.1uF, X4 0.1uF, X40 0.1uF, X41 0.1uF, X42 0.1uF, X43 0.1uF, X44 0.1uF, X45 0.1uF, X46 0.1uF, X47 0.1uF, X48 0.1uF, X49 0.1uF, X5 0.1uF, X50 0.1uF, X51 0.1uF, X52 0.1uF, X53 0.1uF, X54 0.1uF, X55 0.1uF, X56 0.1uF, X57 0.1uF, X58 0.1uF, X59 0.1uF, X6 0.1uF, X60 0.1uF, X61 0.1uF, X62 0.1uF, X63 0.1uF, X64 0.1uF, X65 0.1uF, X66 0.1uF, X67 0.1uF, X68 0.1uF, X69 0.1uF, X7 0.1uF, X70 0.1uF, X71 0.1uF, X72 0.1uF, X73 0.1uF, X74 0.1uF, X75 0.1uF, X76 0.1uF, X77 0.1uF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

Commit message: First draft for an expanded MMU
This version uses vintage parts except for the SRAM, which are IS61C5128AS-25HLI (they could be QLI instead)
Unfortunately, this requires:
* 2 more 74ALS245 to buffer the second byte of PMAP indices in the SMAP
* one more LS2518 (!) to extend the context register
* a couple of 74CBTLV3257 to be able to stay in "normal" Sun3 mode with minimal delays on the signals
* a couple of switches to enabled/disable the new features
* some extra passives
* U231, a PAL16L8, needs another input and another two outputs, or can be split in two PALs (or GAL, CPLDs, ...)

Also this does not include tne necessary decoupling on the new components
Changed lines of the file:
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@@
 (kicad_sch
-	(version 20231120)
+	(version 20250114)
 	(generator "eeschema")
-	(generator_version "8.0")
+	(generator_version "9.0")
 	(paper "A4")
 	(title_block
@@
 		(rev "1")
 	)
+	(text "10 - PD8- for 68030"
+		(exclude_from_sim no)
+		(at 200.66 96.266 0)
+		(effects
+			(font
+				(size 1.27 1.27)
+			)
+		)
+	)
+	(text "9 - CIIN for 68030"
+		(exclude_from_sim no)
+		(at 152.654 96.266 0)
+		(effects
+			(font
+				(size 1.27 1.27)
+			)
+		)
+	)
+	(text "Power"
+		(exclude_from_sim no)
+		(at 39.116 37.592 0)
+		(effects
+			(font
+				(size 1.27 1.27)
+			)
+		)
+	)
 	(junction
 		(at 88.9 149.86)
@@
 		)
 	)
-	(text "10 - PD8- for 68030"
-		(exclude_from_sim no)
-		(at 200.66 96.266 0)
-		(effects
-			(font
-				(size 1.27 1.27)
-			)
-		)
-	)
-	(text "9 - CIIN for 68030"
-		(exclude_from_sim no)
-		(at 152.654 96.266 0)
-		(effects
-			(font
-				(size 1.27 1.27)
-			)
-		)
-	)
-	(text "Power"
-		(exclude_from_sim no)
-		(at 39.116 37.592 0)
-		(effects
-			(font
-				(size 1.27 1.27)
-			)
-		)
-	)

Commit message: draft, ugly and WiP
Parts:
- removed S124, S125, S126, S127: 4.7k Ohm, Resistor_THT:R_Array_SIP10, symbol Device:R_Network09
- removed X1, X10, X11, X12, X13, X14, X15, X16, X17, X18, X19, X2, X20, X21, X22, X23, X24, X25, X26, X27, X28, X29, X3, X30, X31, X32, X33, X34, X35, X36, X37, X38, X39, X4, X40, X41, X42, X43, X44, X45, X46, X47, X48, X49, X5, X50, X51, X52, X53, X54, X55, X56, X57, X58, X59, X6, X60, X61, X62, X63, X64, X65, X66, X67, X68, X69, X7, X70, X71, X72, X73, X74, X75, X76, X77, X78, X79, X8, X80, X9: 0.1uF, Capacitor_THT:C_Rect_L7.0mm_W2.0mm_P5.00mm, symbol Device:C
- added R22, R23, R24, R25, R26, R27, R28, R29, R30, R31, R32, R33, R34, R35, R36, R37, R38, R39, R40, R41, R42, R43, R44, R45, R46, R47, R48, R49, R50, R51, R52, R53: 4.7k, Resistor_SMD:R_0402_1005Metric, symbol Device:R
- S109, S111, S117, S120, S121, S122, S123: MPN (none) -> 4611X-101-472LF; now not fitted; now left out of the parts list
- S113, S115, S116: MPN (none) -> 4611X-101-471LF; now not fitted; now left out of the parts list
- S114: MPN (none) -> 4611X-101-102LF; now not fitted; now left out of the parts list
Connections:
- net D0: now also R22.2
- net D1: now also R23.2
- net D10: now also R32.2
- net D11: now also R33.2
- net D12: now also R34.2
- net D13: now also R35.2
- net D14: now also R36.2
- net D15: now also R37.2
- net D16: now also R38.2
- net D17: now also R39.2
- net D18: now also R40.2
- net D19: now also R41.2
- net D2: now also R24.2
- net D20: now also R42.2
- net D21: now also R43.2
- net D22: now also R44.2
- net D23: now also R45.2
- net D24: now also R46.2
- net D25: now also R47.2
- net D26: now also R48.2
- net D27: now also R49.2
- net D28: now also R50.2
- net D29: now also R51.2
- net D3: now also R25.2
- net D30: now also R52.2
- net D31: now also R53.2
- net D4: now also R26.2
- net D5: now also R27.2
- net D6: now also R28.2
- net D7: now also R29.2
- net D8: now also R30.2
- net D9: now also R31.2
- net VCC: now also R22.1, R23.1, R24.1, R25.1, R26.1, R27.1, R28.1, R29.1, R30.1, R31.1, R32.1, R33.1, R34.1, R35.1, R36.1, R37.1, R38.1, R39.1, R40.1, R41.1, R42.1, R43.1, R44.1, R45.1, R46.1, R47.1, R48.1, R49.1, R50.1, R51.1, R52.1, R53.1
