File: schematics/kicad/sun3_60.kicad_pcb (KiCad board)
At the start: 4 copper layers, 231.1 x 340.4 mm, 225 parts, among them J11 Conn_01x04_Pin, J2 Serial A/B, J200 DIAG, J3 Ethernet, K199 10UF, K500 10 uF, K900 1000uF, K901 1000uF, K903 1000uF, K904 1000uF, U100 68020, U102 PAL16L8, U103 PAL16L8, U104 74F04, U106 PAL16L8, U107 PAL20X10, U108 74F00, U110 40.000 Mhz, U113 74AS74, U114 74F175, U115 74LS590, U122 ALS374, U123 ALS373, U130 74F374, U131 PAL16R6, U132 ALS244, U199 7705, U200 7188, U2003 74AS04, U2004 74LS125, U201 7188, U202 2168, U203 2168, U205 2168, U206 2168, U207 2168, U208 2168, U210 LS2518, U212 ALS245, U213 ALS245, U215 ALS245, U217 ALS245, U218 ALS245, U223 74F534, U224 AM27S19, U225 ALS273, U226 ALS373, U227 ALS273, U228 LED_Block, U229 LED_Block, U230 PAL16L8, U231 PAL16L8, U232 PAL16L8, U300 27512, U301 28C16, U302 7170, U303 32768Hz, U304 ALS273, U305 ALS373, U307 PAL20L8, U309 3-VOLT, U310 PAL20L8, U311 PAL20L8, U312 PAL8L14, U313 PAL16R4, U401 Z8530, U402 4.9152 Mhz, U408 74ALS04, U500 AM7990, U501 AM7992, U502 20 Mhz, U503 TRANSF, U510 ALS373, U511 ALS373, U512 ALS373, U514 ALS652, U515 ALS652, U516 ALS652, U517 ALS652, U518 PAL16L8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

Commit message: draft, ugly and WiP
Parts:
- removed J2: Serial A/B, Connector_PinHeader_2.54mm:PinHeader_1x05_P2.54mm_Vertical
- removed J200: DIAG, Connector_PinHeader_2.54mm:PinHeader_1x03_P2.54mm_Vertical
- removed S109, S111, S117, S120, S121, S122, S123, S124, S125, S126, S127, S800: 4.7k Ohm, Resistor_THT:R_Array_SIP10
- removed S113, S115, S116: 470 Ohm, Resistor_THT:R_Array_SIP10
- removed S114, S502: 1k Ohm, Resistor_THT:R_Array_SIP10
- removed S200: 68 Ohm, Resistor_THT:R_Array_SIP8
- removed S400: 4.7K Ohm, Resistor_THT:R_Array_SIP8
- removed S500: 40.2 Ohm 1%, Resistor_THT:R_Array_SIP10
- removed U102, U230, U231, U232, U714: PAL16L8, Package_DIP:DIP-20_W7.62mm
- removed U113: 74AS74, Package_DIP:DIP-14_W7.62mm
- removed U114: 74F175, Package_DIP:DIP-16_W7.62mm
- removed U122: ALS374, Package_DIP:DIP-20_W7.62mm
- removed U123, U226, U305: ALS373, Package_DIP:DIP-20_W7.62mm
- removed U200, U201: 7188, Package_DIP:DIP-22_W7.62mm
- removed U202, U203, U205, U206, U207, U208: 2168, Package_DIP:DIP-20_W7.62mm
- removed U210: LS2518, Package_DIP:DIP-16_W7.62mm
- removed U212, U213, U215, U217, U218: ALS245, Package_DIP:DIP-20_W7.62mm
- removed U223: 74F534, Package_DIP:DIP-20_W7.62mm
- removed U224: AM27S19, Package_DIP:DIP-16_W7.62mm
- removed U225, U227, U304: ALS273, Package_DIP:DIP-20_W7.62mm
- removed U228, U229: LED_Block, Connector_PinHeader_2.54mm:PinHeader_2x04_P2.54mm_Vertical
- removed U307, U310, U311: PAL20L8, Package_DIP:DIP-24_W7.62mm
- removed U312: PAL8L14, Package_DIP:DIP-24_W7.62mm
- removed U313: PAL16R4, Package_DIP:DIP-20_W7.62mm
- removed U408: 74ALS04, Package_DIP:DIP-14_W7.62mm
- removed U503: TRANSF, Package_DIP:DIP-16_W7.62mm
- removed U600: 74F04, Package_DIP:DIP-14_W7.62mm
- removed U715: PAL20R4, Package_DIP:DIP-24_W7.62mm
- removed U801: 74AS257, Package_DIP:DIP-16_W7.62mm
- removed U909: 22 Ohm, Package_DIP:DIP-16_W7.62mm
- removed X1, X19, X20, X21, X22, X31, X32, X37, X38, X49, X53, X54, X55, X56, X57, X58, X59, X60, X61, X62, X63, X64, X65, X66, X67, X68, X69, X70, X71, X72, X73, X74, X75, X76, X77, X78, X79, X80: 0.1uF, Capacitor_THT:C_Rect_L7.0mm_W2.0mm_P5.00mm
- added C1: 10uF 1206, Capacitor_SMD:C_1206_3216Metric, F.Cu at (56.8, 12.8)
- added C10: 100nF 0402, Capacitor_SMD:C_0402_1005Metric, F.Cu at (165.8, 72.0)
- added C11: 100nF 0402, Capacitor_SMD:C_0402_1005Metric, F.Cu at (165.8, 79.5)
- added C12: 100nF 0402, Capacitor_SMD:C_0402_1005Metric, F.Cu at (173.0, 88.2)
- added C13: 100nF 0402, Capacitor_SMD:C_0402_1005Metric, F.Cu at (177.5, 88.2)
- added C14: 100nF 0402, Capacitor_SMD:C_0402_1005Metric, F.Cu at (163.2, 83.0)
- added C15: 100nF 0402, Capacitor_SMD:C_0402_1005Metric, F.Cu at (163.2, 75.5)
- added C16: 100nF 0402, Capacitor_SMD:C_0402_1005Metric, F.Cu at (155.0, 67.8)
- added C17: 100nF 0402, Capacitor_SMD:C_0402_1005Metric, F.Cu at (152.5, 67.8)
- added C18: 100nF 0402, Capacitor_SMD:C_0402_1005Metric, F.Cu at (142.8, 72.0)
- added C19: 100nF 0402, Capacitor_SMD:C_0402_1005Metric, F.Cu at (142.8, 79.5)
- added C2: 10uF 1206, Capacitor_SMD:C_1206_3216Metric, F.Cu at (73.2, 12.8)
- added C20: 100nF 0402, Capacitor_SMD:C_0402_1005Metric, F.Cu at (150.0, 88.2)
- added C21: 100nF 0402, Capacitor_SMD:C_0402_1005Metric, F.Cu at (154.5, 88.2)
- added C22: 100nF 0402, Capacitor_SMD:C_0402_1005Metric, F.Cu at (186.2, 60.0)
- added C23: 100nF 0402, Capacitor_SMD:C_0402_1005Metric, F.Cu at (186.2, 52.5)
- added C24: 100nF 0402, Capacitor_SMD:C_0402_1005Metric, F.Cu at (178.0, 44.8)
- added C25: 100nF 0402, Capacitor_SMD:C_0402_1005Metric, F.Cu at (175.5, 44.8)
- added C26: 100nF 0402, Capacitor_SMD:C_0402_1005Metric, F.Cu at (165.8, 49.0)
- added C27: 100nF 0402, Capacitor_SMD:C_0402_1005Metric, F.Cu at (165.8, 56.5)
- added C28: 100nF 0402, Capacitor_SMD:C_0402_1005Metric, F.Cu at (173.0, 65.2)
- added C29: 100nF 0402, Capacitor_SMD:C_0402_1005Metric, F.Cu at (177.0, 64.8)
- added C3: 10uF 1206, Capacitor_SMD:C_1206_3216Metric, F.Cu at (56.8, 105.0)
- added C30: 100nF 0402, Capacitor_SMD:C_0402_1005Metric, F.Cu at (190.2, 29.5)
- added C31: 100nF 0402, Capacitor_SMD:C_0402_1005Metric, F.Cu at (182.0, 21.8)
- added C32: 100nF 0402, Capacitor_SMD:C_0402_1005Metric, F.Cu at (179.5, 21.8)
- added C33: 100nF 0402, Capacitor_SMD:C_0402_1005Metric, F.Cu at (169.8, 26.0)
- added C34: 100nF 0402, Capacitor_SMD:C_0402_1005Metric, F.Cu at (169.8, 33.5)
- added C35: 100nF 0402, Capacitor_SMD:C_0402_1005Metric, F.Cu at (177.0, 42.2)
- added C36: 100nF 0402, Capacitor_SMD:C_0402_1005Metric, F.Cu at (181.5, 42.2)
- added C37: 100nF 0402, Capacitor_SMD:C_0402_1005Metric, F.Cu at (84.2, 132.0)
- added C38: 100nF 0402, Capacitor_SMD:C_0402_1005Metric, F.Cu at (84.2, 124.5)
- added C39: 100nF 0402, Capacitor_SMD:C_0402_1005Metric, F.Cu at (76.0, 116.8)
- added C4: 10uF 1206, Capacitor_SMD:C_1206_3216Metric, F.Cu at (73.2, 105.0)
- added C40: 100nF 0402, Capacitor_SMD:C_0402_1005Metric, F.Cu at (73.5, 116.8)
- added C41: 100nF 0402, Capacitor_SMD:C_0402_1005Metric, F.Cu at (63.8, 121.0)
- added C42: 100nF 0402, Capacitor_SMD:C_0402_1005Metric, F.Cu at (63.8, 128.5)
- added C43: 100nF 0402, Capacitor_SMD:C_0402_1005Metric, F.Cu at (71.0, 137.2)
- added C44: 100nF 0402, Capacitor_SMD:C_0402_1005Metric, F.Cu at (75.5, 137.2)
- added C45: 100nF 0402, Capacitor_SMD:C_0402_1005Metric, F.Cu at (81.2, 183.0)
- added C46: 100nF 0402, Capacitor_SMD:C_0402_1005Metric, F.Cu at (81.2, 175.5)
- added C47: 100nF 0402, Capacitor_SMD:C_0402_1005Metric, F.Cu at (73.0, 167.8)
- added C48: 100nF 0402, Capacitor_SMD:C_0402_1005Metric, F.Cu at (70.5, 167.8)
- added C49: 100nF 0402, Capacitor_SMD:C_0402_1005Metric, F.Cu at (60.8, 172.0)
- added C5: 100nF 0402, Capacitor_SMD:C_0402_1005Metric, F.Cu at (190.2, 37.0)
- added C50: 100nF 0402, Capacitor_SMD:C_0402_1005Metric, F.Cu at (60.8, 179.5)
- added C51: 100nF 0402, Capacitor_SMD:C_0402_1005Metric, F.Cu at (68.0, 188.2)
- added C52: 100nF 0402, Capacitor_SMD:C_0402_1005Metric, F.Cu at (72.5, 188.3)
- added C6: 100nF 0402, Capacitor_SMD:C_0402_1005Metric, F.Cu at (186.0, 83.5)
- added C7: 100nF 0402, Capacitor_SMD:C_0402_1005Metric, F.Cu at (186.2, 75.5)
- added C8: 100nF 0402, Capacitor_SMD:C_0402_1005Metric, F.Cu at (178.0, 67.8)
- added C9: 100nF 0402, Capacitor_SMD:C_0402_1005Metric, F.Cu at (175.5, 67.8)
- added D1: LED, LED_SMD:LED_0603_1608Metric, F.Cu at (65.2, 113.2)
- added D2: LED, LED_SMD:LED_0603_1608Metric, F.Cu at (65.2, 111.2)
- added D3: LED, LED_SMD:LED_0603_1608Metric, F.Cu at (65.2, 109.2)
- added D4: LED, LED_SMD:LED_0603_1608Metric, F.Cu at (65.2, 107.2)
- added D5: LED, LED_SMD:LED_0603_1608Metric, F.Cu at (65.2, 105.2)
- added D6: LED, LED_SMD:LED_0603_1608Metric, F.Cu at (65.2, 103.2)
- added D7: LED, LED_SMD:LED_0603_1608Metric, F.Cu at (65.2, 101.2)
- added D8: LED, LED_SMD:LED_0603_1608Metric, F.Cu at (65.2, 99.2)
- added IC1: ATF1504AS-10AU100, sun3_60:QFP50P1600X1600X120-100N, F.Cu at (176.0, 55.0)
- added IC2: ATF1504AS-10AU100, sun3_60:QFP50P1600X1600X120-100N, F.Cu at (153.0, 78.0)
- added IC3: ATF1504AS-10AU100, sun3_60:QFP50P1600X1600X120-100N, F.Cu at (176.0, 78.0)
- added IC4: ATF1504AS-10AU100, sun3_60:QFP50P1600X1600X120-100N, F.Cu at (180.0, 32.0)
- added IC5: ATF1504AS-10AU100, sun3_60:QFP50P1600X1600X120-100N, F.Cu at (74.0, 127.0)
- added IC6: ATF1504AS-10AU100, sun3_60:QFP50P1600X1600X120-100N, F.Cu at (71.0, 178.0)
- added J5: 5747845-4, sun3_60:57478454, F.Cu at (11.0, 260.0)
- added J6: DB25_Socket, sun3_60:D25S33E4PA00LF, F.Cu at (289.0, 126.0)
- added J7: DB25_Socket, sun3_60:D25S33E4PA00LF, F.Cu at (289.0, 66.0)
- added R1: 10k, Resistor_SMD:R_0402_1005Metric, F.Cu at (176.0, 96.0)
- added R10: 22, Resistor_SMD:R_0402_1005Metric, F.Cu at (116.8, 33.2)
- added R11: 22, Resistor_SMD:R_0402_1005Metric, F.Cu at (116.5, 26.8)
- added R12: 22, Resistor_SMD:R_0402_1005Metric, F.Cu at (56.8, 33.2)
- added R13: 22, Resistor_SMD:R_0402_1005Metric, F.Cu at (56.5, 26.8)
- added R14: 22, Resistor_SMD:R_0402_1005Metric, F.Cu at (116.8, 32.0)
- added R15: 22, Resistor_SMD:R_0402_1005Metric, F.Cu at (116.5, 25.5)
- added R16: 22, Resistor_SMD:R_0402_1005Metric, F.Cu at (116.8, 30.8)
- added R17: 22, Resistor_SMD:R_0402_1005Metric, F.Cu at (116.5, 24.2)
- added R18: 22, Resistor_SMD:R_0402_1005Metric, F.Cu at (56.8, 32.0)
- added R19: 22, Resistor_SMD:R_0402_1005Metric, F.Cu at (56.5, 25.5)
- added R2: 10k, Resistor_SMD:R_0402_1005Metric, F.Cu at (176.0, 94.0)
- added R20: 22, Resistor_SMD:R_0402_1005Metric, F.Cu at (56.8, 30.8)
- added R21: 22, Resistor_SMD:R_0402_1005Metric, F.Cu at (56.5, 24.2)
- added R22: 4.7k, Resistor_SMD:R_0402_1005Metric, F.Cu at (57.5, 92.0)
- added R23: 4.7k, Resistor_SMD:R_0402_1005Metric, F.Cu at (74.5, 84.2)
- added R24: 4.7k, Resistor_SMD:R_0402_1005Metric, F.Cu at (71.8, 74.2)
- added R25: 4.7k, Resistor_SMD:R_0402_1005Metric, F.Cu at (57.5, 66.0)
- added R26: 4.7k, Resistor_SMD:R_0402_1005Metric, F.Cu at (55.5, 55.8)
- added R27: 4.7k, Resistor_SMD:R_0402_1005Metric, F.Cu at (71.5, 48.0)
- added R28: 4.7k, Resistor_SMD:R_0402_1005Metric, F.Cu at (74.5, 41.0)
- added R29: 4.7k, Resistor_SMD:R_0402_1005Metric, F.Cu at (71.0, 35.5)
- added R3: 10k, Resistor_SMD:R_0402_1005Metric, F.Cu at (168.2, 97.0)
- added R30: 4.7k, Resistor_SMD:R_0402_1005Metric, F.Cu at (57.5, 93.0)
- added R31: 4.7k, Resistor_SMD:R_0402_1005Metric, F.Cu at (55.2, 85.0)
- added R32: 4.7k, Resistor_SMD:R_0402_1005Metric, F.Cu at (71.8, 75.5)
- added R33: 4.7k, Resistor_SMD:R_0402_1005Metric, F.Cu at (72.2, 66.8)
- added R34: 4.7k, Resistor_SMD:R_0402_1005Metric, F.Cu at (56.8, 55.8)
- added R35: 4.7k, Resistor_SMD:R_0402_1005Metric, F.Cu at (71.5, 46.8)
- added R36: 4.7k, Resistor_SMD:R_0402_1005Metric, F.Cu at (55.2, 41.8)
- added R37: 4.7k, Resistor_SMD:R_0402_1005Metric, F.Cu at (71.0, 34.2)
- added R38: 4.7k, Resistor_SMD:R_0402_1005Metric, F.Cu at (56.2, 95.2)
- added R39: 4.7k, Resistor_SMD:R_0402_1005Metric, F.Cu at (55.2, 83.5)
- added R4: 10k, Resistor_SMD:R_0402_1005Metric, F.Cu at (176.0, 106.0)
- added R40: 4.7k, Resistor_SMD:R_0402_1005Metric, F.Cu at (56.0, 77.2)
- added R41: 4.7k, Resistor_SMD:R_0402_1005Metric, F.Cu at (72.2, 68.0)
- added R42: 4.7k, Resistor_SMD:R_0402_1005Metric, F.Cu at (56.8, 60.3)
- added R43: 4.7k, Resistor_SMD:R_0402_1005Metric, F.Cu at (73.0, 45.0)
- added R44: 4.7k, Resistor_SMD:R_0402_1005Metric, F.Cu at (55.2, 40.0)
- added R45: 4.7k, Resistor_SMD:R_0402_1005Metric, F.Cu at (73.5, 32.2)
- added R46: 4.7k, Resistor_SMD:R_0402_1005Metric, F.Cu at (55.0, 95.2)
- added R47: 4.7k, Resistor_SMD:R_0402_1005Metric, F.Cu at (74.5, 81.8)
- added R48: 4.7k, Resistor_SMD:R_0402_1005Metric, F.Cu at (54.8, 77.2)
- added R49: 4.7k, Resistor_SMD:R_0402_1005Metric, F.Cu at (57.5, 69.0)
- added R5: 10k, Resistor_SMD:R_0402_1005Metric, F.Cu at (176.0, 104.0)
- added R50: 4.7k, Resistor_SMD:R_0402_1005Metric, F.Cu at (55.5, 60.2)
- added R51: 4.7k, Resistor_SMD:R_0402_1005Metric, F.Cu at (74.2, 45.0)
- added R52: 4.7k, Resistor_SMD:R_0402_1005Metric, F.Cu at (74.5, 38.5)
- added R53: 4.7k, Resistor_SMD:R_0402_1005Metric, F.Cu at (74.8, 32.3)
- added R55: 4.7k, Resistor_SMD:R_0402_1005Metric, F.Cu at (129.5, 55.0)
- added R56: 4.7k, Resistor_SMD:R_0402_1005Metric, F.Cu at (132.5, 50.7)
- added R57: 4.7k, Resistor_SMD:R_0402_1005Metric, F.Cu at (140.5, 52.8)
- added R58: 4.7k, Resistor_SMD:R_0402_1005Metric, F.Cu at (142.5, 52.8)
- added R59: 4.7k, Resistor_SMD:R_0402_1005Metric, F.Cu at (133.5, 50.7)
- added R6: 22, Resistor_SMD:R_0402_1005Metric, F.Cu at (116.8, 34.5)
- added R60: 4.7k, Resistor_SMD:R_0402_1005Metric, F.Cu at (143.5, 52.8)
- added R61: 4.7k, Resistor_SMD:R_0402_1005Metric, F.Cu at (141.5, 52.8)
- added R62: 510, Resistor_SMD:R_0402_1005Metric, F.Cu at (61.8, 113.2)
- added R63: 510, Resistor_SMD:R_0402_1005Metric, F.Cu at (61.8, 111.2)
- added R64: 510, Resistor_SMD:R_0402_1005Metric, F.Cu at (61.8, 109.2)
- added R65: 510, Resistor_SMD:R_0402_1005Metric, F.Cu at (61.8, 107.2)
- added R66: 510, Resistor_SMD:R_0402_1005Metric, F.Cu at (61.8, 105.2)
- added R67: 510, Resistor_SMD:R_0402_1005Metric, F.Cu at (61.8, 103.2)
- added R68: 510, Resistor_SMD:R_0402_1005Metric, F.Cu at (61.8, 101.2)
- added R69: 510, Resistor_SMD:R_0402_1005Metric, F.Cu at (61.8, 99.2)
- added R7: 22, Resistor_SMD:R_0402_1005Metric, F.Cu at (56.8, 34.5)
- added R8: 22, Resistor_SMD:R_0402_1005Metric, F.Cu at (116.5, 23.0)
- added R9: 22, Resistor_SMD:R_0402_1005Metric, F.Cu at (56.5, 23.0)
- added S1: SSAJ110100, sun3_60:SW_SSAJ110100, F.Cu at (179.5, 95.0)
- added S2: SSAJ110100, sun3_60:SW_SSAJ110100, F.Cu at (179.5, 105.0)
- added T1: TG01-0506NRLTR, sun3_60:TG010506NRLTR, F.Cu at (25.6, 253.6)
- added U1: IS61C5128AS-25HLI, Package_SO:TSOP-I-32_11.8x8mm_P0.5mm, F.Cu at (135.0, 81.0)
- added U10: CBT3257APW, Package_SO:TSSOP-16_4.4x5mm_P0.65mm, F.Cu at (168.2, 103.2)
- added U101: 68881, sun3_60:MC68882_PGA, F.Cu at (107.0, 130.0)
- added U11: 74CBT3257APW, Package_SO:TSSOP-16_4.4x5mm_P0.65mm, F.Cu at (168.2, 93.2)
- added U14: 74LVC1G04, Package_TO_SOT_SMD:SOT-353_SC-70-5, F.Cu at (189.0, 46.0)
- added U15: 74LVC1G74, sun3_60:74AVC9112GTX, F.Cu at (206.5, 10.6)
- added U17: 74LVC1G74, sun3_60:74AVC9112GTX, F.Cu at (60.6, 137.9)
- added U2: IS61C5128AS-25HLI, Package_SO:TSOP-I-32_11.8x8mm_P0.5mm, F.Cu at (135.0, 60.0)
- added U3: IS61C5128AS-25HLI, Package_SO:TSOP-I-32_11.8x8mm_P0.5mm, F.Cu at (135.0, 102.0)
- added U4: IS61C5128AS-25HLI, Package_SO:TSOP-I-32_11.8x8mm_P0.5mm, F.Cu at (135.0, 123.0)
- added U400: Z8530, Package_DIP:DIP-40_W15.24mm, F.Cu at (239.0, 206.0)
- added U404: 74ALS04, Package_SO:SOIC-14_3.9x8.7mm_P1.27mm, F.Cu at (278.2, 184.0)
- added U7: IS61C5128AS-25HLI, Package_SO:TSOP-I-32_11.8x8mm_P0.5mm, F.Cu at (148.5, 101.0)
- added U8: IS61C5128AS-25HLI, Package_SO:TSOP-I-32_11.8x8mm_P0.5mm, F.Cu at (158.5, 101.0)
- added U920: SIMM, sun3_60:SIMM, F.Cu at (80.0, 60.0)
- added U921: SIMM, sun3_60:SIMM, F.Cu at (90.0, 60.0)
- added U922: SIMM, sun3_60:SIMM, F.Cu at (100.0, 60.0)
- added U923: SIMM, sun3_60:SIMM, F.Cu at (110.0, 60.0)
- added U924: 74AS258, Package_SO:SOIC-16_3.9x9.9mm_P1.27mm, F.Cu at (124.0, 90.0)
- added U925: 74AS258, Package_SO:SOIC-16_3.9x9.9mm_P1.27mm, F.Cu at (124.0, 71.0)
- added U926: 74AS258, Package_SO:SOIC-16_3.9x9.9mm_P1.27mm, F.Cu at (124.0, 52.0)
- added U927: AS1032, Package_SO:SOIC-14_3.9x8.7mm_P1.27mm, F.Cu at (123.0, 34.0)
- added U928: AS1032, Package_SO:SOIC-14_3.9x8.7mm_P1.27mm, F.Cu at (123.0, 24.0)
- added X103: 100nF 0402, Capacitor_SMD:C_0402_1005Metric, F.Cu at (148.8, 110.0)
- added X104: 10nF 0402, Capacitor_SMD:C_0402_1005Metric, F.Cu at (147.8, 110.0)
- added X105: 100nF 0402, Capacitor_SMD:C_0402_1005Metric, F.Cu at (158.8, 110.0)
- added X106: 10nF 0402, Capacitor_SMD:C_0402_1005Metric, F.Cu at (157.8, 110.0)
- added X110: 100nF 0402, Capacitor_SMD:C_0402_1005Metric, F.Cu at (156.2, 35.0)
- added X81: 100nF 0402, Capacitor_SMD:C_0402_1005Metric, F.Cu at (128.5, 20.2)
- added X82: 100nF 0402, Capacitor_SMD:C_0402_1005Metric, F.Cu at (128.5, 30.2)
- added X83: 100nF 0402, Capacitor_SMD:C_0402_1005Metric, F.Cu at (118.5, 56.4)
- added X84: 100nF 0402, Capacitor_SMD:C_0402_1005Metric, F.Cu at (118.5, 75.4)
- added X85: 100nF 0402, Capacitor_SMD:C_0402_1005Metric, F.Cu at (118.5, 94.5)
- added X86: 100nF 0402, Capacitor_SMD:C_0402_1005Metric, F.Cu at (68.5, 20.2)
- added X87: 100nF 0402, Capacitor_SMD:C_0402_1005Metric, F.Cu at (68.5, 30.2)
- added X88: 100nF 0402, Capacitor_SMD:C_0402_1005Metric, F.Cu at (58.5, 56.4)
- added X89: 100nF 0402, Capacitor_SMD:C_0402_1005Metric, F.Cu at (58.5, 75.4)
- added X90: 100nF 0402, Capacitor_SMD:C_0402_1005Metric, F.Cu at (58.5, 94.4)
- added X91: 100nF 0402, Capacitor_SMD:C_0402_1005Metric, F.Cu at (134.8, 71.8)
- added X92: 10nF 0402, Capacitor_SMD:C_0402_1005Metric, F.Cu at (135.8, 71.8)
- added X93: 100nF 0402, Capacitor_SMD:C_0402_1005Metric, F.Cu at (134.8, 50.8)
- added X94: 10nF 0402, Capacitor_SMD:C_0402_1005Metric, F.Cu at (135.8, 50.8)
- added X95: 100nF 0402, Capacitor_SMD:C_0402_1005Metric, F.Cu at (134.8, 92.8)
- added X96: 10nF 0402, Capacitor_SMD:C_0402_1005Metric, F.Cu at (135.8, 92.8)
- added X97: 100nF 0402, Capacitor_SMD:C_0402_1005Metric, F.Cu at (134.8, 113.8)
- added X98: 10nF 0402, Capacitor_SMD:C_0402_1005Metric, F.Cu at (135.8, 113.8)
- C199: value 0.1UF -> 100nF 0402; footprint Capacitor_THT:C_Disc_D3.0mm_W2.0mm_P2.50mm -> Capacitor_SMD:C_0402_1005Metric
- C503, C504, X10, X11, X12, X13, X14, X15, X16, X17, X2, X23, X24, X25, X26, X27, X28, X29, X3, X30, X33, X34, X35, X36, X39, X4, X40, X41, X42, X43, X44, X45, X46, X47, X48, X5, X50, X51, X52, X6, X7, X8, X9: value 0.1uF -> 100nF 0402; footprint Capacitor_THT:C_Rect_L7.0mm_W2.0mm_P5.00mm -> Capacitor_SMD:C_0402_1005Metric
- J3: value Ethernet -> Mini-DIN-8; footprint Connector_PinHeader_2.54mm:PinHeader_1x09_P2.54mm_Vertical -> sun3_60:57492681
- K199: value 10UF -> 10uF tantalum; footprint Capacitor_THT:CP_Radial_Tantal_D6.0mm_P2.50mm -> Capacitor_Tantalum_SMD:CP_EIA-3216-18_Kemet-A
- K500: value 10 uF -> 10uF tantalum; footprint Capacitor_THT:CP_Radial_Tantal_D6.0mm_P2.50mm -> Capacitor_Tantalum_SMD:CP_EIA-3216-18_Kemet-A
- R100: value 150 ohm -> 150 ohm 0805; footprint Resistor_THT:R_Axial_DIN0207_L6.3mm_D2.5mm_P7.62mm_Horizontal -> Resistor_SMD:R_0805_2012Metric
- R101: value 100 ohm -> 100 ohm 0805; footprint Resistor_THT:R_Axial_DIN0207_L6.3mm_D2.5mm_P7.62mm_Horizontal -> Resistor_SMD:R_0805_2012Metric
- U100: footprint sun3_60:68020 -> sun3_60:MC68020RC25
- U104, U108, U2003, U2004, U907, U908: footprint Package_DIP:DIP-14_W7.62mm -> Package_SO:SOIC-14_3.9x8.7mm_P1.27mm
- U110, U402: footprint Oscillator:Oscillator_DIP-14 -> sun3_60:CXO_DIP8+14
- U115: footprint Package_DIP:DIP-16_W7.62mm -> Package_SO:SO-16_3.9x9.9mm_P1.27mm
- U130, U132, U510, U511, U512, U720, U721, U722, U723: footprint Package_DIP:DIP-20_W7.62mm -> Package_SO:SOIC-20W_7.5x12.8mm_P1.27mm
- U199: footprint Package_DIP:DIP-8_W7.62mm -> Package_SO:SOIC-8_3.9x4.9mm_P1.27mm
- U301: value 28C16 -> AT28C64B_PLCC; footprint Package_DIP:DIP-24_W15.24mm -> Package_LCC:PLCC-32_THT-Socket
- U514, U515, U516, U517: footprint Package_DIP:DIP-24_W7.62mm -> Package_SO:SOIC-24W_7.5x15.4mm_P1.27mm
- U520, U904, U905, U906: footprint Package_DIP:DIP-16_W7.62mm -> Package_SO:SOIC-16_3.9x9.9mm_P1.27mm
- U710, U711, U712, U713: value AS286 -> ACT11286; footprint Package_DIP:DIP-14_W7.62mm -> Package_SO:SOIC-14_3.9x8.7mm_P1.27mm
- U900, U901, U902, U903: footprint Connector_PinHeader_2.54mm:PinHeader_1x30_P2.54mm_Vertical -> sun3_60:SIMM
- X18: value 0.1uF -> 10nF 0402; footprint Capacitor_THT:C_Rect_L7.0mm_W2.0mm_P5.00mm -> Capacitor_SMD:C_0402_1005Metric
- moved K901 371.1 mm to (-30.3, 429.8)
- moved U110 335.6 mm to (187.4, 5.19), turned to 180 degrees
- moved U108 308.8 mm to (162.0, 10.0), turned to 180 degrees
- moved U115 308.6 mm to (210.0, 23.0), turned to 180 degrees
- moved X14 305.5 mm to (160.0, 16.0), turned to 0 degrees
- moved U106 286.1 mm to (195.0, 20.0), turned to 0 degrees
- moved C300 285.2 mm to (-143.5, 306.5)
- moved J11 285.2 mm to (-151.1, 255.7)
- moved R300 285.2 mm to (-133.3, 314.1)
- moved R301 285.2 mm to (-129.5, 265.9)
- moved U303 285.2 mm to (-137.5, 307.8)
- moved C301 285.2 mm to (-153.6, 310.6)
- moved K900 285.2 mm to (-120.6, 253.3)
- moved U309 285.2 mm to (-145.8, 277.3)
- moved X301 285.2 mm to (-120.6, 268.4)
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Connections:
- net Net-(U401-PCLK) renamed /sun3_60_serial/SERIAL_PCLK
- C300 pad 2: Net-(C300-Pad2) -> VCC
- C301 pad 1: Net-(C300-Pad2) -> VCC
- J3 pad 1: +12V -> GND
- J3 pad 2: /Ethernet/E.CO+<> -> GND
- J3 pad 3: /Ethernet/E.CO-<> -> VCC
- J3 pad 4: /Ethernet/E.RX+<> -> /sun3_60_serial/RxDB
- J3 pad 5: /Ethernet/E.RX-<> -> /sun3_60_serial/TxDA
- J3 pad 6: /Ethernet/E.TX+<> -> /sun3_60_serial/RxDA
- J3 pad 7: /Ethernet/E.TX-<> -> /sun3_60_serial/TxDB
- J3 pad 8: /Ethernet/E.SMS -> VCC
- U103 pad 15: /sun3_60_cpu/FC1 -> /FC1
- U103 pad 16: /sun3_60_cpu/FC0 -> /FC0
- U104 pad 1: /AS- -> unconnected-(U104-Pad1)
- U104 pad 2: /AS -> unconnected-(U104-Pad2)
- U104 pad 8: /sun3_60_cpu/DS -> unconnected-(U104-Pad8)
- U104 pad 9: /DS- -> unconnected-(U104-Pad9)
- U132 pad 16: /Ethernet/A26 -> /Ethernet/A24
- U132 pad 18: /Ethernet/A24 -> /Ethernet/A27
- U132 pad 5: /Ethernet/A27 -> /Ethernet/A26
- U2004 pad 3: /DSACK0- -> /DSACK1-
- U2004 pad 6: /DSACK1- -> /DSACK0-
- U301 pad 1: /Ethernet/A7 -> unconnected-(U301-DC-Pad1)
- U301 pad 10: /SCSI 2, Parity/IO.D1 -> /Ethernet/A1
- U301 pad 11: /SCSI 2, Parity/IO.D2 -> /Ethernet/A0
- U301 pad 12: GND -> unconnected-(U301-NC-Pad12)
- U301 pad 15: /SCSI 2, Parity/IO.D5 -> /SCSI 2, Parity/IO.D2
- U301 pad 16: /SCSI 2, Parity/IO.D6 -> GND
- U301 pad 17: /SCSI 2, Parity/IO.D7 -> unconnected-(U301-DC-Pad17)
- U301 pad 18: GND -> /SCSI 2, Parity/IO.D5
- U301 pad 19: /Ethernet/A10 -> /SCSI 2, Parity/IO.D1
- U301 pad 2: /Ethernet/A6 -> unconnected-(U301-NC-Pad2)
- U301 pad 20: /sun3_60_eeprom/RD.EEPROM- -> /SCSI 2, Parity/IO.D6
- U301 pad 21: /sun3_60_eeprom/WR.EEPROM- -> /SCSI 2, Parity/IO.D7
- U301 pad 22: /Ethernet/A9 -> /SCSI 2, Parity/IO.D0
- U301 pad 23: /Ethernet/A8 -> GND
- U301 pad 24: VCC -> /Ethernet/A8
- U301 pad 3: /Ethernet/A5 -> GND
- U301 pad 4: /Ethernet/A4 -> /Ethernet/A7
- U301 pad 5: /Ethernet/A3 -> /Ethernet/A6
- U301 pad 6: /Ethernet/A2 -> /Ethernet/A5
- U301 pad 7: /Ethernet/A1 -> /Ethernet/A4
- U301 pad 8: /Ethernet/A0 -> /Ethernet/A3
- U301 pad 9: /SCSI 2, Parity/IO.D0 -> /Ethernet/A2
- U401 pad 13: Net-(U401-RXDA) -> /sun3_60_serial/RXDC
- U401 pad 15: Net-(U401-TXDA) -> /sun3_60_serial/TXDC
- U401 pad 25: Net-(U401-TXDB) -> /sun3_60_serial/TXDD
- U401 pad 27: Net-(U401-RXDB) -> /sun3_60_serial/RXDD
- U512 pad 12: /Ethernet/A20 -> /Ethernet/A16
- U512 pad 13: /Ethernet/E.A20 -> /Ethernet/E.A16
- U512 pad 14: /Ethernet/E.A21 -> /Ethernet/E.A17
- U512 pad 15: /Ethernet/A21 -> /Ethernet/A17
- U512 pad 16: /Ethernet/A22 -> /Ethernet/A18
- U512 pad 17: /Ethernet/E.A22 -> /Ethernet/E.A18
- U512 pad 18: /Ethernet/E.A23 -> /Ethernet/E.A19
- U512 pad 19: /Ethernet/A23 -> /Ethernet/A19
- U512 pad 2: /Ethernet/A16 -> /Ethernet/A20
- U512 pad 3: /Ethernet/E.A16 -> /Ethernet/E.A20
- U512 pad 4: /Ethernet/E.A17 -> /Ethernet/E.A21
- U512 pad 5: /Ethernet/A17 -> /Ethernet/A21
- U512 pad 6: /Ethernet/A18 -> /Ethernet/A22
- U512 pad 7: /Ethernet/E.A18 -> /Ethernet/E.A22
- U512 pad 8: /Ethernet/E.A19 -> /Ethernet/E.A23
- U512 pad 9: /Ethernet/A19 -> /Ethernet/A23
- U514 pad 13: /sun3_60_cpu/D7 -> /D7
- U514 pad 14: /sun3_60_cpu/D6 -> /D6
- U514 pad 15: /sun3_60_cpu/D5 -> /D5
- U514 pad 16: /sun3_60_cpu/D4 -> /D4
- U514 pad 17: /sun3_60_cpu/D3 -> /D3
- U514 pad 18: /sun3_60_cpu/D2 -> /D2
- U514 pad 19: /sun3_60_cpu/D1 -> /D1
- U514 pad 20: /sun3_60_cpu/D0 -> /D0
- U515 pad 13: /sun3_60_cpu/D15 -> /D15
- U515 pad 14: /sun3_60_cpu/D14 -> /D14
- U515 pad 15: /sun3_60_cpu/D13 -> /D13
- U515 pad 16: /sun3_60_cpu/D12 -> /D12
- U515 pad 17: /sun3_60_cpu/D11 -> /D11
- U515 pad 18: /sun3_60_cpu/D10 -> /D10
- U515 pad 19: /sun3_60_cpu/D9 -> /D9
- U515 pad 20: /sun3_60_cpu/D8 -> /D8
- U516 pad 13: /sun3_60_cpu/D23 -> /D23
- U516 pad 14: /sun3_60_cpu/D22 -> /D22
- U516 pad 15: /sun3_60_cpu/D21 -> /D21
- U516 pad 16: /sun3_60_cpu/D20 -> /D20
- U516 pad 17: /sun3_60_cpu/D19 -> /D19
- U516 pad 18: /sun3_60_cpu/D18 -> /D18
- U516 pad 19: /sun3_60_cpu/D17 -> /D17
- U516 pad 20: /sun3_60_cpu/D16 -> /D16
- U517 pad 13: /sun3_60_cpu/D31 -> /D31
- U517 pad 14: /sun3_60_cpu/D30 -> /D30
- U517 pad 15: /sun3_60_cpu/D29 -> /D29
- U517 pad 16: /sun3_60_cpu/D28 -> /D28
- U517 pad 17: /sun3_60_cpu/D27 -> /D27
- U517 pad 18: /sun3_60_cpu/D26 -> /D26
- U517 pad 19: /sun3_60_cpu/D25 -> /D25
- U517 pad 20: /sun3_60_cpu/D24 -> /D24
- U710 pad 1: /sun3_60_cpu/D6 -> /D0
- U710 pad 10: /sun3_60_cpu/D2 -> /D5
- U710 pad 11: /sun3_60_cpu/D3 -> VCC
- U710 pad 12: /sun3_60_cpu/D4 -> /D4
- U710 pad 13: /sun3_60_cpu/D5 -> /D3
- U710 pad 14: VCC -> /D2
- U710 pad 2: /sun3_60_cpu/D7 -> /D1
- U710 pad 3: /WRITE- -> /P3
- U710 pad 4: /SCSI 2, Parity/PAR.TEST- -> GND
- U710 pad 6: /P3 -> /WRITE-
- U710 pad 7: GND -> /SCSI 2, Parity/PAR.TEST-
- U710 pad 8: /sun3_60_cpu/D0 -> /D7
- U710 pad 9: /sun3_60_cpu/D1 -> /D6
- U711 pad 1: /sun3_60_cpu/D14 -> /D8
- U711 pad 10: /sun3_60_cpu/D10 -> /D13
- U711 pad 11: /sun3_60_cpu/D11 -> VCC
- U711 pad 12: /sun3_60_cpu/D12 -> /D12
- U711 pad 13: /sun3_60_cpu/D13 -> /D11
- U711 pad 14: VCC -> /D10
- U711 pad 2: /sun3_60_cpu/D15 -> /D9
- U711 pad 3: /WRITE- -> /P2
- U711 pad 4: /SCSI 2, Parity/PAR.TEST- -> GND
- U711 pad 6: /P2 -> /WRITE-
- U711 pad 7: GND -> /WRITE-
- U711 pad 8: /sun3_60_cpu/D8 -> /D15
- U711 pad 9: /sun3_60_cpu/D9 -> /D14
- U712 pad 1: /sun3_60_cpu/D22 -> /D16
- U712 pad 10: /sun3_60_cpu/D18 -> /D21
- U712 pad 11: /sun3_60_cpu/D19 -> VCC
- U712 pad 12: /sun3_60_cpu/D20 -> /D20
- U712 pad 13: /sun3_60_cpu/D21 -> /D19
- U712 pad 14: VCC -> /D18
- U712 pad 2: /sun3_60_cpu/D23 -> /D17
- U712 pad 3: /WRITE- -> /P1
- U712 pad 4: /SCSI 2, Parity/PAR.TEST- -> GND
- U712 pad 6: /P1 -> /WRITE-
- U712 pad 7: GND -> /WRITE-
- U712 pad 8: /sun3_60_cpu/D16 -> /D23
- U712 pad 9: /sun3_60_cpu/D17 -> /D22
- U713 pad 1: /sun3_60_cpu/D30 -> /D24
- U713 pad 10: /sun3_60_cpu/D26 -> /D29
- U713 pad 11: /sun3_60_cpu/D27 -> VCC
- U713 pad 12: /sun3_60_cpu/D28 -> /D28
- U713 pad 13: /sun3_60_cpu/D29 -> /D27
- U713 pad 14: VCC -> /D26
- U713 pad 2: /sun3_60_cpu/D31 -> /D25
- U713 pad 3: /WRITE- -> /P0
- U713 pad 4: /SCSI 2, Parity/PAR.TEST- -> GND
- U713 pad 6: /P0 -> /WRITE-
- U713 pad 7: GND -> /WRITE-
- U713 pad 8: /sun3_60_cpu/D24 -> /D31
- U713 pad 9: /sun3_60_cpu/D25 -> /D30
- U800 pad 5: /S8A Memory/SEL0- -> GND
- U800 pad 6: /S8A Memory/SEL1 -> VCC
- U802 pad 16: /S8A Memory/TWOWAY- -> unconnected-(U802-IO16-Pad16)
- U802 pad 7: /S8A Memory/PA02/22 -> /S8A Memory/PA22
- U900 pad 10: /sun3_60_cpu/D2 -> /D2
- U900 pad 13: /sun3_60_cpu/D3 -> /D3
- U900 pad 16: /sun3_60_cpu/D4 -> /D4
- U900 pad 19: unconnected-(U900-A10-Pad19) -> /SIMMs 1/M.A10.0
- U900 pad 20: /sun3_60_cpu/D5 -> /D5
- U900 pad 23: /sun3_60_cpu/D6 -> /D6
- U900 pad 25: /sun3_60_cpu/D7 -> /D7
- U900 pad 3: /sun3_60_cpu/D0 -> /D0
- U900 pad 6: /sun3_60_cpu/D1 -> /D1
- U901 pad 10: /sun3_60_cpu/D10 -> /D10
- U901 pad 13: /sun3_60_cpu/D11 -> /D11
- U901 pad 16: /sun3_60_cpu/D12 -> /D12
- U901 pad 19: unconnected-(U901-A10-Pad19) -> /SIMMs 1/M.A10.0
- U901 pad 20: /sun3_60_cpu/D13 -> /D13
- U901 pad 23: /sun3_60_cpu/D14 -> /D14
- U901 pad 25: /sun3_60_cpu/D15 -> /D15
- U901 pad 3: /sun3_60_cpu/D8 -> /D8
- U901 pad 6: /sun3_60_cpu/D9 -> /D9
- U902 pad 10: /sun3_60_cpu/D18 -> /D18
- U902 pad 13: /sun3_60_cpu/D19 -> /D19
- U902 pad 16: /sun3_60_cpu/D20 -> /D20
- U902 pad 19: unconnected-(U902-A10-Pad19) -> /SIMMs 1/M.A10.0
- U902 pad 20: /sun3_60_cpu/D21 -> /D21
- U902 pad 23: /sun3_60_cpu/D22 -> /D22
- U902 pad 25: /sun3_60_cpu/D23 -> /D23
- U902 pad 3: /sun3_60_cpu/D16 -> /D16
- U902 pad 6: /sun3_60_cpu/D17 -> /D17
- U903 pad 10: /sun3_60_cpu/D26 -> /D26
- U903 pad 13: /sun3_60_cpu/D27 -> /D27
- U903 pad 16: /sun3_60_cpu/D28 -> /D28
- U903 pad 19: unconnected-(U903-A10-Pad19) -> /SIMMs 1/M.A10.0
- U903 pad 20: /sun3_60_cpu/D29 -> /D29
- U903 pad 23: /sun3_60_cpu/D30 -> /D30
- U903 pad 25: /sun3_60_cpu/D31 -> /D31
- U903 pad 3: /sun3_60_cpu/D24 -> /D24
- U903 pad 6: /sun3_60_cpu/D25 -> /D25
- U905 pad 11: /S8A Memory/PA19 -> /S8A Memory/PA20
- U905 pad 14: /S8A Memory/PA20 -> /S8A Memory/PA18
- U905 pad 5: /S8A Memory/PA18 -> /S8A Memory/PA19
- U906 pad 12: unconnected-(U906-4Y-Pad12) -> /SIMMs 1/M.A9.0
- U906 pad 13: GND -> /Ethernet/A2
- U906 pad 14: GND -> /S8A Memory/PA23
- U906 pad 5: /S8A Memory/PA22/02 -> /S8A Memory/PA22
- U906 pad 7: /SIMMs 1/M.A9.0 -> /SIMMs 1/M.A10.0
- U907 pad 1: /S8A Memory/RAS- -> /S8A Memory/RE02-
- U907 pad 12: /S8A Memory/RE03- -> /S8A Memory/RAS-
- U907 pad 13: /S8A Memory/RAS- -> /S8A Memory/RE03-
- U907 pad 2: /S8A Memory/RE00- -> /S8A Memory/RAS-
- U907 pad 3: /SIMMs 1/XE00- -> /SIMMs 1/XE02-
- U907 pad 5: /S8A Memory/RE01- -> /S8A Memory/RE00-
- U907 pad 6: /SIMMs 1/XE01- -> /SIMMs 1/XE00-
- U907 pad 8: /SIMMs 1/XE02- -> /SIMMs 1/XE01-
- U907 pad 9: /S8A Memory/RE02- -> /S8A Memory/RE01-
- U908 pad 1: /CAS- -> /S8A Memory/CAS0-
- U908 pad 12: /S8A Memory/CAS0- -> /CAS-
- U908 pad 13: /CAS- -> /S8A Memory/CAS0-
- U908 pad 2: /S8A Memory/CAS0- -> /CAS-
Routing:
- net /DIAG-: track 522.8 -> 0.00 mm, vias 6 -> 0
- net /sun3_60_cpu/D27: track 447.3 -> 0.00 mm, vias 8 -> 0
- net /sun3_60_cpu/D25: track 440.4 -> 0.00 mm, vias 9 -> 0
- net /CLK-: track 633.1 -> 195.0 mm, vias 8 -> 4
- net /sun3_60_cpu/D26: track 431.0 -> 0.00 mm, vias 9 -> 0
- net /S8A Memory/M.PU: track 429.2 -> 0.00 mm, vias 1 -> 0
- net /RTC-: track 458.3 -> 29.8 mm, vias 7 -> 0
- net /sun3_60_cpu/D24: track 417.4 -> 0.00 mm, vias 6 -> 0
- net VCC: track 0.00 -> 416.8 mm, vias 0 -> 159
- net /sun3_60_mmu_diag/WR.DIAG-: track 411.6 -> 0.00 mm, vias 3 -> 0
- net /WDOG-: track 411.1 -> 0.00 mm, vias 2 -> 0
- net /sun3_60_cpu/D30: track 404.3 -> 0.00 mm, vias 10 -> 0
- net /D31: track 0.00 -> 396.3 mm, vias 0 -> 6
- net /sun3_60_cpu/BERR.V-: track 476.0 -> 79.8 mm, vias 6 -> 1
- net /RERUN-: track 404.9 -> 9.90 mm, vias 11 -> 1
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Other:
- board size 231.1 x 340.4 mm -> 300 x 400 mm
- board text added: "1"
