File: schematics/kicad/sun3_60.kicad_pcb (KiCad board)
At the start: 4 copper layers, 300 x 400 mm, 306 parts, among them IC1 ATF1504AS-10AU100, IC2 ATF1504AS-10AU100, IC3 ATF1504AS-10AU100, IC4 ATF1504AS-10AU100, IC5 ATF1504AS-10AU100, IC6 ATF1504AS-10AU100, J11 Conn_01x04_Pin, J3 Mini-DIN-8, J5 5747845-4, J6 DB25_Socket, J7 DB25_Socket, K199 10uF tantalum, K500 10uF tantalum, K900 1000uF, K901 1000uF, K903 1000uF, K904 1000uF, T1 TG01-0506NRLTR, U1 IS61C5128AS-25HLI, U10 CBT3257APW, U100 68020, U101 68881, U103 PAL16L8, U104 74F04, U106 PAL16L8, U108 74F00, U11 74CBT3257APW, U110 40.000 Mhz, U115 74LS590, U130 74F374, U131 PAL16R6, U132 ALS244, U14 74LVC1G04, U15 74LVC1G74, U17 74LVC1G74, U199 7705, U2 IS61C5128AS-25HLI, U2003 74AS04, U2004 74LS125, U3 IS61C5128AS-25HLI, U300 27512, U301 AT28C64B_PLCC, U302 7170, U303 32768Hz, U309 3-VOLT, U4 IS61C5128AS-25HLI, U400 Z8530, U401 Z8530, U402 4.9152 Mhz, U404 74ALS04, U500 AM7990, U501 AM7992, U502 20 Mhz, U510 ALS373, U511 ALS373, U512 ALS373, U514 ALS652, U515 ALS652, U516 ALS652, U517 ALS652, U518 PAL16L8, U519 PAL16L8, U520 74F175, U7 IS61C5128AS-25HLI, U710 ACT11286, U711 ACT11286, U712 ACT11286, U713 ACT11286, U720 ALS374, U721 ALS374, U722 ALS374, U723 ALS374, U8 IS61C5128AS-25HLI, U800 PAL16L8, U802 PAL20L8, U803 74F64, U804 74F64, U805 PAL16L8, U900 SIMM, U901 SIMM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

Commit message: ongoing ethernet pld
Parts:
- removed U518, U519: PAL16L8, Package_DIP:DIP-20_W7.62mm
- removed U520: 74F175, Package_SO:SOIC-16_3.9x9.9mm_P1.27mm
- removed X43, X44, X45: 100nF 0402, Capacitor_SMD:C_0402_1005Metric
- added C61: 100nF 0402, Capacitor_SMD:C_0402_1005Metric, F.Cu at (30.2, 237.0)
- added C62: 100nF 0402, Capacitor_SMD:C_0402_1005Metric, F.Cu at (30.2, 229.5)
- added C63: 100nF 0402, Capacitor_SMD:C_0402_1005Metric, F.Cu at (22.0, 221.8)
- added C64: 100nF 0402, Capacitor_SMD:C_0402_1005Metric, F.Cu at (19.5, 221.8)
- added C65: 100nF 0402, Capacitor_SMD:C_0402_1005Metric, F.Cu at (9.75, 226.0)
- added C66: 100nF 0402, Capacitor_SMD:C_0402_1005Metric, F.Cu at (9.75, 233.5)
- added C67: 100nF 0402, Capacitor_SMD:C_0402_1005Metric, F.Cu at (17.0, 242.2)
- added C68: 100nF 0402, Capacitor_SMD:C_0402_1005Metric, F.Cu at (21.5, 242.2)
- added IC8: ATF1504AS-10AU100, sun3_60:QFP50P1600X1600X120-100N, F.Cu at (20.0, 232.0)
- moved J5 283.0 mm to (289.0, 207.0), turned to 90 degrees
- moved T1 252.1 mm to (274.4, 213.4), turned to -90 degrees
Connections:
- IC5 pad 65: unconnected-(IC5-I/O_37-Pad65) -> /E.IRQ-
- IC5 pad 83: /E.IRQ- -> unconnected-(IC5-I/O_47-Pad83)
Routing:
- net /Ethernet/E.RX-: track 47.5 -> 269.0 mm
- net /Ethernet/E.RX+: track 52.9 -> 272.7 mm
- net /Ethernet/E.TX-: track 31.2 -> 246.4 mm
- net /Ethernet/E.TX+: track 35.9 -> 247.6 mm
- net /Ethernet/E.CO-: track 61.6 -> 259.4 mm
- net /Ethernet/E.CO+: track 65.8 -> 260.7 mm
- net /E.HOLD-: track 0.00 -> 121.8 mm, vias 0 -> 1
- net /Ethernet/E.GBA0-: track 29.9 -> 149.1 mm
- net /Ethernet/E.GAB: track 61.2 -> 164.3 mm
- net /Ethernet/E.GBA1-: track 23.9 -> 120.7 mm
- net /Ethernet/E.CBA: track 87.5 -> 182.7 mm
- net /E.IRQ-: track 0.00 -> 89.2 mm, vias 0 -> 1
- net /Ethernet/E.WE-: track 0.00 -> 51.9 mm
- net /E.ACK-: track 36.6 -> 86.4 mm
- net /Ethernet/E.DAS-: track 0.00 -> 41.7 mm
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
Commit message: ongoing
Parts:
- removed C300: 18-PF, Capacitor_THT:C_Disc_D3.0mm_W2.0mm_P2.50mm
- removed C301: 9-35PF, Capacitor_THT:C_Radial_D6.3mm_H5.0mm_P2.50mm
- removed C500, C501: 20 pF, Capacitor_THT:C_Rect_L7.0mm_W2.0mm_P5.00mm
- removed R300: 200Kohm, Resistor_THT:R_Axial_DIN0207_L6.3mm_D2.5mm_P7.62mm_Horizontal
- removed U303: 32768Hz, Crystal:Crystal_AT310_D3.0mm_L10.0mm_Horizontal
- removed U502: 20 Mhz, Crystal:Crystal_HC49-U_Vertical
- added U16: 20 MHz, Oscillator:Oscillator_SMD_SeikoEpson_SG8002LB-4Pin_5.0x3.2mm, F.Cu at (30.0, 218.9)
- added X53: 100nF 0402, Capacitor_SMD:C_0402_1005Metric, F.Cu at (232.5, 154.0)
- added X54: 10nF 0402, Capacitor_SMD:C_0402_1005Metric, F.Cu at (235.0, 154.0)
- added X55: 100nF 0402, Capacitor_SMD:C_0402_1005Metric, F.Cu at (28.2, 215.5)
- added X56: 10nF 0402, Capacitor_SMD:C_0402_1005Metric, F.Cu at (25.8, 217.3)
- added X57: 100nF 0402, Capacitor_SMD:C_0402_1005Metric, F.Cu at (87.8, 145.9)
- added X58: 10nF 0402, Capacitor_SMD:C_0402_1005Metric, F.Cu at (85.4, 148.2)
- added Y1: SiT8008xx-2x-xxS, Crystal:Crystal_SMD_3225-4Pin_3.2x2.5mm, F.Cu at (84.8, 145.5)
- C502, C505: footprint Capacitor_THT:C_Rect_L7.0mm_W2.0mm_P5.00mm -> Capacitor_SMD:C_0402_1005Metric
- R301: footprint Resistor_THT:R_Axial_DIN0207_L6.3mm_D2.5mm_P7.62mm_Horizontal -> Capacitor_SMD:C_0402_1005Metric
- R501, R502: footprint Resistor_THT:R_Axial_DIN0207_L6.3mm_D2.5mm_P7.62mm_Horizontal -> Resistor_SMD:R_0402_1005Metric
- U309: footprint Battery:Battery_Panasonic_CR2032-VS1N_Vertical_CircularHoles -> Battery:BatteryHolder_MYOUNG_BS-07-A1BJ001_CR2032
- X301: footprint Capacitor_THT:CP_Radial_D10.0mm_P5.00mm -> Capacitor_SMD:CP_Elec_6.3x7.7
- moved K904 613.1 mm to (-70.8, 417.5)
- moved K903 559.2 mm to (-80.8, 400.0)
- moved R502 435.4 mm to (32.0, 211.5)
- moved C502 419.4 mm to (31.0, 212.8)
- moved C503 399.8 mm to (46.0, 215.2), turned to 0 degrees
- moved R501 392.9 mm to (32.0, 210.2), turned to 180 degrees
- moved K500 389.9 mm to (47.2, 212.7)
- moved C504 388.4 mm to (46.0, 220.3), turned to 0 degrees
- moved C505 380.1 mm to (46.0, 217.8), turned to 0 degrees
- moved U402 245.4 mm to (237.5, 142.2), turned to 180 degrees
- moved R301 214.3 mm to (84.8, 270.0), turned to 90 degrees
- moved X301 210.6 mm to (90.0, 266.5)
- moved U309 203.8 mm to (57.9, 269.5)
- moved K900 189.6 mm to (-48.8, 428.8)
- moved X24 0.89 mm to (46.5, 152.8), turned to 90 degrees
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Connections:
- IC5 pad 10: /sun3_60_eeprom/RSVD3 -> unconnected-(IC5-I/O_4-Pad10)
- IC5 pad 12: unconnected-(IC5-I/O/PD1-Pad12) -> /sun3_60_eeprom/RSVD1
- IC5 pad 13: /sun3_60_eeprom/RSVD4 -> /sun3_60_eeprom/RSVD2
- IC5 pad 14: /sun3_60_eeprom/RSVD5 -> /sun3_60_eeprom/RSVD3
- IC5 pad 16: unconnected-(IC5-I/O_7-Pad16) -> /sun3_60_eeprom/RSVD4
- IC5 pad 17: unconnected-(IC5-I/O_8-Pad17) -> /sun3_60_eeprom/RSVD5
- IC5 pad 21: /V.INT- -> unconnected-(IC5-I/O_11-Pad21)
- IC5 pad 8: /sun3_60_eeprom/RSVD1 -> unconnected-(IC5-I/O_2-Pad8)
- IC5 pad 9: /sun3_60_eeprom/RSVD2 -> unconnected-(IC5-I/O_3-Pad9)
- IC5 pad 96: /RESET- -> /V.INT-
- IC5 pad 97: unconnected-(IC5-I/O_53-Pad97) -> /RESET-
- IC8 pad 35: unconnected-(IC8-I/O_19-Pad35) -> /E.REQ-
- IC8 pad 65: /R/W- -> unconnected-(IC8-I/O_37-Pad65)
- IC8 pad 94: /E.REQ- -> unconnected-(IC8-I/O_51-Pad94)
- U302 pad 10: Net-(U302-OIN) -> /sun3_60_eeprom/CMCLK_32768_RTC
- U302 pad 9: Net-(U302-OOUT) -> unconnected-(U302-OOUT-Pad9)
- U501 pad 8: Net-(U501-X1) -> /Ethernet/CLK_20MHZ_ETH
- U501 pad 9: Net-(U501-X2) -> unconnected-(U501-X2-Pad9)
Routing:
- net /E.REQ-: track 1.40 -> 435.3 mm, vias 1 -> 4
- net /E.ACK-: track 86.4 -> 515.6 mm, vias 2 -> 4
- net /CLK-: track 169.2 -> 543.1 mm
- net /V.INT-: track 0.00 -> 267.5 mm, vias 0 -> 2
- net /RESET-: track 76.2 -> 199.2 mm, vias 1 -> 3
- net VCC: track 435.8 -> 483.4 mm, vias 166 -> 177
- net /sun3_60_eeprom/CMCLK_32768_RTC: track 0.00 -> 20.3 mm, vias 0 -> 1
- net GND: track 371.8 -> 384.7 mm, vias 236 -> 248
- net /sun3_60_serial/SERIAL_PCLK: track 23.4 -> 29.0 mm
- net Net-(U501-TSEL): track 0.00 -> 3.83 mm
- net /Ethernet/CLK_20MHZ_ETH: track 0.00 -> 3.73 mm
- net /WRITE-: track 293.2 -> 296.6 mm
- net Net-(U501-RF): track 0.00 -> 2.90 mm
- net Net-(U501-PF): track 0.00 -> 2.90 mm
- net /CAS-: track 295.9 -> 293.9 mm
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
Commit message: update (lost cause?)
Parts:
- added R70: 4.7k, Resistor_SMD:R_0402_1005Metric, F.Cu at (143.5, 7.00)
- added R71: 4.7k, Resistor_SMD:R_0402_1005Metric, F.Cu at (156.2, 37.5)
- added R72: 4.7k, Resistor_SMD:R_0402_1005Metric, F.Cu at (172.2, 166.8)
- added R75: 4.7k, Resistor_SMD:R_0402_1005Metric, F.Cu at (206.0, 14.2)
- added R76: 4.7k, Resistor_SMD:R_0402_1005Metric, F.Cu at (49.8, 137.8)
- added R77: 4.7k, Resistor_SMD:R_0402_1005Metric, F.Cu at (49.8, 136.5)
- added R78: 4.7k, Resistor_SMD:R_0402_1005Metric, F.Cu at (204.8, 14.2)
- U14: footprint Package_TO_SOT_SMD:SOT-353_SC-70-5 -> Package_TO_SOT_SMD:SOT-23-5
- moved R100 1.92 mm to (129.3, 179.8), turned to 0 degrees
- moved R101 1.92 mm to (129.3, 176.8), turned to 180 degrees
- moved X42 0.31 mm to (188.3, 48.8)
- turned X88 to 180 degrees
- turned X89 to 180 degrees
- turned X90 to 180 degrees
Connections:
- IC8 pad 16: unconnected-(IC8-I/O_7-Pad16) -> /DSACK1-
- IC8 pad 17: unconnected-(IC8-I/O_8-Pad17) -> /R/W-
- IC8 pad 19: unconnected-(IC8-I/O_9-Pad19) -> /SIZ1
- IC8 pad 20: unconnected-(IC8-I/O_10-Pad20) -> /SIZ0
- IC8 pad 58: unconnected-(IC8-I/O_32-Pad58) -> /EN.E-
- IC8 pad 6: /EN.E- -> unconnected-(IC8-I/O_1-Pad6)
- IC8 pad 60: /DSACK1- -> unconnected-(IC8-I/O_33-Pad60)
- IC8 pad 61: /R/W- -> unconnected-(IC8-I/O_34-Pad61)
- IC8 pad 63: /SIZ1 -> unconnected-(IC8-I/O_35-Pad63)
- IC8 pad 64: /SIZ0 -> unconnected-(IC8-I/O_36-Pad64)
- U15 pad 6: /PU3 -> /sun3_60_cpu/PU.3a
- U15 pad 7: /PU2 -> /sun3_60_cpu/PU.2a
- U17 pad 6: /PU3 -> /sun3_60_cpu/PU.3b
- U17 pad 7: /PU2 -> /sun3_60_cpu/PU.2b
- U800 pad 11: /S8A Memory/M.PD- -> /S8A Memory/M.PDa-
- U802 pad 23: /S8A Memory/M.PD- -> /S8A Memory/M.PDb-
- U805 pad 5: /S8A Memory/M.PD- -> /S8A Memory/M.PDc-
- U904 pad 15: /S8A Memory/M.PD- -> GND
- U905 pad 15: /S8A Memory/M.PD- -> GND
- U906 pad 15: /S8A Memory/M.PD- -> GND
- U924 pad 15: /S8A Memory/M.PD- -> GND
- U925 pad 15: /S8A Memory/M.PD- -> GND
- U926 pad 15: /S8A Memory/M.PD- -> GND
Routing:
- net /EN.E-: track 0.00 -> 389.1 mm
- net /S8A Memory/M.PD-: track 61.9 -> 0.00 mm, vias 2 -> 0
- net GND: track 384.7 -> 425.0 mm, vias 248 -> 259
- net /sun3_60_cpu/BR-: track 0.00 -> 17.0 mm
- net /sun3_60_cpu/BG-: track 0.00 -> 14.0 mm
- net /sun3_60_cpu/BACK-: track 0.00 -> 11.5 mm
- net VCC: track 483.4 -> 489.2 mm, vias 177 -> 175
- net /sun3_60_cpu/PU.3b: track 0.00 -> 3.74 mm
- net /sun3_60_cpu/PU.2b: track 0.00 -> 3.43 mm
- net /sun3_60_cpu/PU.3a: track 0.00 -> 3.26 mm
- net /sun3_60_cpu/PU.2a: track 0.00 -> 2.80 mm
- net /S8A Memory/M.PDc-: track 0.00 -> 2.24 mm
- net /S8A Memory/M.PDb-: track 0.00 -> 2.12 mm
- net /S8A Memory/M.PDa-: track 0.00 -> 1.99 mm
- net /sun3_60_cpu/CLK1: track 300.2 -> 299.3 mm
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