File: schematics/kicad/sun3_60_FIRST_DRAFT_NOT_FINISHED.kicad_pcb (KiCad board)
At the start: 4 copper layers, 300 x 400 mm, 306 parts, among them IC1 ATF1504AS-10AU100, IC2 ATF1504AS-10AU100, IC3 ATF1504AS-10AU100, IC4 ATF1504AS-10AU100, IC5 ATF1504AS-10AU100, IC6 ATF1504AS-10AU100, J11 Conn_01x04_Pin, J3 Mini-DIN-8, J5 5747845-4, J6 DB25_Socket, J7 DB25_Socket, K199 10uF tantalum, K500 10uF tantalum, K900 1000uF, K901 1000uF, K903 1000uF, K904 1000uF, T1 TG01-0506NRLTR, U1 IS61C5128AS-25HLI, U10 CBT3257APW, U100 68020, U101 68881, U103 PAL16L8, U104 74F04, U106 PAL16L8, U108 74F00, U11 74CBT3257APW, U110 40.000 Mhz, U115 74LS590, U130 74F374, U131 PAL16R6, U132 ALS244, U14 74LVC1G04, U15 74LVC1G74, U17 74LVC1G74, U199 7705, U2 IS61C5128AS-25HLI, U2003 74AS04, U2004 74LS125, U3 IS61C5128AS-25HLI, U300 27512, U301 AT28C64B_PLCC, U302 7170, U303 32768Hz, U309 3-VOLT, U4 IS61C5128AS-25HLI, U400 Z8530, U401 Z8530, U402 4.9152 Mhz, U404 74ALS04, U500 AM7990, U501 AM7992, U502 20 Mhz, U510 ALS373, U511 ALS373, U512 ALS373, U514 ALS652, U515 ALS652, U516 ALS652, U517 ALS652, U518 PAL16L8, U519 PAL16L8, U520 74F175, U7 IS61C5128AS-25HLI, U710 ACT11286, U711 ACT11286, U712 ACT11286, U713 ACT11286, U720 ALS374, U721 ALS374, U722 ALS374, U723 ALS374, U8 IS61C5128AS-25HLI, U800 PAL16L8, U802 PAL20L8, U803 74F64, U804 74F64, U805 PAL16L8, U900 SIMM, U901 SIMM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

Commit message: update
Parts:
- removed C37, C38, C39, C40, C41, C42, C43, C44, C45, C46, C47, C48, C49, C50, C51, C52, X50, X51, X52: 100nF 0402, Capacitor_SMD:C_0402_1005Metric
- removed IC5, IC6: ATF1504AS-10AU100, sun3_60:QFP50P1600X1600X120-100N
- removed J5: 5747845-4, sun3_60:57478454
- removed J6, J7: DB25_Socket, sun3_60:D25S33E4PA00LF
- removed T1: TG01-0506NRLTR, sun3_60:TG010506NRLTR
- removed U15, U17: 74LVC1G74, sun3_60:74AVC9112GTX
- removed U400: Z8530, Package_DIP:DIP-40_W15.24mm
- removed U404: 74ALS04, Package_SO:SOIC-14_3.9x8.7mm_P1.27mm
- added J2: Serial A/B, Connector_PinHeader_2.54mm:PinHeader_1x05_P2.54mm_Vertical, F.Cu at (448.3, 364.2)
- added U107: PAL20X10, Package_DIP:DIP-24_W7.62mm, F.Cu at (230.0, 38.0)
- added U113: 74AS74, Package_SO:SOIC-14_3.9x8.7mm_P1.27mm, F.Cu at (210.0, 10.0)
- added U114: 74F175, Package_SO:SOIC-16_3.9x9.9mm_P1.27mm, F.Cu at (162.0, 23.0)
- added U122: ALS374, Package_SO:SOIC-20W_7.5x12.8mm_P1.27mm, F.Cu at (67.5, 134.5)
- added U123: ALS373, Package_SO:SOIC-20W_7.5x12.8mm_P1.27mm, F.Cu at (67.5, 117.5)
- added U13: 74LVC1G04, Package_TO_SOT_SMD:SOT-353_SC-70-5, F.Cu at (58.5, 140.1)
- added U224: AM27S19, sun3_60:AM27S19, F.Cu at (233.3, 83.1)
- added U227: ALS273, Package_SO:SOIC-20W_7.5x12.8mm_P1.27mm, F.Cu at (198.0, 199.0)
- added U304: ALS273, Package_SO:SOIC-20W_7.5x12.8mm_P1.27mm, F.Cu at (59.0, 199.0)
- added U305: ALS373, Package_SO:SOIC-20W_7.5x12.8mm_P1.27mm, F.Cu at (74.5, 199.0)
- added U307: PAL20L8, Package_DIP:DIP-24_W7.62mm, F.Cu at (81.2, 181.0)
- added U503: TRANSF, Package_DIP:DIP-16_W7.62mm, F.Cu at (50.0, 212.0)
- added U714: PAL16L8, Package_DIP:DIP-20_W7.62mm, F.Cu at (67.0, 220.0)
- added U715: PAL20R4, Package_DIP:DIP-24_W7.62mm, F.Cu at (81.2, 169.5)
- added X19: 100nF 0402, Capacitor_SMD:C_0402_1005Metric, F.Cu at (167.2, 18.6)
- added X21: 100nF 0402, Capacitor_SMD:C_0402_1005Metric, F.Cu at (75.8, 139.2)
- added X22: 100nF 0402, Capacitor_SMD:C_0402_1005Metric, F.Cu at (75.8, 122.2)
- added X31: 100nF 0402, Capacitor_SMD:C_0402_1005Metric, F.Cu at (66.8, 193.3)
- added X32: 100nF 0402, Capacitor_SMD:C_0402_1005Metric, F.Cu at (82.2, 193.3)
- added X37: 100nF 0402, Capacitor_SMD:C_0402_1005Metric, F.Cu at (56.1, 139.6)
- added X38: 100nF 0402, Capacitor_SMD:C_0402_1005Metric, F.Cu at (84.5, 177.1)
- added X48: 100nF 0402, Capacitor_SMD:C_0402_1005Metric, F.Cu at (221.9, 40.5)
- added X49: 100nF 0402, Capacitor_SMD:C_0402_1005Metric, F.Cu at (205.5, 193.3)
- J3: value Mini-DIN-8 -> Ethernet; footprint sun3_60:57492681 -> Connector_PinHeader_2.54mm:PinHeader_1x09_P2.54mm_Vertical
- U199: footprint Package_SO:SOIC-8_3.9x4.9mm_P1.27mm -> Package_DIP:DIP-8_W7.62mm
- U301: value AT28C64B_PLCC -> 28C16; footprint Package_LCC:PLCC-32_THT-Socket -> Package_DIP:DIP-24_W15.24mm
- moved J3 209.1 mm to (88.0, 230.0)
- moved R69 186.2 mm to (215.0, 205.0), turned to 0 degrees
- moved R68 184.0 mm to (215.0, 203.0), turned to 0 degrees
- moved R67 181.8 mm to (215.0, 201.0), turned to 0 degrees
- moved D8 180.5 mm to (211.5, 205.0), turned to 0 degrees
- moved R66 179.7 mm to (215.0, 199.0), turned to 0 degrees
- moved D7 178.2 mm to (211.5, 203.0), turned to 0 degrees
- moved R65 177.6 mm to (215.0, 197.0), turned to 0 degrees
- moved D6 175.9 mm to (211.5, 201.0), turned to 0 degrees
- moved R64 175.6 mm to (215.0, 195.0), turned to 0 degrees
- moved D5 173.7 mm to (211.5, 199.0), turned to 0 degrees
- moved R63 173.7 mm to (215.0, 193.0), turned to 0 degrees
- moved R62 171.8 mm to (215.0, 191.0), turned to 0 degrees
- moved D4 171.6 mm to (211.5, 197.0), turned to 0 degrees
- moved D3 169.5 mm to (211.5, 195.0), turned to 0 degrees
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Connections:
- net /D0 renamed /sun3_60_cpu/D0
- net /D1 renamed /sun3_60_cpu/D1
- net /D10 renamed /sun3_60_cpu/D10
- net /D11 renamed /sun3_60_cpu/D11
- net /D12 renamed /sun3_60_cpu/D12
- net /D13 renamed /sun3_60_cpu/D13
- net /D14 renamed /sun3_60_cpu/D14
- net /D15 renamed /sun3_60_cpu/D15
- net /D16 renamed /sun3_60_cpu/D16
- net /D17 renamed /sun3_60_cpu/D17
- net /D18 renamed /sun3_60_cpu/D18
- net /D19 renamed /sun3_60_cpu/D19
- net /D2 renamed /sun3_60_cpu/D2
- net /D20 renamed /sun3_60_cpu/D20
- net /D21 renamed /sun3_60_cpu/D21
- net /D22 renamed /sun3_60_cpu/D22
- net /D23 renamed /sun3_60_cpu/D23
- net /D24 renamed /sun3_60_cpu/D24
- net /D25 renamed /sun3_60_cpu/D25
- net /D26 renamed /sun3_60_cpu/D26
- net /D27 renamed /sun3_60_cpu/D27
- net /D28 renamed /sun3_60_cpu/D28
- net /D29 renamed /sun3_60_cpu/D29
- net /D3 renamed /sun3_60_cpu/D3
- net /D30 renamed /sun3_60_cpu/D30
- net /D31 renamed /sun3_60_cpu/D31
- net /D4 renamed /sun3_60_cpu/D4
- net /D5 renamed /sun3_60_cpu/D5
- net /D6 renamed /sun3_60_cpu/D6
- net /D7 renamed /sun3_60_cpu/D7
- net /D8 renamed /sun3_60_cpu/D8
- net /D9 renamed /sun3_60_cpu/D9
- net /sun3_60_serial/SERIAL_PCLK renamed Net-(U401-PCLK)
- D1 pad 1: /sun3_60_eeprom/LED0 -> /sun3_60_mmu_diag/LED0
- D2 pad 1: /sun3_60_eeprom/LED1 -> /sun3_60_mmu_diag/LED1
- D3 pad 1: /sun3_60_eeprom/LED2 -> /sun3_60_mmu_diag/LED2
- D4 pad 1: /sun3_60_eeprom/LED3 -> /sun3_60_mmu_diag/LED3
- D5 pad 1: /sun3_60_eeprom/LED4 -> /sun3_60_mmu_diag/LED4
- D6 pad 1: /sun3_60_eeprom/LED5 -> /sun3_60_mmu_diag/LED5
- D7 pad 1: /sun3_60_eeprom/LED6 -> /sun3_60_mmu_diag/LED6
- D8 pad 1: /sun3_60_eeprom/LED7 -> /sun3_60_mmu_diag/LED7
- IC1 pad 100: ENABLE_S3E -> unconnected-(IC1-I/O_56-Pad100)
- IC1 pad 35: unconnected-(IC1-I/O_19-Pad35) -> /sun3_60_mmu_diag/RD.ID-
- IC1 pad 8: /sun3_60_mmu_diag/RD.ID- -> ENABLE_S3E
- IC3 pad 10: /Ethernet/A2 -> unconnected-(IC3-I/O_4-Pad10)
- IC3 pad 12: /WDOG- -> unconnected-(IC3-I/O/PD1-Pad12)
- IC3 pad 13: /Ethernet/A1 -> unconnected-(IC3-I/O_5-Pad13)
- IC3 pad 14: /Ethernet/A0 -> unconnected-(IC3-I/O_6-Pad14)
- IC3 pad 16: /INIT- -> unconnected-(IC3-I/O_7-Pad16)
- IC3 pad 17: /BERR.T- -> /sun3_60_cpu/BERR.T-
- IC3 pad 19: /sun3_60_mmu_diag/RD.ID- -> unconnected-(IC3-I/O_9-Pad19)
- IC3 pad 6: unconnected-(IC3-I/O_1-Pad6) -> /INIT-
- IC3 pad 68: unconnected-(IC3-I/O_39-Pad68) -> /WDOG-
- IC3 pad 8: /Ethernet/A4 -> unconnected-(IC3-I/O_2-Pad8)
- IC3 pad 9: /Ethernet/A3 -> unconnected-(IC3-I/O_3-Pad9)
- IC3 pad 92: /sun3_60_cpu/EN.FPP -> unconnected-(IC3-I/O_49-Pad92)
- IC3 pad 93: /sun3_60_mmu_diag/EN.VIDEO -> unconnected-(IC3-I/O_50-Pad93)
- IC3 pad 97: unconnected-(IC3-I/O_53-Pad97) -> /sun3_60_cpu/EN.FPP
- IC3 pad 99: unconnected-(IC3-I/O_55-Pad99) -> /sun3_60_mmu_diag/EN.VIDEO
- IC4 pad 10: /sun3_60_eeprom/RD.SCC1- -> /EN.UART-
- IC4 pad 100: /SCSI 2, Parity/WR_PARX- -> /sun3_60_eeprom/WR.INT-
- IC4 pad 12: /sun3_60_eeprom/RD.SCC0- -> unconnected-(IC4-I/O/PD1-Pad12)
- IC4 pad 13: /sun3_60_eeprom/WR.SCC0- -> unconnected-(IC4-I/O_5-Pad13)
- IC4 pad 14: /HALT- -> unconnected-(IC4-I/O_6-Pad14)
- IC4 pad 16: /sun3_60_eeprom/RD.INT- -> unconnected-(IC4-I/O_7-Pad16)
- IC4 pad 17: /sun3_60_eeprom/WR.INT- -> unconnected-(IC4-I/O_8-Pad17)
- IC4 pad 19: /sun3_60_eeprom/RD.RTC- -> /sun3_60_eeprom/WR.EEPROM-
- IC4 pad 20: /sun3_60_eeprom/WR.RTC- -> /sun3_60_eeprom/RD.EEPROM-
- IC4 pad 29: /sun3_60_eeprom/EN.S- -> unconnected-(IC4-I/O_14-Pad29)
- IC4 pad 30: /sun3_60_eeprom/EN.V- -> /sun3_60_eeprom/EN.IO-
- IC4 pad 33: unconnected-(IC4-I/O_18-Pad33) -> /SCSI 2, Parity/RD.PAR0-
- IC4 pad 35: unconnected-(IC4-I/O_19-Pad35) -> /SCSI 2, Parity/WR.PAR0-
- IC4 pad 36: unconnected-(IC4-I/O_20-Pad36) -> /SCSI 2, Parity/RD.PAR4-
- IC4 pad 37: unconnected-(IC4-I/O_21-Pad37) -> /SCSI 2, Parity/RD.PAR5-
- IC4 pad 40: unconnected-(IC4-I/O_22-Pad40) -> /SCSI 2, Parity/RD.PAR6-
- IC4 pad 41: unconnected-(IC4-I/0-Pad41) -> /SCSI 2, Parity/RD.PAR7-
- IC4 pad 42: unconnected-(IC4-I/O/PD2-Pad42) -> /SCSI 2, Parity/WR.PAR4-
- IC4 pad 45: /EN.E- -> unconnected-(IC4-I/O_24-Pad45)
- IC4 pad 46: unconnected-(IC4-I/O_25-Pad46) -> /IOLOCK-
- IC4 pad 47: /EN.CAS -> /EN.E-
- IC4 pad 48: /C.S5 -> unconnected-(IC4-I/O_27-Pad48)
- IC4 pad 52: /IOLOCK- -> /sun3_60_cpu/C.S9-
- IC4 pad 54: /sun3_60_cpu/C.S9- -> /sun3_60_eeprom/WR.SCC0-
- IC4 pad 56: unconnected-(IC4-I/O_30-Pad56) -> /sun3_60_eeprom/EN.S-
- IC4 pad 57: unconnected-(IC4-I/O_31-Pad57) -> /sun3_60_eeprom/RD.SCC0-
- IC4 pad 58: /POR- -> /sun3_60_eeprom/EN.V-
- IC4 pad 6: /BERR.T- -> unconnected-(IC4-I/O_1-Pad6)
- IC4 pad 60: /C.S3 -> /EN.CAS
- IC4 pad 61: /AS -> unconnected-(IC4-I/O_34-Pad61)
- IC4 pad 65: unconnected-(IC4-I/O_37-Pad65) -> /Ethernet/A2
- IC4 pad 75: unconnected-(IC4-I/O_42-Pad75) -> /Ethernet/A0
- IC4 pad 76: /WDOG- -> /Ethernet/A1
- IC4 pad 8: /EN.UART- -> /sun3_60_eeprom/RD.SCC1-
- IC4 pad 81: /sun3_60_eeprom/C.S7 -> unconnected-(IC4-I/O_46-Pad81)
- IC4 pad 90: /CLK- -> unconnected-(IC4-INPUT/GCLK2-Pad90)
- IC4 pad 97: /sun3_60_eeprom/RD.EEPROM- -> /sun3_60_eeprom/RD.RTC-
- IC4 pad 98: /sun3_60_eeprom/WR.EEPROM- -> /sun3_60_eeprom/WR.RTC-
- IC4 pad 99: /SCSI 2, Parity/RD_PARX- -> /sun3_60_eeprom/RD.INT-
- J3 pad 1: GND -> +12V
- J3 pad 2: GND -> /Ethernet/E.CO+<>
- J3 pad 3: VCC -> /Ethernet/E.CO-<>
- J3 pad 4: /sun3_60_serial/RxDB -> /Ethernet/E.RX+<>
- J3 pad 5: /sun3_60_serial/TxDA -> /Ethernet/E.RX-<>
- J3 pad 6: /sun3_60_serial/RxDA -> /Ethernet/E.TX+<>
- J3 pad 7: /sun3_60_serial/TxDB -> /Ethernet/E.TX-<>
- J3 pad 8: VCC -> /Ethernet/E.SMS
- U106 pad 3: /BERR.T- -> /sun3_60_cpu/BERR.T-
- U2004 pad 3: /DSACK1- -> /DSACK0-
- U2004 pad 6: /DSACK0- -> /DSACK1-
- U301 pad 1: unconnected-(U301-DC-Pad1) -> /Ethernet/A7
- U301 pad 10: /Ethernet/A1 -> /SCSI 2, Parity/IO.D1
- U301 pad 11: /Ethernet/A0 -> /SCSI 2, Parity/IO.D2
- U301 pad 12: unconnected-(U301-NC-Pad12) -> GND
- U301 pad 15: /SCSI 2, Parity/IO.D2 -> /SCSI 2, Parity/IO.D5
- U301 pad 16: GND -> /SCSI 2, Parity/IO.D6
- U301 pad 17: unconnected-(U301-DC-Pad17) -> /SCSI 2, Parity/IO.D7
- U301 pad 18: /SCSI 2, Parity/IO.D5 -> GND
- U301 pad 19: /SCSI 2, Parity/IO.D1 -> /Ethernet/A10
- U301 pad 2: unconnected-(U301-NC-Pad2) -> /Ethernet/A6
- U301 pad 20: /SCSI 2, Parity/IO.D6 -> /sun3_60_eeprom/RD.EEPROM-
- U301 pad 21: /SCSI 2, Parity/IO.D7 -> /sun3_60_eeprom/WR.EEPROM-
- U301 pad 22: /SCSI 2, Parity/IO.D0 -> /Ethernet/A9
- U301 pad 23: GND -> /Ethernet/A8
- U301 pad 24: /Ethernet/A8 -> VCC
- U301 pad 3: GND -> /Ethernet/A5
- U301 pad 4: /Ethernet/A7 -> /Ethernet/A4
- U301 pad 5: /Ethernet/A6 -> /Ethernet/A3
- U301 pad 6: /Ethernet/A5 -> /Ethernet/A2
- U301 pad 7: /Ethernet/A4 -> /Ethernet/A1
- U301 pad 8: /Ethernet/A3 -> /Ethernet/A0
- U301 pad 9: /Ethernet/A2 -> /SCSI 2, Parity/IO.D0
- U401 pad 13: /sun3_60_serial/RXDC -> Net-(J2-Pin_3)
- U401 pad 15: /sun3_60_serial/TXDC -> Net-(J2-Pin_2)
- U401 pad 25: /sun3_60_serial/TXDD -> Net-(J2-Pin_4)
- U401 pad 27: /sun3_60_serial/RXDD -> Net-(J2-Pin_5)
Routing:
- net /E.ACK-: track 36.6 -> 516.3 mm, vias 2 -> 6
- net /CLK: track 505.6 -> 88.5 mm, vias 3 -> 1
- net /E.HOLD-: track 0.00 -> 413.7 mm, vias 0 -> 2
- net /E.REQ-: track 1.40 -> 358.3 mm
- net /SCSI 2, Parity/WR_PARX-: track 349.9 -> 0.00 mm
- net /INIT-: track 455.6 -> 106.0 mm, vias 6 -> 1
- net /SCSI 2, Parity/RD_PARX-: track 346.4 -> 0.00 mm
- net /sun3_60_eeprom/RD.EEPROM-: track 331.5 -> 0.00 mm
- net /sun3_60_eeprom/WR.EEPROM-: track 330.7 -> 0.00 mm
- net /RERUN-: track 9.90 -> 335.4 mm, vias 1 -> 4
- net /EN.E-: track 0.00 -> 289.6 mm, vias 0 -> 2
- net /IOLOCK-: track 324.3 -> 43.4 mm
- net /E.CS-: track 208.0 -> 475.3 mm, vias 5 -> 2
- net /SCC.IRQ-: track 258.3 -> 0.00 mm, vias 3 -> 0
- net /Ethernet/A12: track 413.2 -> 172.0 mm, vias 5 -> 3
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