File: schematics/kicad/sun3_60_mmu_diag.kicad_sch (KiCad schematic)
At the start: 37 parts, among them SW1 SW_SPDT, SW2 SW_SPDT, U1 IS61C5128AS-25HLI, U10 74CBTLV3257, U11 74CBTLV3257, U12 ALS245, U2 IS61C5128AS-25HLI, U210 LS2518, U212 ALS245, U213 ALS245, U215 ALS245, U217 ALS245, U218 ALS245, U223 74F534, U224 AM27S19, U225 ALS273, U226 ALS373, U227 ALS273, U228 LED_Block, U229 LED_Block, U230 PAL16L8, U231 PAL16L8, U232 PAL16L8, U3 IS61C5128AS-25HLI, U4 IS61C5128AS-25HLI, U5 ALS245, U6 IS61C5128AS-25HLI, U7 IS61C5128AS-25HLI, U8 IS61C5128AS-25HLI, U9 LS2518

Commit message: draft, ugly and WiP
Parts:
- removed S3: 4.7k Ohm, Resistor_THT:R_Array_SIP10, symbol Device:R_Network09
- removed SW1, SW2: SW_SPDT, symbol Switch:SW_SPDT
- added C10, C11, C12, C13, C14, C15, C16, C17, C18, C19, C20, C21, C22, C23, C24, C25, C26, C27, C28, C29, C6, C7, C8, C9, X1, X100, X101, X102, X103, X105, X107, X108, X109, X3, X4, X49, X91, X93, X95, X97, X99: 100nF 0402, Capacitor_SMD:C_0402_1005Metric, symbol Device:C
- added IC1, IC2, IC3: ATF1504AS-10AU100, sun3_60:QFP50P1600X1600X120-100N, symbol ATF1504AS-10AU100:ATF1504AS-10AU100
- added R54, R55, R56, R57, R58, R59, R60, R61: 4.7k, Resistor_SMD:R_0402_1005Metric, symbol Device:R
- added S1, S2: SSAJ110100, SW_SSAJ110100, symbol SSAJ110100:SSAJ110100
- added X104, X106, X92, X94, X96, X98: 10nF 0402, Capacitor_SMD:C_0402_1005Metric, symbol Device:C
- R1, R2, R3, R4, R5: footprint (none) -> Resistor_SMD:R_0402_1005Metric; MPN (none) -> 0402WGF1002TCE
- S200, U210, U224, U228, U229, U230, U231, U232, U9: now not fitted; now left out of the parts list
- U1, U2, U3, U4, U7, U8: MPN (none) -> IS61C5128AS-25HLI
- U10: value 74CBTLV3257 -> CBT3257APW; footprint (none) -> Package_SO:TSSOP-16_4.4x5mm_P0.65mm; MPN (none) -> SN74CBT3257CDR; MPN-ALT (none) -> CBT3257APW,118
- U11: value 74CBTLV3257 -> 74CBT3257APW; footprint (none) -> Package_SO:TSSOP-16_4.4x5mm_P0.65mm; MPN (none) -> SN74CBT3257CDR; MPN-ALT (none) -> CBT3257APW,118
- U212, U213, U215, U217, U218, U5: footprint sun3_60:ALS245 -> Package_SO:SOIC-20W_7.5x12.8mm_P1.27mm; MPN (none) -> SN74ALS245ADWR; now not fitted; now left out of the parts list
- U223: footprint Package_DIP:DIP-20_W7.62mm -> Package_SO:SOIC-20W_7.5x12.8mm_P1.27mm; MPN (none) -> SN74ABT534ADWR; now not fitted; now left out of the parts list
- U225, U227: footprint sun3_60:ALS273 -> Package_SO:SOIC-20W_7.5x12.8mm_P1.27mm; MPN (none) -> SN74ALS273DWR; now not fitted; now left out of the parts list
- U226: footprint sun3_60:ALS373 -> Package_SO:SOIC-20W_7.5x12.8mm_P1.27mm; MPN (none) -> SN74ALS373ADWR; now not fitted; now left out of the parts list
Connections:
- net A0: now also IC1.48 (I/O_27), IC3.14 (I/O_6)
- net A1: now also IC1.47 (I/O_26), IC3.13 (I/O_5)
- net A13: now also U1.19 (A1), U2.19 (A1), U3.19 (A1), U4.19 (A1), U6.19 (A1); no longer U1.20 (A0), U2.20 (A0), U3.20 (A0), U4.20 (A0), U6.20 (A0)
- net A14: now also U1.20 (A0), U2.20 (A0), U3.20 (A0), U4.20 (A0), U6.20 (A0); no longer U1.19 (A1), U2.19 (A1), U3.19 (A1), U4.19 (A1), U6.19 (A1)
- net A17: now also U8.3 (A8); no longer U8.14 (A6)
- net A18: now also U7.15 (A5), U8.2 (A9); no longer U7.13 (A7), U8.13 (A7)
- net A19: now also U7.16 (A4), U8.1 (A11); no longer U7.3 (A8), U8.3 (A8)
- net A2: now also IC3.10 (I/O_4)
- net A20: now also U7.12 (A12), U8.6 (A18); no longer U7.2 (A9), U8.2 (A9)
- net A21: now also U7.11 (A14), U8.7 (A15); no longer U7.31 (A10), U8.31 (A10)
- net A22: now also U7.13 (A7), U8.4 (A13); no longer U7.1 (A11), U8.1 (A11)
- net A23: now also U7.10 (A16), U8.9 (A17); no longer U7.12 (A12), U8.12 (A12)
- net A24: now also U7.31 (A10), U8.31 (A10); no longer U7.4 (A13), U8.4 (A13)
- net A25: now also U7.9 (A17), U8.10 (A16); no longer U7.11 (A14), U8.11 (A14)
- net A26: now also U7.3 (A8), U8.14 (A6); no longer U7.7 (A15), U8.7 (A15)
- net A27: now also U7.4 (A13), U8.13 (A7); no longer U7.10 (A16), U8.10 (A16)
- net A28: now also U10.14, IC1.90 (INPUT/GCLK2); no longer U10.5
- net A29: now also IC1.89 (INPUT/GCLR)
- net A3: now also IC3.9 (I/O_3)
- net A30: now also U10.11, IC1.88 (INPUT/OE1); no longer U10.2
- net A31: now also IC1.87 (INPUT/GCLK1)
- net A4: now also IC3.8 (I/O_2)
- net ACCESS: now also U3.22 (I/O1), IC1.64 (I/O_36), IC2.29 (I/O_14); no longer U3.23 (I/O2)
- net BERR.P-: now also IC1.80 (I/O_45), IC3.47 (I/O_26)
- net BERR.T-: now also IC3.17 (I/O_8)
- net BERR.V-: now also IC1.81 (I/O_46), IC3.46 (I/O_25)
- net BERRCLK: now also IC3.90 (INPUT/GCLK2)
- net C.S3-: now also IC1.44 (I/O_23)
- net C.S5-: now also IC1.42 (I/O/PD2)
- net C.S7X-: now also IC1.36 (I/O_20)
- net CX0: now also U8.17 (A3), IC3.76 (I/O_43); no longer U8.20 (A0)
- net CX1: now also U8.18 (A2), IC3.79 (I/O_44); no longer U8.19 (A1)
- net CX2: now also U8.19 (A1), IC3.80 (I/O_45); no longer U8.18 (A2)
- net CX3: now also IC3.81 (I/O_46)
- net CX4: now also U7.2 (A9), U8.15 (A5), IC3.84 (I/O_48); no longer U7.16 (A4), U8.16 (A4)
- net CX5: now also U7.1 (A11), U8.16 (A4), IC3.83 (I/O_47); no longer U7.15 (A5), U8.15 (A5)
- net D24: now also U212.9 (A7), IC3.33 (I/O_18); no longer U212.2 (A0)
- net D25: now also U212.8 (A6), IC3.32 (I/O_17); no longer U212.3 (A1)
- net D26: now also U212.7 (A5), IC3.31 (I/O_16); no longer U212.4 (A2)
- net D27: now also U212.6 (A4), IC3.30 (I/O_15); no longer U212.5 (A3)
- net D28: now also U212.5 (A3), IC3.29 (I/O_14); no longer U212.6 (A4)
- net D29: now also U212.4 (A2), IC3.21 (I/O_11); no longer U212.7 (A5)
- net D30: now also U212.3 (A1), IC3.23 (I/O_12); no longer U212.8 (A6)
- net D31: now also U212.2 (A0), IC3.25 (I/O_13); no longer U212.9 (A7)
- net DIAG-: now also IC3.37 (I/O_21)
- net DISACC-: now also IC1.45 (I/O_24)
- net DSACK0-: now also IC1.21 (I/O_11)
- net EN.BOOT-: now also IC1.6 (I/O_1), IC3.20 (I/O_10)
- net EN.CTL-: now also IC1.83 (I/O_47), IC1.9 (I/O_3), IC3.45 (I/O_24)
- net EN.DEV-: now also IC1.23 (I/O_12), IC1.25 (I/O_13)
- net EN.FPP: now also IC3.92 (I/O_49)
- net EN.PMAP0-: now also IC1.60 (I/O_33), IC2.32 (I/O_17)
- net EN.PMAP2-: now also IC1.58 (I/O_32), IC2.33 (I/O_18)
- net EN.PMAP3-: now also IC1.57 (I/O_31), IC2.35 (I/O_19)
- net EN.SMAP-: now also IC1.63 (I/O_35), IC2.30 (I/O_15)
- net EN.SMAP1-: now also IC1.61 (I/O_34), IC2.31 (I/O_16); no longer U11.5
- net EN.VIDEO: now also IC3.93 (I/O_50)
- net ENABLE_S3E: now also IC1.100 (I/O_56), IC3.87 (INPUT/GCLK1), S1.C
- net ENABLE_S3E_V: now also S2.C
- net FC2: now also IC1.14 (I/O_6)
- net GND: now also U10.2, U10.5, U11.13, U11.14, U11.5, U11.6, C10.2, C11.2, C12.2, C13.2, C14.2, C15.2, C16.2, C17.2, C18.2, C19.2, C20.2, C21.2, C22.2, C23.2, C24.2, C25.2, C26.2, C27.2, C28.2, C29.2, C6.2, C7.2, C8.2, C9.2, IC1.11 (GND_1), IC1.26 (GND_2), IC1.38 (GND_3), IC1.43 (GND_4), IC1.59 (GND_5), IC1.74 (GND_6), IC1.86 (GND_7), IC1.95 (GND_8), IC2.11 (GND_1), IC2.26 (GND_2), IC2.38 (GND_3), IC2.43 (GND_4), IC2.59 (GND_5), IC2.74 (GND_6), IC2.86 (GND_7), IC2.95 (GND_8), IC3.11 (GND_1), IC3.26 (GND_2), IC3.38 (GND_3), IC3.43 (GND_4), IC3.59 (GND_5), IC3.74 (GND_6), IC3.86 (GND_7), IC3.95 (GND_8), R54.2, R55.2, R56.2, R57.2, R58.2, R59.2, R60.2, R61.2, X1.2, X100.2, X101.2, X102.2, X103.2, X104.2, X105.2, X106.2, X107.2, X108.2, X109.2, X3.2, X4.2, X49.2, X91.2, X92.2, X93.2, X94.2, X95.2, X96.2, X97.2, X98.2, X99.2; no longer U10.11, U10.14
- net INIT-: now also IC3.16 (I/O_7)
- net LED0: no longer U228.2 (K)
- net LED1: no longer U228.4
- net LED2: no longer U228.6 (K)
- net LED3: no longer U228.8 (K)
- net LED4: no longer U229.2 (K)
- net LED5: no longer U229.4
- net LED6: no longer U229.6 (K)
- net LED7: no longer U229.8 (K)
- net MMU.S: now also IC1.65 (I/O_37), IC2.17 (I/O_8)
- net MMU.V: now also IC1.71 (I/O_41), IC2.20 (I/O_10)
- net MMU.W: now also IC1.75 (I/O_42), IC2.19 (I/O_9)
- net MMU.X: now also IC2.93 (I/O_50)
- net MMU0: now also U212.11 (B7), IC2.6 (I/O_1), IC3.63 (I/O_35); no longer U212.18 (B0)
- net MMU1: now also U212.12 (B6), IC2.8 (I/O_2), IC3.61 (I/O_34); no longer U212.17 (B1)
- net MMU2: now also U212.13 (B5), IC2.9 (I/O_3), IC3.60 (I/O_33); no longer U212.16 (B2)
- net MMU3: now also U212.14 (B4), IC2.10 (I/O_4), IC3.58 (I/O_32); no longer U212.15 (B3)
- net MMU4: now also U212.15 (B3), IC2.12 (I/O/PD1), IC3.57 (I/O_31); no longer U212.14 (B4)
- net MMU5: now also U212.16 (B2), IC2.13 (I/O_5), IC3.56 (I/O_30); no longer U212.13 (B5)
- net MMU6: now also U212.17 (B1), IC2.14 (I/O_6), IC3.54 (I/O_29); no longer U212.12 (B6)
- net MMU7: now also U212.18 (B0), IC2.16 (I/O_7), IC3.52 (I/O_28); no longer U212.11 (B7)
- net MODIFY: now also IC1.67 (I/O_38), IC2.25 (I/O_13)
- net PA13: now also IC2.92 (I/O_49)
- net PA14: now also IC2.85 (I/O/GCLK3)
- net PA15: now also IC2.84 (I/O_48)
- net PA16: now also IC2.83 (I/O_47)
- net PA17: now also IC2.81 (I/O_46)
- net PA18: now also IC2.80 (I/O_45)
- net PA19: now also IC2.79 (I/O_44)
- net PA20: now also IC2.76 (I/O_43)
- net PA21: now also IC2.48 (I/O_27)
- net PA22: now also IC2.47 (I/O_26)
- net PA23: now also IC2.46 (I/O_25)
- net PA24: now also IC2.45 (I/O_24)
- net PA25: now also IC2.44 (I/O_23)
- net PA26: now also IC2.41 (I/0)
- net PA27: now also IC2.40 (I/O_22)
- net PA28: now also IC2.37 (I/O_21)
- net RD.BERR-: now also IC1.79 (I/O_44), IC3.48 (I/O_27)
- net RD.CX-: now also IC1.85 (I/O/GCLK3), IC3.40 (I/O_22)
- net RD.ID-: now also IC1.8 (I/O_2), IC3.19 (I/O_9)
- net RD.SYSEN-: now also IC1.94 (I/O_51), IC3.35 (I/O_19)
- net READ-: now also IC2.36 (I/O_20), IC3.75 (I/O_42)
- net S3E_A28: now also U10.12, U7.7 (A15), U8.11 (A14); no longer U10.7, U7.9 (A17), U8.9 (A17)
- net S3E_A30: now also U10.9, U8.12 (A12); no longer U10.4, U8.6 (A18)
- net S3E_CX3: now also U8.20 (A0); no longer U8.17 (A3)
- net S3E_EN.SMAP1-: no longer U11.7
- net S3E_WR.CX-: no longer U11.12
- net SA17: now also U8.21 (I/O0), IC2.71 (I/O_41); no longer U7.21 (I/O0)
- net SA18: now also U8.22 (I/O1), IC2.69 (I/O_40); no longer U7.22 (I/O1)
- net SA19: now also U8.23 (I/O2), IC2.68 (I/O_39); no longer U7.23 (I/O2)
- net SA20: now also U8.25 (I/O3), IC2.67 (I/O_38); no longer U7.25 (I/O3)
- net SA21: now also IC2.56 (I/O_30)
- net SA22: now also IC2.57 (I/O_31)
- net SA23: now also U7.29 (I/O7), IC2.75 (I/O_42); no longer U7.28 (I/O6)
- net SA24: now also U7.28 (I/O6), IC2.58 (I/O_32); no longer U7.29 (I/O7)
- net SA25: now also U8.26 (I/O4), IC2.65 (I/O_37), R55.1; no longer U8.21 (I/O0)
- net SA26: now also U1.11 (A14), U2.11 (A14), U3.11 (A14), U4.11 (A14), U6.11 (A14), U8.27 (I/O5), IC2.64 (I/O_36), R56.1; no longer U1.4 (A13), U2.4 (A13), U3.4 (A13), U4.4 (A13), U6.4 (A13), U8.22 (I/O1)
- net SA27: now also U1.4 (A13), U2.4 (A13), U3.4 (A13), U4.4 (A13), U6.4 (A13), U7.25 (I/O3), IC2.54 (I/O_29), R57.1; no longer U1.11 (A14), U2.11 (A14), U3.11 (A14), U4.11 (A14), U6.11 (A14), U8.23 (I/O2)
- net SA28: now also U7.22 (I/O1), IC2.60 (I/O_33), R58.1; no longer U8.25 (I/O3)
- net SA29: now also U8.28 (I/O6), IC2.63 (I/O_35), R59.1; no longer U8.26 (I/O4)
- net SA30: now also U7.21 (I/O0), IC2.61 (I/O_34), R60.1; no longer U8.27 (I/O5)
- net SA31: now also U7.23 (I/O2), IC2.52 (I/O_28), R61.1; no longer U8.28 (I/O6)
- net TYPE0: now also U3.21 (I/O0), IC1.69 (I/O_40), IC2.21 (I/O_11); no longer U3.22 (I/O1)
- net TYPE1: now also U3.23 (I/O2), IC1.68 (I/O_39), IC2.23 (I/O_12); no longer U3.21 (I/O0)
- net VCC: now also C10.1, C11.1, C12.1, C13.1, C14.1, C15.1, C16.1, C17.1, C18.1, C19.1, C20.1, C21.1, C22.1, C23.1, C24.1, C25.1, C26.1, C27.1, C28.1, C29.1, C6.1, C7.1, C8.1, C9.1, IC1.18 (VCCIO_2), IC1.3 (VCCIO_1), IC1.34 (VCCIO_3), IC1.39 (VCCINT_1), IC1.51 (VCCIO_4), IC1.66 (VCCIO_5), IC1.82 (VCCIO_6), IC1.91 (VCCINT_2), IC2.18 (VCCIO_2), IC2.3 (VCCIO_1), IC2.34 (VCCIO_3), IC2.39 (VCCINT_1), IC2.51 (VCCIO_4), IC2.66 (VCCIO_5), IC2.82 (VCCIO_6), IC2.91 (VCCINT_2), IC3.18 (VCCIO_2), IC3.3 (VCCIO_1), IC3.34 (VCCIO_3), IC3.39 (VCCINT_1), IC3.51 (VCCIO_4), IC3.66 (VCCIO_5), IC3.82 (VCCIO_6), IC3.91 (VCCINT_2), X1.1, X100.1, X101.1, X102.1, X103.1, X104.1, X105.1, X106.1, X107.1, X108.1, X109.1, X3.1, X4.1, X49.1, X91.1, X92.1, X93.1, X94.1, X95.1, X96.1, X97.1, X98.1, X99.1; no longer U11.13, U11.6, U228.1 (A), U228.3 (A), U228.5, U228.7, U229.1 (A), U229.3 (A), U229.5, U229.7
- net WDOG-: now also IC3.68 (I/O_39)
- net WE.PMAP0-: now also IC1.96 (I/O_52), IC1.97 (I/O_53)
- net WE.PMAP2-: now also IC1.54 (I/O_29)
- net WE.PMAP3-: now also IC1.56 (I/O_30)
- net WE.SMAP-: now also IC1.98 (I/O_54)
- net WE.SMAP1-: now also IC1.99 (I/O_55)
- net WE.STAT-: now also IC1.76 (I/O_43)
- net WR.CX-: now also IC1.84 (I/O_48), IC3.44 (I/O_23); no longer U11.14
- net WR.DIAG-: now also IC1.16 (I/O_7)
- net WR.SYSEN-: now also IC1.93 (I/O_50), IC3.36 (I/O_20)
- net WRITE-: now also IC1.46 (I/O_25)
- net at R4.2: now also S2.1
- net at R5.2: now also S2.2
- net SAunused: now reaches U5.18 (B0)
- net SAunused: now also R54.1
- net at R2.2: now also S1.2
- net at R1.2: now also S1.1
- new net AS: IC1.40 (I/O_22)
- new net DIS.RAS-: IC1.41 (I/0)
- new net EN.UART-: IC1.20 (I/O_10)
- new net FC0: IC1.10 (I/O_4)
- new net FC1: IC1.13 (I/O_5)
- new net JTAG_TCK1: IC1.62 (I/O/TCK)
- new net JTAG_TCK2: IC2.62 (I/O/TCK)
- new net JTAG_TCK3: IC3.62 (I/O/TCK)
- new net JTAG_TDI1: IC1.4 (I/O/TDI)
- new net JTAG_TDI2: IC2.4 (I/O/TDI)
- new net JTAG_TDI3: IC3.4 (I/O/TDI)
- new net JTAG_TDO1: IC1.73 (I/O/TDO)
- new net JTAG_TDO2: IC2.73 (I/O/TDO)
- new net JTAG_TDO3: IC3.73 (I/O/TDO)
- new net JTAG_TMS1: IC1.15 (I/O/TMS)
- new net JTAG_TMS2: IC2.15 (I/O/TMS)
- new net JTAG_TMS3: IC3.15 (I/O/TMS)
- new net OE.BOOT-: IC1.33 (I/O_18)
- new net R.ACK-: IC1.52 (I/O_28)
- no-connect marks 16 -> 71
Other:
- note added: "CPLD MAPBUF"
- note added: "CPLD MMU"
- note added: "CPLD SYSREG"
- note added: "READ- == R/W- after one inverter, can we drop it ?"
- note added: "WRITE- == R/W- after two inverters, can we drop it ? (also, WRITE- == !READ- after one inverter and READ- == !R/W- after one iverter)"

Commit message: update
Connections:
- net WDOG-: now also IC3.12 (I/O/PD1); no longer IC3.68 (I/O_39)
Changed lines of the file:
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@@
 	)
 	(hierarchical_label "BERR.P-"
-		(shape input)
+		(shape output)
 		(at 124.46 172.72 0)
 		(effects
@@
 	)
 	(hierarchical_label "BERR.V-"
-		(shape input)
+		(shape output)
 		(at 124.46 154.94 0)
 		(effects
@@
 	(hierarchical_label "WDOG-"
 		(shape input)
-		(at -138.43 302.26 0)
-		(effects
-			(font
-				(size 1.27 1.27)
-			)
-			(justify left)
-		)
-	)
+		(at -214.63 312.42 180)
+		(effects
+			(font
+				(size 1.27 1.27)
+			)
+			(justify right)
+		)
+	)
