File: schematics/kicad/sun3_60_scsi2_parity.kicad_sch (KiCad schematic)
At the start: 10 parts, among them U710 AS286, U711 AS286, U712 AS286, U713 AS286, U714 PAL16L8, U715 PAL20R4, U720 ALS374, U721 ALS374, U722 ALS374, U723 ALS374

Commit message: draft, ugly and WiP
Parts:
- added C45, C46, C47, C48, C49, C50, C51, C52, X27, X28, X29, X30, X38, X5, X6, X7, X8: 100nF 0402, Capacitor_SMD:C_0402_1005Metric, symbol Device:C
- added IC6: ATF1504AS-10AU100, sun3_60:QFP50P1600X1600X120-100N, symbol ATF1504AS-10AU100:ATF1504AS-10AU100
- U710, U711, U712, U713: value AS286 -> ACT11286; footprint Package_DIP:DIP-14_W7.62mm -> Package_SO:SOIC-14_3.9x8.7mm_P1.27mm; symbol custom:74AS286 -> custom:74ACT11286; MPN (none) -> 74ACT11286D
- U714, U715: now not fitted; now left out of the parts list
- U720, U721, U722, U723: footprint sun3_60:ALS373 -> Package_SO:SOIC-20W_7.5x12.8mm_P1.27mm; MPN (none) -> SN74ALS374ADWR
Connections:
- net A0: now also IC6.46 (I/O_25)
- net A1: now also IC6.47 (I/O_26)
- net A2: now also IC6.48 (I/O_27)
- net CAS-: now also IC6.32 (I/O_17)
- net CLK: now also IC6.87 (INPUT/GCLK1)
- net D0: now also U710.1 (P2); no longer U710.8 (P1)
- net D1: now also U710.2 (P1); no longer U710.9 (P2)
- net D10: now also U711.14 (P3); no longer U711.10 (P3)
- net D11: now also U711.13 (P4); no longer U711.11 (P4)
- net D13: now also U711.10 (P6); no longer U711.13 (P6)
- net D14: now also U711.9 (P7); no longer U711.1 (P7)
- net D15: now also U711.8 (P8); no longer U711.2 (P8)
- net D16: now also U712.1 (P2); no longer U712.8 (P1)
- net D17: now also U712.2 (P1); no longer U712.9 (P2)
- net D18: now also U712.14 (P3); no longer U712.10 (P3)
- net D19: now also U712.13 (P4); no longer U712.11 (P4)
- net D2: now also U710.14 (P3); no longer U710.10 (P3)
- net D21: now also U712.10 (P6); no longer U712.13 (P6)
- net D22: now also U712.9 (P7); no longer U712.1 (P7)
- net D23: now also U712.8 (P8); no longer U712.2 (P8)
- net D24: now also U713.1 (P2); no longer U713.8 (P1)
- net D25: now also U713.2 (P1); no longer U713.9 (P2)
- net D26: now also U713.14 (P3); no longer U713.10 (P3)
- net D27: now also U713.13 (P4); no longer U713.11 (P4)
- net D29: now also U713.10 (P6); no longer U713.13 (P6)
- net D3: now also U710.13 (P4); no longer U710.11 (P4)
- net D30: now also U713.9 (P7); no longer U713.1 (P7)
- net D31: now also U713.8 (P8); no longer U713.2 (P8)
- net D5: now also U710.10 (P6); no longer U710.13 (P6)
- net D6: now also U710.9 (P7); no longer U710.1 (P7)
- net D7: now also U710.8 (P8); no longer U710.2 (P8)
- net D8: now also U711.1 (P2); no longer U711.8 (P1)
- net D9: now also U711.2 (P1); no longer U711.9 (P2)
- net EN.DEV-: now also IC6.30 (I/O_15)
- net GND: now also U710.4 (GND), U711.4 (GND), U712.4 (GND), U713.4 (GND), C45.2, C46.2, C47.2, C48.2, C49.2, C50.2, C51.2, C52.2, IC6.11 (GND_1), IC6.26 (GND_2), IC6.38 (GND_3), IC6.43 (GND_4), IC6.59 (GND_5), IC6.74 (GND_6), IC6.86 (GND_7), IC6.95 (GND_8), X27.2, X28.2, X29.2, X30.2, X38.2, X5.2, X6.2, X7.2, X8.2; no longer U710.7 (GND), U711.7 (GND), U712.7 (GND), U713.7 (GND)
- net INIT-: now also IC6.76 (I/O_43)
- net IO.D0: now also IC6.84 (I/O_48)
- net IO.D1: now also IC6.83 (I/O_47)
- net IO.D2: now also IC6.81 (I/O_46)
- net IO.D3: now also IC6.80 (I/O_45)
- net IO.D4: now also IC6.93 (I/O_50)
- net IO.D5: now also IC6.94 (I/O_51)
- net IO.D6: now also IC6.96 (I/O_52)
- net IO.D7: now also IC6.92 (I/O_49)
- net P0: now also U713.3 (P_I/O); no longer U713.6 (P_I/O)
- net P1: now also U712.3 (P_I/O); no longer U712.6 (P_I/O)
- net P2: now also U711.3 (P_I/O); no longer U711.6 (P_I/O)
- net P3: now also U710.3 (P_I/O); no longer U710.6 (P_I/O)
- net PAR.CHK-: now also IC6.25 (I/O_13)
- net PAR.IRQ-: now also IC6.21 (I/O_11)
- net PAR.SAMPLE: now also IC6.79 (I/O_44)
- net PAR.TEST-: now also U710.7 (P9), IC6.23 (I/O_12); no longer U710.4 (P9), U711.4 (P9), U712.4 (P9), U713.4 (P9)
- net PAR0-: now also IC6.52 (I/O_28)
- net PAR1-: now also IC6.54 (I/O_29)
- net PAR2-: now also IC6.56 (I/O_30)
- net PAR3-: now also IC6.57 (I/O_31)
- net RD.PAR0-: now also IC6.35 (I/O_19)
- net RD.PAR4-: now also IC6.100 (I/O_56)
- net RD.PAR5-: now also IC6.99 (I/O_55)
- net RD.PAR6-: now also IC6.98 (I/O_54)
- net RD.PAR7-: now also IC6.97 (I/O_53)
- net R/W-: now also IC6.17 (I/O_8)
- net VCC: now also U710.11 (VCC), U711.11 (VCC), U712.11 (VCC), U713.11 (VCC), C45.1, C46.1, C47.1, C48.1, C49.1, C50.1, C51.1, C52.1, IC6.18 (VCCIO_2), IC6.3 (VCCIO_1), IC6.34 (VCCIO_3), IC6.39 (VCCINT_1), IC6.51 (VCCIO_4), IC6.66 (VCCIO_5), IC6.82 (VCCIO_6), IC6.91 (VCCINT_2), X27.1, X28.1, X29.1, X30.1, X38.1, X5.1, X6.1, X7.1, X8.1; no longer U710.14 (VCC), U711.14 (VCC), U712.14 (VCC), U713.14 (VCC)
- net WR.PAR0-: now also IC6.42 (I/O/PD2)
- net WR.PAR4-: now also IC6.44 (I/O_23)
- net WRITE-: now also U710.6 (XMIT-), U711.6 (XMIT-), U711.7 (P9), U712.6 (XMIT-), U712.7 (P9), U713.6 (XMIT-), U713.7 (P9); no longer U710.3 (XMIT-), U711.3 (XMIT-), U712.3 (XMIT-), U713.3 (XMIT-)
- net XACK-: now also IC6.33 (I/O_18)
- new net CLK-: IC6.90 (INPUT/GCLK2)
- new net JTAG_TCK6: IC6.62 (I/O/TCK)
- new net JTAG_TDI6: IC6.4 (I/O/TDI)
- new net JTAG_TDO6: IC6.73 (I/O/TDO)
- new net JTAG_TMS6: IC6.15 (I/O/TMS)
- new net RD_PARX-: IC6.75 (I/O_42)
- new net WR_PARX-: IC6.71 (I/O_41)
- no-connect marks 3 -> 19
Other:
- note added: "Memory Address Register (long @ 0x00080004)"
- note added: "Memory Control Register (byte @ 0x00080000"
- note added: "PARITY+DVMA"

Commit message: update
Connections:
- net CAS-: now also IC6.20 (I/O_10); no longer IC6.32 (I/O_17)
Changed lines of the file:
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@@
 	(hierarchical_label "CAS-"
 		(shape input)
-		(at -107.95 220.98 270)
+		(at -130.81 187.96 180)
 		(effects
 			(font

Commit message: ongoing ethernet pld
Other:
- note added: "CPLD PARITY"
- note removed: "PARITY+DVMA"
Changed lines of the file:
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@@
 		)
 	)
-	(text "PARITY+DVMA"
+	(text "CPLD PARITY"
 		(exclude_from_sim no)
 		(at -134.874 113.03 0)
