File: schematics/kicad/sun3_60_eeprom.kicad_sch (KiCad schematic)
At the start: 19 parts, among them U2001 PAL16L8, U300 27512, U301 28C16, U302 7170, U303 32768Hz, U304 ALS273, U305 ALS373, U307 PAL20L8, U309 3-VOLT, U310 PAL20L8, U311 PAL20L8, U312 PAL8L14, U313 PAL16R4, U314 Z8068, X301 470UF

Commit message: First draft for an expanded MMU
This version uses vintage parts except for the SRAM, which are IS61C5128AS-25HLI (they could be QLI instead)
Unfortunately, this requires:
* 2 more 74ALS245 to buffer the second byte of PMAP indices in the SMAP
* one more LS2518 (!) to extend the context register
* a couple of 74CBTLV3257 to be able to stay in "normal" Sun3 mode with minimal delays on the signals
* a couple of switches to enabled/disable the new features
* some extra passives
* U231, a PAL16L8, needs another input and another two outputs, or can be split in two PALs (or GAL, CPLDs, ...)

Also this does not include tne necessary decoupling on the new components
Changed lines of the file:
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@@
 (kicad_sch
-	(version 20231120)
+	(version 20250114)
 	(generator "eeschema")
-	(generator_version "8.0")
+	(generator_version "9.0")
 	(paper "USLegal")
 	(title_block
@@
 		(rev "1")
 	)
+	(text "DECODE2"
+		(exclude_from_sim no)
+		(at 86.36 140.97 0)
+		(effects
+			(font
+				(size 1.27 1.27)
+			)
+			(justify left bottom)
+		)
+	)
+	(text "VIDEO"
+		(exclude_from_sim no)
+		(at 162.052 167.64 0)
+		(effects
+			(font
+				(size 1.27 1.27)
+			)
+		)
+	)
+	(text "INTERRUPT"
+		(exclude_from_sim no)
+		(at 261.62 120.65 0)
+		(effects
+			(font
+				(size 1.27 1.27)
+			)
+			(justify left bottom)
+		)
+	)
+	(text "TOD-CLOCK"
+		(exclude_from_sim no)
+		(at 170.18 82.55 0)
+		(effects
+			(font
+				(size 1.27 1.27)
+			)
+			(justify left bottom)
+		)
+	)
+	(text "DCP"
+		(exclude_from_sim no)
+		(at 318.77 26.67 0)
+		(effects
+			(font
+				(size 1.27 1.27)
+			)
+			(justify left bottom)
+		)
+	)
+	(text "DECODE1"
+		(exclude_from_sim no)
+		(at 81.28 87.63 0)
+		(effects
+			(font
+				(size 1.27 1.27)
+			)
+			(justify right bottom)
+		)
+	)
+	(text "EPROM"
+		(exclude_from_sim no)
+		(at 101.6 26.67 0)
+		(effects
+			(font
+				(size 1.27 1.27)
+			)
+			(justify left bottom)
+		)
+	)
+	(text "DECODE3"
+		(exclude_from_sim no)
+		(at 33.02 132.08 0)
+		(effects
+			(font
+				(size 1.27 1.27)
+			)
+			(justify left bottom)
+		)
+	)
+	(text "INTERRUPT REGISTER"
+		(exclude_from_sim no)
+		(at 205.74 26.67 0)
+		(effects
+			(font
+				(size 1.27 1.27)
+			)
+			(justify left bottom)
+		)
+	)
+	(text "15-nsec"
+		(exclude_from_sim no)
+		(at 69.85 93.98 0)
+		(effects
+			(font
+				(size 1.27 1.27)
+			)
+			(justify right bottom)
+		)
+	)
+	(text "Optional"
+		(exclude_from_sim no)
+		(at 175.26 148.59 0)
+		(effects
+			(font
+				(size 1.27 1.27)
+			)
+			(justify right bottom)
+		)
+	)
+	(text "Excluded"
+		(exclude_from_sim no)
+		(at 317.5 22.86 0)
+		(effects
+			(font
+				(size 1.27 1.27)
+				(color 255 0 0 1)
+			)
+			(justify left bottom)
+		)
+	)
+	(text "EXCLUDED\nOnly for Video"
+		(exclude_from_sim no)
+		(at 161.798 164.338 0)
+		(effects
+			(font
+				(size 1.27 1.27)
+				(color 255 0 0 1)
+			)
+		)
+	)
+	(text "DCP"
+		(exclude_from_sim no)
+		(at 283.21 76.2 0)
+		(effects
+			(font
+				(size 1.27 1.27)
+			)
+			(justify right bottom)
+		)
+	)
+	(text "EEPROM"
+		(exclude_from_sim no)
+		(at 156.21 26.67 0)
+		(effects
+			(font
+				(size 1.27 1.27)
+			)
+			(justify left bottom)
+		)
+	)
 	(junction
 		(at 335.28 63.5)
@@
 		)
 	)
-	(text "DECODE2"
-		(exclude_from_sim no)
-		(at 86.36 140.97 0)
-		(effects
-			(font
-				(size 1.27 1.27)
-			)
-			(justify left bottom)
-		)
-	)
-	(text "VIDEO"
-		(exclude_from_sim no)
-		(at 162.052 167.64 0)
-		(effects
-			(font
-				(size 1.27 1.27)
-			)
-		)
-	)
-	(text "INTERRUPT"
-		(exclude_from_sim no)
-		(at 261.62 120.65 0)
-		(effects
-			(font
-				(size 1.27 1.27)
-			)
-			(justify left bottom)
-		)
-	)
-	(text "TOD-CLOCK"
-		(exclude_from_sim no)
-		(at 170.18 82.55 0)
-		(effects
-			(font
-				(size 1.27 1.27)
-			)
-			(justify left bottom)
-		)
-	)
-	(text "DCP"
-		(exclude_from_sim no)
-		(at 318.77 26.67 0)
-		(effects
-			(font
-				(size 1.27 1.27)
-			)
-			(justify left bottom)
-		)
-	)
-	(text "DECODE1"
-		(exclude_from_sim no)
-		(at 81.28 87.63 0)
-		(effects
-			(font
-				(size 1.27 1.27)
-			)
-			(justify right bottom)
-		)
-	)
-	(text "EPROM"
-		(exclude_from_sim no)
-		(at 101.6 26.67 0)
-		(effects
-			(font
-				(size 1.27 1.27)
-			)
-			(justify left bottom)
-		)
-	)
-	(text "DECODE3"
-		(exclude_from_sim no)
-		(at 33.02 132.08 0)
-		(effects
-			(font
-				(size 1.27 1.27)
-			)
-			(justify left bottom)
-		)
-	)
-	(text "INTERRUPT REGISTER"
-		(exclude_from_sim no)
-		(at 205.74 26.67 0)
-		(effects
-			(font
-				(size 1.27 1.27)
-			)
-			(justify left bottom)
-		)
-	)
-	(text "15-nsec"
-		(exclude_from_sim no)
-		(at 69.85 93.98 0)
-		(effects
-			(font
-				(size 1.27 1.27)
-			)
-			(justify right bottom)
-		)
-	)
-	(text "Optional"
-		(exclude_from_sim no)
-		(at 175.26 148.59 0)
-		(effects
-			(font
-				(size 1.27 1.27)
-			)
-			(justify right bottom)
-		)
-	)
-	(text "Excluded"
-		(exclude_from_sim no)
-		(at 317.5 22.86 0)
-		(effects
-			(font
-				(size 1.27 1.27)
-				(color 255 0 0 1)
-			)
-			(justify left bottom)
-		)
-	)
-	(text "EXCLUDED\nOnly for Video"
-		(exclude_from_sim no)
-		(at 161.798 164.338 0)
-		(effects
-			(font
-				(size 1.27 1.27)
-				(color 255 0 0 1)
-			)
-		)
-	)
-	(text "DCP"
-		(exclude_from_sim no)
-		(at 283.21 76.2 0)
-		(effects
-			(font
-				(size 1.27 1.27)
-			)
-			(justify right bottom)
-		)
-	)
-	(text "EEPROM"
-		(exclude_from_sim no)
-		(at 156.21 26.67 0)
-		(effects
-			(font
-				(size 1.27 1.27)
-			)
-			(justify left bottom)
-		)
-	)

Commit message: draft, ugly and WiP
Parts:
- removed U301: 28C16, Package_DIP:DIP-24_W15.24mm, symbol custom:28C16
- added C30, C31, C32, C33, C34, C35, C36, C37, C38, C39, C40, C41, C42, C43, C44, C5, X20, X23, X31, X32, X35, X36: 100nF 0402, Capacitor_SMD:C_0402_1005Metric, symbol Device:C
- added D1, D2, D3, D4, D5, D6, D7, D8: LED, LED_SMD:LED_0603_1608Metric, symbol Device:LED
- added IC4, IC5: ATF1504AS-10AU100, sun3_60:QFP50P1600X1600X120-100N, symbol ATF1504AS-10AU100:ATF1504AS-10AU100
- added R62, R63, R64, R65, R66, R67, R68, R69: 510, Resistor_SMD:R_0402_1005Metric, symbol Device:R
- added U301: AT28C64B_PLCC, Package_LCC:PLCC-32_THT-Socket, symbol custom:AT28C64B_PLCC
- U2001, U307, U310, U311, U312, U313, U314: now not fitted; now left out of the parts list
- U304: footprint sun3_60:ALS273 -> Package_SO:SOIC-20W_7.5x12.8mm_P1.27mm; MPN (none) -> SN74ALS273DWR; now not fitted; now left out of the parts list
- U305: footprint sun3_60:ALS373 -> Package_SO:SOIC-20W_7.5x12.8mm_P1.27mm; MPN (none) -> SN74ALS373ADWR; MPN-ALT (none) -> DM74ALS373WM; now not fitted; now left out of the parts list
Connections:
- net A0: now also U301.11 (A0)
- net A1: now also U301.10 (A1)
- net A10: now also U301.29 (A8)
- net A2: now also U301.9 (A2)
- net A3: now also U301.8 (A3)
- net A4: now also U301.7 (A4)
- net A5: now also U301.6 (A5)
- net A6: now also U301.5 (A6)
- net A7: now also U301.4 (A7)
- net A8: now also U301.24 (A10)
- net A9: now also U301.28 (A9)
- net C.S21-: now also IC4.23 (I/O_12)
- net C.S3-: now also IC4.79 (I/O_44)
- net C.S5-: now also IC4.80 (I/O_45)
- net C.S9-: now also IC4.48 (I/O_27)
- net CLK-: now also IC4.90 (INPUT/GCLK2)
- net DISACC-: now also IC4.87 (INPUT/GCLK1)
- net DS-: now also IC4.63 (I/O_35)
- net DSACK0-: now also IC4.94 (I/O_51), IC5.6 (I/O_1)
- net E.IRQ-: now also IC5.83 (I/O_47)
- net EN.CAS: now also IC4.60 (I/O_33)
- net EN.DEV-: now also IC4.93 (I/O_50)
- net EN.E-: now also IC4.47 (I/O_26)
- net EN.IO-: now also IC4.30 (I/O_15)
- net EN.S-: now also IC4.57 (I/O_31)
- net EN.UART-: now also IC4.8 (I/O_2)
- net EN.V-: now also IC4.58 (I/O_32)
- net GND: now also C30.2, C31.2, C32.2, C33.2, C34.2, C35.2, C36.2, C37.2, C38.2, C39.2, C40.2, C41.2, C42.2, C43.2, C44.2, C5.2, IC4.11 (GND_1), IC4.26 (GND_2), IC4.38 (GND_3), IC4.43 (GND_4), IC4.59 (GND_5), IC4.74 (GND_6), IC4.86 (GND_7), IC4.95 (GND_8), IC5.11 (GND_1), IC5.26 (GND_2), IC5.38 (GND_3), IC5.43 (GND_4), IC5.59 (GND_5), IC5.74 (GND_6), IC5.86 (GND_7), IC5.95 (GND_8), U301.16 (GND), U301.23 (~{CS}), U301.27 (A11), U301.3 (A12), X20.2, X23.2, X31.2, X32.2, X35.2, X36.2
- net INIT-: now also IC4.25 (I/O_13), IC5.84 (I/O_48)
- net IO.D0: now also IC5.80 (I/O_45), U301.22 (D7)
- net IO.D1: now also IC5.79 (I/O_44), U301.19 (D4)
- net IO.D2: now also IC5.76 (I/O_43), U301.15 (D2)
- net IO.D3: now also IC5.75 (I/O_42), U301.13 (D0)
- net IO.D4: now also IC5.71 (I/O_41), U301.14 (D1)
- net IO.D5: now also IC5.69 (I/O_40), U301.18 (D3)
- net IO.D6: now also IC5.68 (I/O_39), U301.20 (D5)
- net IO.D7: now also IC5.67 (I/O_38), U301.21 (D6)
- net IO2CPU-: now also IC4.92 (I/O_49), IC5.30 (I/O_15)
- net IOLOCK-: now also IC4.46 (I/O_25)
- net IPL0-: now also IC5.100 (I/O_56)
- net IPL1-: now also IC5.99 (I/O_55)
- net IPL2-: now also IC5.98 (I/O_54)
- net OE.BOOT-: now also IC4.83 (I/O_47)
- net OE.EPROM-: now also IC4.44 (I/O_23)
- net PA17: now also IC4.67 (I/O_38)
- net PA18: now also IC4.68 (I/O_39)
- net PA19: now also IC4.69 (I/O_40)
- net PA20: now also IC4.71 (I/O_41)
- net PA28: now also IC4.64 (I/O_36)
- net PAR.IRQ-: now also IC5.93 (I/O_50)
- net RD.EEPROM-: now also IC4.97 (I/O_53), U301.25 (~{OE})
- net RD.INT-: now also IC4.16 (I/O_7), IC5.20 (I/O_10)
- net RD.RTC-: now also IC4.19 (I/O_9)
- net RD.SCC0-: now also IC4.13 (I/O_5)
- net RD.SCC1-: now also IC4.10 (I/O_4)
- net RERUN-: now also IC4.21 (I/O_11)
- net RESET-: now also IC5.96 (I/O_52)
- net RTC-: now also IC5.81 (I/O_46)
- net S.IRQ-: now also IC5.94 (I/O_51)
- net SCC.IRQ-: now also IC5.92 (I/O_49)
- net TYPE0: now also IC4.85 (I/O/GCLK3)
- net TYPE1: now also IC4.84 (I/O_48)
- net V.INT-: now also IC5.21 (I/O_11)
- net VCC: now also C300.2, C301.1, C30.1, C31.1, C32.1, C33.1, C34.1, C35.1, C36.1, C37.1, C38.1, C39.1, C40.1, C41.1, C42.1, C43.1, C44.1, C5.1, IC4.18 (VCCIO_2), IC4.3 (VCCIO_1), IC4.34 (VCCIO_3), IC4.39 (VCCINT_1), IC4.51 (VCCIO_4), IC4.66 (VCCIO_5), IC4.82 (VCCIO_6), IC4.91 (VCCINT_2), IC5.18 (VCCIO_2), IC5.3 (VCCIO_1), IC5.34 (VCCIO_3), IC5.39 (VCCINT_1), IC5.51 (VCCIO_4), IC5.66 (VCCIO_5), IC5.82 (VCCIO_6), IC5.91 (VCCINT_2), R62.2, R63.2, R64.2, R65.2, R66.2, R67.2, R68.2, R69.2, U301.32 (VCC), X20.1, X23.1, X31.1, X32.1, X35.1, X36.1
- net WR.EEPROM-: now also IC4.98 (I/O_54), U301.31 (~{WE})
- net WR.INT-: now also IC4.17 (I/O_8), IC5.19 (I/O_9)
- net WR.RTC-: now also IC4.20 (I/O_10)
- net WR.SCC0-: now also IC4.14 (I/O_6)
- net WR.SCC1-: now also IC4.9 (I/O_3)
- net WRITE-: now also IC4.88 (INPUT/OE1), IC5.48 (I/O_27)
- new net: D6.2 (A), R67.1
- new net: D7.2 (A), R68.1
- new net: D5.2 (A), R66.1
- new net: D4.2 (A), R65.1
- new net: D8.2 (A), R69.1
- new net: D1.2 (A), R62.1
- new net: D2.2 (A), R63.1
- new net: D3.2 (A), R64.1
- new net AS: IC4.56 (I/O_30)
- new net C.S3: IC4.54 (I/O_29)
- new net C.S5: IC4.52 (I/O_28)
- new net C.S7: IC4.81 (I/O_46)
- new net D24: IC5.63 (I/O_35)
- new net D25: IC5.61 (I/O_34)
- new net D26: IC5.60 (I/O_33)
- new net D27: IC5.58 (I/O_32)
- new net D28: IC5.57 (I/O_31)
- new net D29: IC5.56 (I/O_30)
- new net D30: IC5.54 (I/O_29)
- new net D31: IC5.52 (I/O_28)
- new net DS: IC5.32 (I/O_17)
- new net JTAG_TCK4: IC4.62 (I/O/TCK)
- new net JTAG_TCK5: IC5.62 (I/O/TCK)
- new net JTAG_TDI4: IC4.4 (I/O/TDI)
- new net JTAG_TDI5: IC5.4 (I/O/TDI)
- new net JTAG_TDO4: IC4.73 (I/O/TDO)
- new net JTAG_TDO5: IC5.73 (I/O/TDO)
- new net JTAG_TMS4: IC4.15 (I/O/TMS)
- new net JTAG_TMS5: IC5.15 (I/O/TMS)
- new net LED0: D1.1 (K), IC5.47 (I/O_26)
- new net LED1: D2.1 (K), IC5.46 (I/O_25)
- new net LED2: D3.1 (K), IC5.45 (I/O_24)
- new net LED3: D4.1 (K), IC5.44 (I/O_23)
- new net LED4: D5.1 (K), IC5.41 (I/0)
- new net LED5: D6.1 (K), IC5.40 (I/O_22)
- new net LED6: D7.1 (K), IC5.37 (I/O_21)
- new net LED7: D8.1 (K), IC5.36 (I/O_20)
- new net RD_PARX-: IC4.99 (I/O_55)
- new net RSVD1: IC5.8 (I/O_2)
- new net RSVD2: IC5.9 (I/O_3)
- new net RSVD3: IC5.10 (I/O_4)
- new net RSVD4: IC5.13 (I/O_5)
- new net RSVD5: IC5.14 (I/O_6)
- new net WR.DIAG-: IC5.31 (I/O_16)
- new net WR_PARX-: IC4.100 (I/O_56)
- no-connect marks 16 -> 48
Other:
- note added: "CPLD DECODE"
- note added: "CPLD IOBUS"
- note added: "EXCLUDED Only for DCP"

Commit message: update
Connections:
- net AS: now also IC4.61 (I/O_34); no longer IC4.56 (I/O_30)
- net C.S3: now also IC4.60 (I/O_33); no longer IC4.54 (I/O_29)
- net C.S5: now also IC4.48 (I/O_27); no longer IC4.52 (I/O_28)
- net C.S9-: now also IC4.54 (I/O_29); no longer IC4.48 (I/O_27)
- net EN.CAS: now also IC4.47 (I/O_26); no longer IC4.60 (I/O_33)
- net EN.E-: now also IC4.45 (I/O_24); no longer IC4.47 (I/O_26)
- net EN.IO-: no longer IC4.30 (I/O_15)
- net EN.S-: now also IC4.29 (I/O_14); no longer IC4.57 (I/O_31)
- net EN.V-: now also IC4.30 (I/O_15); no longer IC4.58 (I/O_32)
- net IOLOCK-: now also IC4.52 (I/O_28); no longer IC4.46 (I/O_25)
- net RD.SCC0-: now also IC4.12 (I/O/PD1); no longer IC4.13 (I/O_5)
- net WR.SCC0-: now also IC4.13 (I/O_5); no longer IC4.14 (I/O_6)
- net BERR.T-: now reaches IC4.6 (I/O_1)
- net WDOG-: now reaches IC4.76 (I/O_43)
- new net HALT-: IC4.14 (I/O_6)
- new net POR-: IC4.58 (I/O_32)
- no-connect marks 48 -> 56
Changed lines of the file:
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@@
 	)
 	(no_connect
+		(at -77.47 191.77)
+	)
+	(no_connect
 		(at -41.91 191.77)
 	)
@@
 	)
 	(no_connect
+		(at -74.93 191.77)
+	)
+	(no_connect
 		(at 101.6 156.21)
 	)
@@
 	)
 	(no_connect
+		(at -64.77 191.77)
+	)
+	(no_connect
 		(at 279.4 147.32)
 	)
@@
 	)
 	(no_connect
+		(at -62.23 191.77)
+	)
+	(no_connect
 		(at 293.37 97.79)
 	)
@@
 	)
 	(no_connect
+		(at 26.67 115.57)
+	)
+	(no_connect
 		(at 335.28 87.63)
 	)
@@
 	)
 	(no_connect
+		(at -104.14 189.23)
+	)
+	(no_connect
 		(at 279.4 144.78)
 	)
+	(no_connect
+		(at -104.14 201.93)
+	)
+	(no_connect
+		(at -72.39 191.77)
+	)
 	(bus_entry
 		(at -21.59 307.34)
@@
 	(hierarchical_label "EN.CAS"
 		(shape output)
-		(at -31.75 148.59 0)
+		(at -46.99 191.77 270)
 		(effects
 			(font
 				(size 1.27 1.27)
 			)
-			(justify left)
+			(justify right)
 		)
 	)
@@
 	(hierarchical_label "EN.IO-"
 		(shape output)
-		(at -90.17 191.77 270)
+		(at -104.14 201.93 0)
 		(effects
 			(font
 				(size 1.27 1.27)
 			)
-			(justify right)
+			(justify left)
 		)
 	)
@@
 		)
 	)
+	(hierarchical_label "POR-"
+		(shape input)
+		(at -31.75 153.67 0)
+		(effects
+			(font
+				(size 1.27 1.27)
+			)
+			(justify left)
+		)
+	)
 	(hierarchical_label "TEST4-"
 		(shape input)
@@
 	(hierarchical_label "C.S5"
 		(shape input)
-		(at -31.75 168.91 0)
+		(at -44.45 191.77 270)
 		(effects
 			(font
 				(size 1.27 1.27)
 			)
-			(justify left)
+			(justify right)
 		)
 	)
@@
 	(hierarchical_label "C.S3"
 		(shape input)
-		(at -31.75 163.83 0)
+		(at -31.75 148.59 0)
 		(effects
 			(font
@@
 	(hierarchical_label "EN.S-"
 		(shape output)
-		(at -31.75 156.21 0)
+		(at -92.71 191.77 270)
 		(effects
 			(font
 				(size 1.27 1.27)
 			)
-			(justify left)
+			(justify right)
 		)
 	)
 	(hierarchical_label "EN.V-"
 		(shape output)
-		(at -31.75 153.67 0)
+		(at -90.17 191.77 270)
 		(effects
 			(font
 				(size 1.27 1.27)
 			)
-			(justify left)
+			(justify right)
 		)
 	)
 	(hierarchical_label "RD.SCC0-"
 		(shape output)
-		(at -107.95 140.97 180)
+		(at -107.95 138.43 180)
 		(effects
 			(font
@@
 	(hierarchical_label "C.S9-"
 		(shape input)
-		(at -44.45 191.77 270)
+		(at -31.75 163.83 0)
 		(effects
 			(font
 				(size 1.27 1.27)
 			)
-			(justify right)
+			(justify left)
 		)
 	)
@@
 	(hierarchical_label "AS"
 		(shape input)
-		(at -31.75 158.75 0)
+		(at -31.75 146.05 0)
+		(effects
+			(font
+				(size 1.27 1.27)
+			)
+			(justify left)
+		)
+	)
+	(hierarchical_label "WDOG-"
+		(shape output)
+		(at -39.37 85.09 90)
 		(effects
 			(font
@@
 		)
 	)
+	(hierarchical_label "BERR.T-"
+		(shape input)
+		(at -107.95 123.19 180)
+		(effects
+			(font
+				(size 1.27 1.27)
+			)
+			(justify right)
+		)
+	)
 	(hierarchical_label "WRITE-"
 		(shape input)
@@
 	(hierarchical_label "EN.E-"
 		(shape output)
-		(at -46.99 191.77 270)
+		(at -52.07 191.77 270)
 		(effects
 			(font
@@
 	(hierarchical_label "IOLOCK-"
 		(shape input)
-		(at -49.53 191.77 270)
+		(at -31.75 168.91 0)
 		(effects
 			(font
 				(size 1.27 1.27)
 			)
-			(justify right)
+			(justify left)
 		)
 	)
@@
 		)
 	)
+	(hierarchical_label "HALT-"
+		(shape input)
+		(at -107.95 143.51 180)
+		(effects
+			(font
+				(size 1.27 1.27)
+			)
+			(justify right)
+		)
+	)
 	(hierarchical_label "WR.SCC0-"
 		(shape output)
-		(at -107.95 143.51 180)
+		(at -107.95 140.97 180)
 		(effects
 			(font

Commit message: ongoing ethernet pld
Connections:
- net E.IRQ-: now also IC5.65 (I/O_37); no longer IC5.83 (I/O_47)
Changed lines of the file:
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@@
 	(hierarchical_label "E.IRQ-"
 		(shape input)
-		(at -58.42 236.22 90)
+		(at -33.02 287.02 0)
 		(effects
 			(font

Commit message: ongoing
Parts:
- added X57: 100nF 0402, Capacitor_SMD:C_0402_1005Metric, symbol Device:C
- added X58: 10nF 0402, Capacitor_SMD:C_0402_1005Metric, symbol Device:C
- added Y1: SiT8008xx-2x-xxS, Crystal:Crystal_SMD_3225-4Pin_3.2x2.5mm, symbol Oscillator:SiT8008xx-2x-xxS
- C300, C301, R300, U303: now not fitted; now left out of the parts list
- R301: footprint Resistor_THT:R_Axial_DIN0207_L6.3mm_D2.5mm_P7.62mm_Horizontal -> Capacitor_SMD:C_0402_1005Metric; MPN (none) -> 0402WGF4700TCE
- U309: footprint Battery:Battery_Panasonic_CR2032-VS1N_Vertical_CircularHoles -> Battery:BatteryHolder_MYOUNG_BS-07-A1BJ001_CR2032; MPN (none) -> BS-07-A1BJ001
- X301: footprint Capacitor_THT:CP_Radial_D10.0mm_P5.00mm -> Capacitor_SMD:CP_Elec_6.3x7.7; MPN (none) -> RVT1A471M0607
Connections:
- net GND: now also X57.2, X58.2, Y1.2 (GND)
- net RESET-: now also IC5.97 (I/O_53); no longer IC5.96 (I/O_52)
- net RSVD1: now also IC5.12 (I/O/PD1); no longer IC5.8 (I/O_2)
- net RSVD2: now also IC5.13 (I/O_5); no longer IC5.9 (I/O_3)
- net RSVD3: now also IC5.14 (I/O_6); no longer IC5.10 (I/O_4)
- net RSVD4: now also IC5.16 (I/O_7); no longer IC5.13 (I/O_5)
- net RSVD5: now also IC5.17 (I/O_8); no longer IC5.14 (I/O_6)
- net V.INT-: now also IC5.96 (I/O_52); no longer IC5.21 (I/O_11)
- net VCC: now also X57.1, X58.1, Y1.4 (Vdd)
- net at C300.1, U303.2: no longer U302.10 (OIN)
- net at U302.9 (OOUT): no longer R300.1
- new net CMCLK_32768_RTC: U302.10 (OIN), Y1.3 (OUT)
- no-connect marks 56 -> 58
