File: schematics/kicad/sun3_60_serial.kicad_sch (KiCad schematic)
At the start: 9 parts, among them J1 KB/Mouse, J2 Serial A/B, U400 Z8530, U401 Z8530, U402 4.9152 Mhz, U404 74ALS04, U408 74ALS04

Commit message: draft, ugly and WiP
Parts:
- added J3: Mini-DIN-8, sun3_60:57492681, symbol Connector:Mini-DIN-8
- added J6, J7: DB25_Socket, sun3_60:D25S33E4PA00LF, symbol Connector:DB25_Socket
- added X52: 100nF 0402, Capacitor_SMD:C_0402_1005Metric, symbol Device:C
- J1, J2, U408: now not fitted; now left out of the parts list
- S400, S401: MPN (none) -> 4608X-102-472LF; now not fitted; now left out of the parts list
- U402: footprint Oscillator:Oscillator_DIP-14 -> sun3_60:CXO_DIP8+14
- U404: footprint Package_DIP:DIP-14_W7.62mm -> Package_SO:SOIC-14_3.9x8.7mm_P1.27mm; MPN (none) -> SN74ALS04BDR
Connections:
- net GND: now also J3.1, J3.2, J6.7, J7.7, X52.2
- net VCC: now also J3.3, J3.8, X52.1
- net at U408.8: no longer U401.13 (RXDA)
- net at U408.1: no longer U401.15 (TXDA)
- net SERIAL_PCLK: now reaches U400.20 (PCLK), U401.20 (PCLK), U402.8 (OUT)
- net at U408.5: no longer U401.25 (TXDB)
- net at U408.4: no longer U401.27 (RXDB)
- net at U408.2: no longer J2.2 (Pin_2)
- net RXDC: now reaches J2.3 (Pin_3), S400.7 (R4.1)
- net RXDC: now also U401.13 (RXDA), J6.3; no longer U408.9
- net at U408.6: no longer J2.4 (Pin_4)
- net RXDD: now reaches J2.5 (Pin_5), S400.3 (R2.1)
- net RXDD: now also U401.27 (RXDB), J7.3; no longer U408.3
- net TxDB: now reaches J1.4 (Pin_4), U404.6
- net TxDB: now also J3.7
- net RxDA: now reaches J1.5 (Pin_5), S401.3 (R2.1), U404.3
- net RxDA: now also J3.6
- net TxDA: now reaches J1.2 (Pin_2), U404.2
- net TxDA: now also J3.5
- net RxDB: now reaches J1.3 (Pin_3), S401.7 (R4.1), U404.9
- net RxDB: now also J3.4
- new net -5V: J6.25 (P25), J7.25 (P25)
- new net CTSC: J6.5
- new net CTSD: J7.5
- new net DAC: J6.24 (P24)
- new net DAD: J7.24 (P24)
- new net DBC: J6.15 (P15)
- new net DBD: J7.15 (P15)
- new net DCDC: J6.8
- new net DCDD: J7.8
- new net DDC: J6.17 (P17)
- new net DDD: J7.17 (P17)
- new net DSRC: J6.6
- new net DSRD: J7.6
- new net DTRC: J6.20 (P20)
- new net DTRD: J7.20 (P20)
- new net RTSC: J6.4
- new net RTSD: J7.4
- new net TXDC: J2.2 (Pin_2), J6.2, U401.15 (TXDA)
- new net TXDD: J2.4 (Pin_4), J7.2, U401.25 (TXDB)
- no-connect marks 39 -> 65
Other:
- note added: "The pinout of the DB15 connector (on the CPU) is: 1 RxD0 (keyboard) 8 GND 2 GND 9 GND 3 TxD0 (keyboard) 10 VCC 4 GND 11 VCC 5 RxD1 (mouse) 12 VCC 6 GND 14 VCC 7 TxD1 (mouse) 15 VCC"
- note added: "The pinout of the DIN-8 connector (female, on the CPU) is: 7 1 GND 5 TxDA (Keyboard) 8 6 2 GND 6 RxDA (Keyboard) 5 4 3 3 Vcc 7 TxDB (Mouse) 2 1 4 RxDB (Mouse) 8 Vcc"

Commit message: ongoing
Parts:
- added X53: 100nF 0402, Capacitor_SMD:C_0402_1005Metric, symbol Device:C
- added X54: 10nF 0402, Capacitor_SMD:C_0402_1005Metric, symbol Device:C
Connections:
- net GND: now also X53.2, X54.2
- net VCC: now also X53.1, X54.1
Changed lines of the file:
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@@
+	(wire
+		(pts
+			(xy 16.51 88.9) (xy 21.59 88.9)
+		)
+		(stroke
+			(width 0)
+			(type default)
+		)
+	)
 	(wire
 		(pts
@@
 		(pts
 			(xy 144.78 154.94) (xy 148.59 154.94)
+		)
+		(stroke
+			(width 0)
+			(type default)
+		)
+	)
+	(wire
+		(pts
+			(xy 16.51 96.52) (xy 21.59 96.52)
 		)
 		(stroke
@@
 		)
 	)
+	(label "VCC"
+		(at 16.51 88.9 90)
+		(effects
+			(font
+				(size 1.27 1.27)
+			)
+			(justify left bottom)
+		)
+	)
 	(label "A2"
 		(at 55.88 74.93 180)
@@
 			)
 			(justify left bottom)
+		)
+	)
+	(label "GND"
+		(at 16.51 96.52 270)
+		(effects
+			(font
+				(size 1.27 1.27)
+			)
+			(justify right bottom)
 		)
 	)
@@
 	)
 	(symbol
+		(lib_id "Device:C")
+		(at 21.59 92.71 0)
+		(unit 1)
+		(exclude_from_sim no)
+		(in_bom yes)
+		(on_board yes)
+		(dnp no)
+		(fields_autoplaced yes)
+		(property "Reference" "X54"
+			(at 25.4 91.4399 0)
+			(effects
+				(font
+					(size 1.27 1.27)
+				)
+				(justify left)
+			)
+		)
+		(property "Value" "10nF 0402"
+			(at 25.4 93.9799 0)
+			(effects
+				(font
+					(size 1.27 1.27)
+				)
+				(justify left)
+			)
+		)
+		(property "Footprint" "Capacitor_SMD:C_0402_1005Metric"
+			(at 22.5552 96.52 0)
+			(effects
+				(font
+					(size 1.27 1.27)
+				)
+				(hide yes)
+			)
+		)
+		(property "Datasheet" "~"
+			(at 21.59 92.71 0)
+			(effects
+				(font
+					(size 1.27 1.27)
+				)
+				(hide yes)
+			)
+		)
+		(property "Description" "Unpolarized capacitor"
+			(at 21.59 92.71 0)
+			(effects
+				(font
+					(size 1.27 1.27)
+				)
+				(hide yes)
+			)
+		)
+		(property "MPN" "CL05B103KB5NNNC"
+			(at 21.59 92.71 0)
+			(effects
+				(font
+					(size 1.27 1.27)
+				)
+				(hide yes)
+			)
+		)
+		(pin "1"
+		)
+		(pin "2"
+		)
+		(instances
+			(project "sun3_60"
+				(path "/d6b5cf90-8df0-4384-868a-524abed7c432/054c9f34-4c69-4214-aead-9eddc8182f56"
+					(reference "X54")
+					(unit 1)
+				)
+			)
+		)
+	)
+	(symbol
 		(lib_id "Device:R_Pack04_SIP")
 		(at 201.93 129.54 90)
@@
 				)
 			)
+		)
+	)
+	(symbol
+		(lib_id "Device:C")
+		(at 16.51 92.71 0)
+		(unit 1)
+		(exclude_from_sim no)
+		(in_bom yes)
+		(on_board yes)
+		(dnp no)
+		(fields_autoplaced yes)
+		(property "Reference" "X53"
+			(at 20.32 91.4399 0)
+			(effects
+				(font
+					(size 1.27 1.27)
+				)
+				(justify left)
+			)
+		)
+		(property "Value" "100nF 0402"
+			(at 20.32 93.9799 0)
+			(effects
+				(font
+					(size 1.27 1.27)
+				)
+				(justify left)
+			)
+		)
+		(property "Footprint" "Capacitor_SMD:C_0402_1005Metric"
+			(at 17.4752 96.52 0)
+			(effects
+				(font
+					(size 1.27 1.27)
+				)
+				(hide yes)
+			)
+		)
+		(property "Datasheet" "~"
+			(at 16.51 92.71 0)
+			(effects
+				(font
+					(size 1.27 1.27)
+				)
+				(hide yes)
+			)
+		)
+		(property "Description" "Unpolarized capacitor"
+			(at 16.51 92.71 0)
+			(effects
+				(font
+					(size 1.27 1.27)
+				)
+				(hide yes)
+			)
+		)
+		(property "MPN" "CL05B104KO5NNNC"
+			(at 16.51 92.71 0)
+			(effects
+				(font
+					(size 1.27 1.27)
+				)
+				(hide yes)
+			)
+		)
+		(pin "1"
+		)
+		(pin "2"
+		)
+		(instances
+			(project "sun3_60"
+				(path "/d6b5cf90-8df0-4384-868a-524abed7c432/054c9f34-4c69-4214-aead-9eddc8182f56"
+					(reference "X53")
+					(unit 1)
+				)
+			)
