File: schematics/kicad/sun3_60_cpu.kicad_sch (KiCad schematic)
At the start: 24 parts, among them K199 10UF, U100 68020, U101 68881, U102 PAL16L8, U103 PAL16L8, U104 74F04, U106 PAL16L8, U107 PAL20X10, U108 74F00, U110 40.000 Mhz, U113 74AS74, U114 74F175, U115 74LS590, U122 ALS374, U123 ALS373, U130 74F374, U131 PAL16R6, U132 ALS244, U199 7705, U2003 74AS04, U2004 74LS125

Commit message: First draft for an expanded MMU
This version uses vintage parts except for the SRAM, which are IS61C5128AS-25HLI (they could be QLI instead)
Unfortunately, this requires:
* 2 more 74ALS245 to buffer the second byte of PMAP indices in the SMAP
* one more LS2518 (!) to extend the context register
* a couple of 74CBTLV3257 to be able to stay in "normal" Sun3 mode with minimal delays on the signals
* a couple of switches to enabled/disable the new features
* some extra passives
* U231, a PAL16L8, needs another input and another two outputs, or can be split in two PALs (or GAL, CPLDs, ...)

Also this does not include tne necessary decoupling on the new components
Changed lines of the file:
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@@
 (kicad_sch
-	(version 20231120)
+	(version 20250114)
 	(generator "eeschema")
-	(generator_version "8.0")
+	(generator_version "9.0")
 	(paper "USLedger")
 	(title_block
@@
 		(rev "1")
 	)
+	(text "REF CLOCK"
+		(exclude_from_sim no)
+		(at 50.8 217.17 0)
+		(effects
+			(font
+				(size 1.27 1.27)
+			)
+			(justify left bottom)
+		)
+	)
+	(text "BERR"
+		(exclude_from_sim no)
+		(at 107.95 220.98 0)
+		(effects
+			(font
+				(size 1.27 1.27)
+			)
+			(justify right bottom)
+		)
+	)
+	(text "FCDECODE"
+		(exclude_from_sim no)
+		(at 285.75 24.13 0)
+		(effects
+			(font
+				(size 1.27 1.27)
+			)
+			(justify left bottom)
+		)
+	)
+	(text "DVMA"
+		(exclude_from_sim no)
+		(at 345.44 190.5 0)
+		(effects
+			(font
+				(size 1.27 1.27)
+			)
+			(justify right bottom)
+		)
+	)
+	(text "Excluded"
+		(exclude_from_sim no)
+		(at 181.61 31.75 0)
+		(effects
+			(font
+				(size 1.27 1.27)
+				(color 255 0 0 1)
+			)
+			(justify left bottom)
+		)
+	)
+	(text "FPPDECODE"
+		(exclude_from_sim no)
+		(at 342.9 24.13 0)
+		(effects
+			(font
+				(size 1.27 1.27)
+			)
+			(justify left bottom)
+		)
+	)
+	(text "RESET"
+		(exclude_from_sim no)
+		(at 102.87 158.75 0)
+		(effects
+			(font
+				(size 1.27 1.27)
+			)
+			(justify left bottom)
+		)
+	)
 	(junction
 		(at 201.93 48.26)
@@
 		)
 	)
-	(text "REF CLOCK"
-		(exclude_from_sim no)
-		(at 50.8 217.17 0)
-		(effects
-			(font
-				(size 1.27 1.27)
-			)
-			(justify left bottom)
-		)
-	)
-	(text "BERR"
-		(exclude_from_sim no)
-		(at 107.95 220.98 0)
-		(effects
-			(font
-				(size 1.27 1.27)
-			)
-			(justify right bottom)
-		)
-	)
-	(text "FCDECODE"
-		(exclude_from_sim no)
-		(at 285.75 24.13 0)
-		(effects
-			(font
-				(size 1.27 1.27)
-			)
-			(justify left bottom)
-		)
-	)
-	(text "DVMA"
-		(exclude_from_sim no)
-		(at 345.44 190.5 0)
-		(effects
-			(font
-				(size 1.27 1.27)
-			)
-			(justify right bottom)
-		)
-	)
-	(text "Excluded"
-		(exclude_from_sim no)
-		(at 181.61 31.75 0)
-		(effects
-			(font
-				(size 1.27 1.27)
-				(color 255 0 0 1)
-			)
-			(justify left bottom)
-		)
-	)
-	(text "FPPDECODE"
-		(exclude_from_sim no)
-		(at 342.9 24.13 0)
-		(effects
-			(font
-				(size 1.27 1.27)
-			)
-			(justify left bottom)
-		)
-	)
-	(text "RESET"
-		(exclude_from_sim no)
-		(at 102.87 158.75 0)
-		(effects
-			(font
-				(size 1.27 1.27)
-			)
-			(justify left bottom)
-		)
-	)

Commit message: draft, ugly and WiP
Parts:
- removed U113: 74AS74, Package_DIP:DIP-14_W7.62mm, symbol custom:74AS74
- added U13, U14: 74LVC1G04, Package_TO_SOT_SMD:SOT-353_SC-70-5, symbol 74xGxx:74LVC1G04
- added U15, U17: 74LVC1G74, sun3_60:74AVC9112GTX, symbol 74xGxx:74AUC1G74
- added X13, X14, X17, X19, X21, X22, X33, X34, X37, X39, X40, X41, X42, X46, X47, X48, X50, X51: 100nF 0402, Capacitor_SMD:C_0402_1005Metric, symbol Device:C
- added X18: 10nF 0402, Capacitor_SMD:C_0402_1005Metric, symbol Device:C
- C199: value 0.1UF -> 100nF 0402; footprint Capacitor_THT:C_Disc_D3.0mm_W2.0mm_P2.50mm -> Capacitor_SMD:C_0402_1005Metric; MPN (none) -> CL05B104KO5NNNC
- K199: value 10UF -> 10uF tantalum; footprint Capacitor_THT:CP_Radial_Tantal_D6.0mm_P2.50mm -> Capacitor_Tantalum_SMD:CP_EIA-3216-18_Kemet-A; MPN (none) -> TAJA106K016RNJ
- R100: value 150 ohm -> 150 ohm 0805; footprint Resistor_THT:R_Axial_DIN0207_L6.3mm_D2.5mm_P7.62mm_Horizontal -> Resistor_SMD:R_0805_2012Metric; MPN (none) -> 0805W8F1500T5E
- R101: value 100 ohm -> 100 ohm 0805; footprint Resistor_THT:R_Axial_DIN0207_L6.3mm_D2.5mm_P7.62mm_Horizontal -> Resistor_SMD:R_0805_2012Metric; MPN (none) -> 0805W8F1000T5E
- U100: footprint sun3_60:68020 -> sun3_60:MC68020RC25
- U101: footprint sun3_60:68881 -> sun3_60:MC68882_PGA
- U102: now not fitted; now left out of the parts list
- U104: footprint Package_DIP:DIP-14_W7.62mm -> Package_SO:SOIC-14_3.9x8.7mm_P1.27mm; MPN (none) -> SN74F04DR
- U108: footprint Package_DIP:DIP-14_W7.62mm -> Package_SO:SOIC-14_3.9x8.7mm_P1.27mm; MPN (none) -> SN74F00DR
- U110: footprint Oscillator:Oscillator_DIP-14 -> sun3_60:CXO_DIP8+14
- U114: footprint Package_DIP:DIP-16_W7.62mm -> Package_SO:SOIC-16_3.9x9.9mm_P1.27mm; MPN (none) -> SN74F175DR; now not fitted; now left out of the parts list
- U115: footprint Package_DIP:DIP-16_W7.62mm -> Package_SO:SO-16_3.9x9.9mm_P1.27mm; MPN (none) -> SN74LS590D
- U122: footprint sun3_60:ALS373 -> Package_SO:SOIC-20W_7.5x12.8mm_P1.27mm; MPN (none) -> SN74ALS374ADWR; now not fitted; now left out of the parts list
- U123: footprint sun3_60:ALS373 -> Package_SO:SOIC-20W_7.5x12.8mm_P1.27mm; MPN (none) -> SN74ALS373ADWR; MPN-ALT (none) -> DM74ALS373WM; now not fitted; now left out of the parts list
- U130: footprint Package_DIP:DIP-20_W7.62mm -> Package_SO:SOIC-20W_7.5x12.8mm_P1.27mm; MPN (none) -> SN74F374DWR
- U132: footprint Package_DIP:DIP-20_W7.62mm -> Package_SO:SOIC-20W_7.5x12.8mm_P1.27mm; MPN (none) -> SN74ALS244CDWR
- U2003: footprint Package_DIP:DIP-14_W7.62mm -> Package_SO:SOIC-14_3.9x8.7mm_P1.27mm; MPN (none) -> SN74AS04DR
- U2004: footprint Package_DIP:DIP-14_W7.62mm -> Package_SO:SOIC-14_3.9x8.7mm_P1.27mm; MPN (none) -> SN74LS125ADR
Connections:
- net A0: now also U100.C4 (A00); no longer U100.30 (A00)
- net A1: now also U100.A2 (A01), U101.K1 (A01); no longer U100.2 (A01), U101.91 (A01)
- net A10: now also U100.B12 (A10); no longer U100.25 (A10)
- net A11: now also U100.A12 (A11); no longer U100.12 (A11)
- net A12: now also U100.C10 (A12); no longer U100.36 (A12)
- net A13: now also U100.B11 (A13); no longer U100.24 (A13)
- net A14: now also U100.A11 (A14); no longer U100.11 (A14)
- net A15: now also U100.B10 (A15); no longer U100.23 (A15)
- net A16: now also U100.C9 (A16); no longer U100.35 (A16)
- net A17: now also U100.C8 (A17); no longer U100.34 (A17)
- net A18: now also U100.B8 (A18); no longer U100.21 (A18)
- net A19: now also U100.A8 (A19); no longer U100.8 (A19)
- net A2: now also U100.E12 (A02), U101.H2 (A02); no longer U100.64 (A02), U101.72 (A02)
- net A20: now also U100.B7 (A20); no longer U100.20 (A20)
- net A21: now also U100.C7 (A21); no longer U100.33 (A21)
- net A22: now also U100.A7 (A22); no longer U100.7 (A22)
- net A23: now also U100.A6 (A23); no longer U100.6 (A23)
- net A24: now also U100.B6 (A24), U132.16 (1Y2); no longer U100.19 (A24), U132.18 (1Y1)
- net A25: now also U100.C6 (A25); no longer U100.32 (A25)
- net A26: now also U100.A5 (A26), U132.5 (2Y3); no longer U100.5 (A26), U132.16 (1Y2)
- net A27: now also U100.B5 (A27), U132.18 (1Y1); no longer U100.18 (A27), U132.5 (2Y3)
- net A28: now also U100.A4 (A28); no longer U100.4 (A28)
- net A29: now also U100.C5 (A29); no longer U100.31 (A29)
- net A3: now also U100.D13 (A03), U101.J1 (A03); no longer U100.52 (A03), U101.81 (A03)
- net A30: now also U100.B4 (A30); no longer U100.17 (A30)
- net A31: now also U100.A3 (A31); no longer U100.3 (A31)
- net A4: now also U100.D12 (A04), U101.G2 (A04); no longer U100.51 (A04), U101.62 (A04)
- net A5: now also U100.C13 (A05); no longer U100.39 (A05)
- net A6: now also U100.B13 (A06); no longer U100.26 (A06)
- net A7: now also U100.C12 (A07); no longer U100.38 (A07)
- net A8: now also U100.A13 (A08); no longer U100.13 (A08)
- net A9: now also U100.C11 (A09); no longer U100.37 (A09)
- net AS: now also U14.4; no longer U104.2
- net AS-: now also U100.L1 (AS-), U101.H1 (AS-), U14.2; no longer U100.131 (AS-), U101.71 (AS-), U104.1
- net BACK-: now also U100.A1 (BGACK-); no longer U100.1 (BGACK-)
- net BERR-: now also U100.J2 (BERR-); no longer U100.106 (BERR-)
- net BG-: now also U100.B2 (BG-); no longer U100.15 (BG-)
- net BR-: now also U100.B3 (BR-); no longer U100.16 (BR-)
- net CDIS-: now also U100.H1 (CDIS-); no longer U100.92 (CDIS-)
- net CLK1: now also U100.C2 (CLK), U101.C2 (CLK); no longer U100.28 (CLK), U101.22 (CLK)
- net CLK2X: now also U15.1 (C)
- net CLKA: now also U15.5 (Q)
- net CLKA-: now also U15.2 (D), U15.3 (~{Q})
- net CS.FPP-: now also U101.J3 (CS-); no longer U101.83 (CS-)
- net D0: now also U100.K13 (D00), U101.A3 (D00); no longer U100.130 (D00), U101.3 (D00)
- net D1: now also U100.K12 (D01), U101.A4 (D01); no longer U100.129 (D01), U101.4 (D01)
- net D10: now also U100.M10 (D10), U101.B9 (D10); no longer U100.153 (D10), U101.19 (D10)
- net D11: now also U100.L9 (D11), U101.B10 (D11); no longer U100.139 (D11), U101.20 (D11)
- net D12: now also U100.N10 (D12), U101.D9 (D12); no longer U100.166 (D12), U101.39 (D12)
- net D13: now also U100.M9 (D13), U101.C9 (D13); no longer U100.152 (D13), U101.29 (D13)
- net D14: now also U100.N9 (D14), U101.C10 (D14); no longer U100.165 (D14), U101.30 (D14)
- net D15: now also U100.L8 (D15), U101.D10 (D15); no longer U100.138 (D15), U101.40 (D15)
- net D16: now also U100.M7 (D16), U101.F10 (D16); no longer U100.150 (D16), U101.60 (D16)
- net D17: now also U100.N6 (D17), U101.F9 (D17); no longer U100.162 (D17), U101.59 (D17)
- net D18: now also U100.M6 (D18), U101.G10 (D18); no longer U100.149 (D18), U101.70 (D18)
- net D19: now also U100.L6 (D19), U101.H10 (D19); no longer U100.136 (D19), U101.80 (D19)
- net D2: now also U100.L13 (D02), U101.B5 (D02); no longer U100.143 (D02), U101.15 (D02)
- net D20: now also U100.N5 (D20), U101.G9 (D20); no longer U100.161 (D20), U101.69 (D20)
- net D21: now also U100.M5 (D21), U101.J10 (D21); no longer U100.148 (D21), U101.90 (D21)
- net D22: now also U100.N4 (D22), U101.K10 (D22); no longer U100.160 (D22), U101.100 (D22)
- net D23: now also U100.L5 (D23), U101.J9 (D23); no longer U100.135 (D23), U101.89 (D23)
- net D24: now also U100.M4 (D24), U101.K9 (D24); no longer U100.147 (D24), U101.99 (D24)
- net D25: now also U100.N3 (D25), U101.J7 (D25); no longer U100.159 (D25), U101.87 (D25)
- net D26: now also U100.M3 (D26), U101.K8 (D26); no longer U100.146 (D26), U101.98 (D26)
- net D27: now also U100.L4 (D27), U101.K7 (D27); no longer U100.134 (D27), U101.97 (D27)
- net D28: now also U100.N2 (D28), U101.J6 (D28); no longer U100.158 (D28), U101.86 (D28)
- net D29: now also U100.M2 (D29), U101.K6 (D29); no longer U100.145 (D29), U101.96 (D29)
- net D3: now also U100.L12 (D03), U101.A5 (D03); no longer U100.142 (D03), U101.5 (D03)
- net D30: now also U100.L3 (D30), U101.K5 (D30); no longer U100.133 (D30), U101.95 (D30)
- net D31: now also U100.N1 (D31), U101.J5 (D31); no longer U100.157 (D31), U101.85 (D31)
- net D4: now also U100.M13 (D04), U101.A6 (D04); no longer U100.156 (D04), U101.6 (D04)
- net D5: now also U100.M12 (D05), U101.B6 (D05); no longer U100.155 (D05), U101.16 (D05)
- net D6: now also U100.M11 (D06), U101.A7 (D06); no longer U100.154 (D06), U101.7 (D06)
- net D7: now also U100.L10 (D07), U101.A8 (D07); no longer U100.140 (D07), U101.8 (D07)
- net D8: now also U100.N12 (D08), U101.A9 (D08); no longer U100.168 (D08), U101.9 (D08)
- net D9: now also U100.N11 (D09), U101.C8 (D09); no longer U100.167 (D09), U101.28 (D09)
- net DS: now also U13.4; no longer U104.8
- net DS-: now also U100.M1 (DS-), U101.G1 (DS-), U13.2; no longer U100.144 (DS-), U101.61 (DS-), U104.9
- net DSACK0-: now also U100.H3 (DSACK0-), U101.J4 (DSACK0-), U2004.6; no longer U100.94 (DSACK0-), U101.84 (DSACK0-), U2004.3
- net DSACK1-: now also U100.J1 (DSACK1-), U101.K4 (DSACK1-), U2004.3; no longer U100.105 (DSACK1-), U101.94 (DSACK1-), U2004.6
- net E.CS-: now also U100.G1 (ECS-), U17.1 (C); no longer U100.79 (ECS-)
- net E.HOLD-: now also U17.2 (D)
- net FC0: now also U100.E1 (FC0); no longer U100.53 (FC0)
- net FC1: now also U100.F3 (FC1); no longer U100.68 (FC1)
- net FC2: now also U100.F2 (FC2); no longer U100.67 (FC2)
- net GND: now also U100.A10 (GND), U100.B1 (GND), U100.B9 (GND), U100.C3 (GND), U100.F12 (GND), U100.G12 (GND), U100.H13 (GND), U100.H2 (AVEC-), U100.J3 (GND), U100.K1 (GND), U100.K3 (GND), U100.L11 (GND), U100.L7 (GND), U100.N7 (GND), U101.A10 (GND), U101.A2 (GND), U101.B2 (GND), U101.B3 (GND), U101.B4 (~{SENSE}), U101.B7 (GND), U101.C1 (GND), U101.C3 (GND), U101.D2 (GND), U101.E10 (GND), U101.F2 (GND), U101.H9 (GND), U101.J8 (GND), U101.K3 (GND), U13.3 (GND), U14.3 (GND), U15.4 (GND), U17.4 (GND), X13.2, X14.2, X17.2, X18.2, X19.2, X21.2, X22.2, X33.2, X34.2, X37.2, X39.2, X40.2, X41.2, X42.2, X46.2, X47.2, X48.2, X50.2, X51.2; no longer U100.10 (GND), U100.104 (GND), U100.107 (GND), U100.118 (GND), U100.137 (GND), U100.163 (GND), U100.22 (GND), U100.90 (GND), U100.93 (AVEC-), U101.10 (GND), U101.12 (GND), U101.13 (GND), U101.14 (GND), U101.17 (GND), U101.2 (GND), U101.21 (GND), U101.23 (GND), U101.32 (GND), U101.50 (GND), U101.52 (GND), U101.79 (GND), U101.88 (GND), U101.93 (GND)
- net HALT-: now also U100.K2 (HALT-); no longer U100.119 (HALT-)
- net IOLOCK-: now also U17.5 (Q)
- net IPL0-: now also U100.J12 (IPL0-); no longer U100.116 (IPL0-)
- net IPL1-: now also U100.J13 (IPL1-); no longer U100.117 (IPL1-)
- net IPL2-: now also U100.H12 (IPL2-); no longer U100.103 (IPL2-)
- net PU.2: now also U15.7 (~{PRE}), U17.7 (~{PRE})
- net PU.3: now also U15.6 (~{CLR}), U17.6 (~{CLR})
- net RESET-: now also U100.C1 (RESET-), U101.D1 (RESET-); no longer U100.27 (RESET-), U101.31 (RESET-)
- net R/W-: now also U100.L2 (R/W-), U101.K2 (R/W-); no longer U100.132 (R/W-), U101.92 (R/W-)
- net SIZ0: now also U100.F1 (SIZ0); no longer U100.66 (SIZ0)
- net SIZ1: now also U100.G2 (SIZ1); no longer U100.80 (SIZ1)
- net VCC: now also U100.A9 (VCC), U100.D1 (VCC), U100.D2 (VCC), U100.D3 (VCC), U100.E3 (VCC), U100.G11 (VCC), U100.G13 (VCC), U100.M8 (VCC), U100.N13 (VCC), U100.N8 (VCC), U101.A1 (VCC), U101.B1 (VCC), U101.B8 (VCC), U101.E2 (VCC), U101.E9 (VCC), U101.F1 (Size-), U101.H3 (A00), U101.H8 (VCC), U101.J2 (VCC), U13.5 (VCC), U14.5 (VCC), U15.8 (VCC), U17.8 (VCC), X13.1, X14.1, X17.1, X18.1, X19.1, X21.1, X22.1, X33.1, X34.1, X37.1, X39.1, X40.1, X41.1, X42.1, X46.1, X47.1, X48.1, X50.1, X51.1; no longer U100.151 (VCC), U100.164 (VCC), U100.40 (VCC), U100.41 (VCC), U100.55 (VCC), U100.89 (VCC), U100.9 (VCC), U100.91 (VCC), U101.1 (VCC), U101.11 (VCC), U101.18 (VCC), U101.42 (VCC), U101.49 (VCC), U101.51 (Size-), U101.73 (A00), U101.78 (VCC), U101.82 (VCC)
- no-connect marks 34 -> 40
Other:
- note added: "CLK1 termination: CHECKME (position, values)"
- note removed: "Excluded"
- moved on the sheet: U104A

Commit message: update
Parts:
- U107, X48: now not fitted; now left out of the parts list
- U199: footprint Package_DIP:DIP-8_W7.62mm -> Package_SO:SOIC-8_3.9x4.9mm_P1.27mm; MPN (none) -> TL7705AID
Changed lines of the file:
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@@
 	)
 	(hierarchical_label "IOLOCK-"
-		(shape input)
+		(shape output)
 		(at 288.29 151.13 0)
 		(effects
@@
 		(unit 1)
 		(exclude_from_sim no)
-		(in_bom yes)
-		(on_board yes)
-		(dnp no)
+		(in_bom no)
+		(on_board no)
+		(dnp yes)
 		(property "Reference" "U107"
 			(at 105.41 162.179 0)
@@
 			)
 		)
-		(property "Footprint" "Package_DIP:DIP-8_W7.62mm"
+		(property "Footprint" "Package_SO:SOIC-8_3.9x4.9mm_P1.27mm"
 			(at 66.04 162.56 0)
 			(effects
@@
 			)
 		)
-		(property "MPN" ""
+		(property "MPN" "TL7705AID"
 			(at 66.04 162.56 0)
 			(effects
@@
 		(unit 1)
 		(exclude_from_sim no)
-		(in_bom yes)
-		(on_board yes)
-		(dnp no)
+		(in_bom no)
+		(on_board no)
+		(dnp yes)
 		(fields_autoplaced yes)
 		(property "Reference" "X48"

Commit message: ongoing ethernet pld
Parts:
- added C53, C54, C55, C56, C57, C58, C59, C60: 100nF 0402, Capacitor_SMD:C_0402_1005Metric, symbol Device:C
- added IC7: ATF1504AS-10AU100, sun3_60:QFP50P1600X1600X120-100N, symbol ATF1504AS-10AU100:ATF1504AS-10AU100
Connections:
- net AS-: now also IC7.68 (I/O_39)
- net BACK-: now also IC7.63 (I/O_35)
- net BERR-: now also IC7.99 (I/O_55)
- net BERR.P-: now also IC7.57 (I/O_31)
- net BERR.T-: now also IC7.58 (I/O_32)
- net BERR.V-: now also IC7.56 (I/O_30)
- net BERRCLK: now also IC7.100 (I/O_56)
- net BG-: now also IC7.64 (I/O_36)
- net BR-: now also IC7.65 (I/O_37)
- net C.S5-: now also IC7.12 (I/O/PD1)
- net C.S7X-: now also IC7.6 (I/O_1)
- net CLK-: now also IC7.87 (INPUT/GCLK1)
- net DDIS-: now also IC7.17 (I/O_8)
- net DMA: now also IC7.40 (I/O_22)
- net DMA-: now also IC7.14 (I/O_6), IC7.37 (I/O_21)
- net DMAX-: now also IC7.36 (I/O_20)
- net DSACK0-: now also IC7.69 (I/O_40)
- net DXACK-: now also IC7.16 (I/O_7)
- net E.ACK-: now also IC7.20 (I/O_10)
- net E.REQ-: now also IC7.9 (I/O_3)
- net E.REX-: now also IC7.30 (I/O_15)
- net EMULATE-: now also IC7.41 (I/0)
- net GND: now also C53.2, C54.2, C55.2, C56.2, C57.2, C58.2, C59.2, C60.2, IC7.11 (GND_1), IC7.26 (GND_2), IC7.38 (GND_3), IC7.43 (GND_4), IC7.59 (GND_5), IC7.74 (GND_6), IC7.86 (GND_7), IC7.95 (GND_8)
- net HALT-: now also IC7.61 (I/O_34)
- net INIT-: now also IC7.54 (I/O_29)
- net MUX-: now also IC7.35 (I/O_19)
- net R.ACK-: now also IC7.19 (I/O_9)
- net R.CLK-: now also IC7.90 (INPUT/GCLK2)
- net R.REQ-: now also IC7.8 (I/O_2)
- net R.REX-: now also IC7.29 (I/O_14)
- net RERUN-: now also IC7.42 (I/O/PD2)
- net RESET-: now also IC7.71 (I/O_41)
- net S.ACK-: now also IC7.21 (I/O_11)
- net S.REQ-: now also IC7.10 (I/O_4)
- net S.REX-: now also IC7.31 (I/O_16)
- net VCC: now also C53.1, C54.1, C55.1, C56.1, C57.1, C58.1, C59.1, C60.1, IC7.18 (VCCIO_2), IC7.3 (VCCIO_1), IC7.34 (VCCIO_3), IC7.39 (VCCINT_1), IC7.51 (VCCIO_4), IC7.66 (VCCIO_5), IC7.82 (VCCIO_6), IC7.91 (VCCINT_2)
- net XACK-: now also IC7.23 (I/O_12)
- net XACK5-: now also IC7.13 (I/O_5)
- new net JTAG_TCK7: IC7.62 (I/O/TCK)
- new net JTAG_TDI7: IC7.4 (I/O/TDI)
- new net JTAG_TDO7: IC7.73 (I/O/TDO)
- new net JTAG_TMS7: IC7.15 (I/O/TMS)
- no-connect marks 40 -> 56
Other:
- note added: "CPLD DVMA"

Commit message: update (lost cause?)
Parts:
- added R75, R76, R77, R78: 4.7k, Resistor_SMD:R_0402_1005Metric, symbol Device:R
- U14: footprint Package_TO_SOT_SMD:SOT-353_SC-70-5 -> Package_TO_SOT_SMD:SOT-23-5; MPN (none) -> SN74LVC1G04DBVR
Connections:
- net VCC: now also R75.1, R76.1, R77.1, R78.1
- net PU.2 renamed PU.2a
- net PU.2a: now also R75.2; no longer U17.7 (~{PRE})
- net PU.3 renamed PU.3a
- net PU.3a: now also R78.2; no longer U17.6 (~{CLR})
- new net PU.2b: R76.2, U17.7 (~{PRE})
- new net PU.3b: R77.2, U17.6 (~{CLR})
