File: schematics/kicad/sun3_60_ethernet.kicad_sch (KiCad schematic)
At the start: 28 parts, among them J3 Ethernet, K500 10 uF, U500 AM7990, U501 AM7992, U502 20 Mhz, U503 TRANSF, U508 DG303A, U509 DG303A, U510 ALS373, U511 ALS373, U512 ALS373, U514 ALS652, U515 ALS652, U516 ALS652, U517 ALS652, U518 PAL16L8, U519 PAL16L8, U520 74F175

Commit message: First draft for an expanded MMU
This version uses vintage parts except for the SRAM, which are IS61C5128AS-25HLI (they could be QLI instead)
Unfortunately, this requires:
* 2 more 74ALS245 to buffer the second byte of PMAP indices in the SMAP
* one more LS2518 (!) to extend the context register
* a couple of 74CBTLV3257 to be able to stay in "normal" Sun3 mode with minimal delays on the signals
* a couple of switches to enabled/disable the new features
* some extra passives
* U231, a PAL16L8, needs another input and another two outputs, or can be split in two PALs (or GAL, CPLDs, ...)

Also this does not include tne necessary decoupling on the new components
Changed lines of the file:
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@@
 (kicad_sch
-	(version 20231120)
+	(version 20250114)
 	(generator "eeschema")
-	(generator_version "8.0")
+	(generator_version "9.0")
 	(paper "USLedger")
 	(title_block
@@
 		(rev "1")
 	)
+	(text "EXCLUDED"
+		(exclude_from_sim no)
+		(at 233.172 96.774 0)
+		(effects
+			(font
+				(size 1.27 1.27)
+				(color 255 0 0 1)
+			)
+		)
+	)
+	(text "ETHER2"
+		(exclude_from_sim no)
+		(at 387.858 75.184 0)
+		(effects
+			(font
+				(size 1.27 1.27)
+			)
+		)
+	)
+	(text "COAX/AUI SELECTOR"
+		(exclude_from_sim no)
+		(at 233.68 93.98 0)
+		(effects
+			(font
+				(size 1.27 1.27)
+			)
+		)
+	)
 	(junction
 		(at 184.15 29.21)
@@
 		)
 	)
-	(text "EXCLUDED"
-		(exclude_from_sim no)
-		(at 233.172 96.774 0)
-		(effects
-			(font
-				(size 1.27 1.27)
-				(color 255 0 0 1)
-			)
-		)
-	)
-	(text "ETHER2"
-		(exclude_from_sim no)
-		(at 387.858 75.184 0)
-		(effects
-			(font
-				(size 1.27 1.27)
-			)
-		)
-	)
-	(text "COAX/AUI SELECTOR"
-		(exclude_from_sim no)
-		(at 233.68 93.98 0)
-		(effects
-			(font
-				(size 1.27 1.27)
-			)
-		)
-	)

Commit message: draft, ugly and WiP
Parts:
- removed J3: Ethernet, Connector_PinHeader_2.54mm:PinHeader_1x09_P2.54mm_Vertical, symbol Connector:Conn_01x09_Pin
- removed U503: TRANSF, Package_DIP:DIP-16_W7.62mm, symbol custom:PE-64102
- added J4: Ethernet, Connector_PinHeader_2.54mm:PinHeader_1x09_P2.54mm_Vertical, symbol Connector:Conn_01x09_Pin
- added J5: 5747845-4, 57478454, symbol 5747845-4:5747845-4
- added T1: TG01-0506NRLTR, TG010506NRLTR, symbol TG01-0506NRLTR:TG01-0506NRLTR
- added X10, X11, X12, X24, X25, X26, X43, X44, X45, X9: 100nF 0402, Capacitor_SMD:C_0402_1005Metric, symbol Device:C
- C503, C504: value 0.1uF -> 100nF 0402; footprint Capacitor_THT:C_Rect_L7.0mm_W2.0mm_P5.00mm -> Capacitor_SMD:C_0402_1005Metric; MPN (none) -> CL05B104KO5NNNC
- K500: value 10 uF -> 10uF tantalum; footprint Capacitor_THT:CP_Radial_Tantal_D6.0mm_P2.50mm -> Capacitor_Tantalum_SMD:CP_EIA-3216-18_Kemet-A
- S500, U508, U509: now not fitted; now left out of the parts list
- S502: MPN (none) -> 4611X-101-102LF; now not fitted; now left out of the parts list
- U510, U511, U512: footprint sun3_60:ALS373 -> Package_SO:SOIC-20W_7.5x12.8mm_P1.27mm; MPN (none) -> SN74ALS373ADWR; MPN-ALT (none) -> DM74ALS373WM
- U514, U515, U516, U517: footprint Package_DIP:DIP-24_W7.62mm -> Package_SO:SOIC-24W_7.5x15.4mm_P1.27mm; MPN (none) -> SN74ALS652ADW; MPN-ALT (none) -> DM74ALS652WM
- U520: footprint Package_DIP:DIP-16_W7.62mm -> Package_SO:SOIC-16_3.9x9.9mm_P1.27mm; MPN (none) -> SN74F175DR
Connections:
- net +12V: now also J4.1 (Pin_1), J5.13
- net A16: now also U512.12 (Q4); no longer U512.2 (Q0)
- net A17: now also U512.15 (Q5); no longer U512.5 (Q1)
- net A18: now also U512.16 (Q6); no longer U512.6 (Q2)
- net A19: now also U512.19 (Q7); no longer U512.9 (Q3)
- net A20: now also U512.2 (Q0); no longer U512.12 (Q4)
- net A21: now also U512.5 (Q1); no longer U512.15 (Q5)
- net A22: now also U512.6 (Q2); no longer U512.16 (Q6)
- net A23: now also U512.9 (Q3); no longer U512.19 (Q7)
- net E.A16: now also U512.13 (D4); no longer U512.3 (D0)
- net E.A17: now also U512.14 (D5); no longer U512.4 (D1)
- net E.A18: now also U512.17 (D6); no longer U512.7 (D2)
- net E.A19: now also U512.18 (D7); no longer U512.8 (D3)
- net E.A20: now also U512.3 (D0); no longer U512.13 (D4)
- net E.A21: now also U512.4 (D1); no longer U512.14 (D5)
- net E.A22: now also U512.7 (D2); no longer U512.17 (D6)
- net E.A23: now also U512.8 (D3); no longer U512.18 (D7)
- net E.CO+: now also T1.1 (PRI_1)
- net E.CO+<>: now also J4.2 (Pin_2), J5.2, T1.16 (SEC_6)
- net E.CO-: now also T1.2 (PRI_2)
- net E.CO-<>: now also J4.3 (Pin_3), J5.9, T1.15 (SEC_5)
- net E.RX+: now also T1.7 (PRI_5)
- net E.RX+<>: now also J4.4 (Pin_4), J5.5, T1.10 (SEC_2)
- net E.RX-: now also T1.8 (PRI_6)
- net E.RX-<>: now also J4.5 (Pin_5), J5.12, T1.9 (SEC_1)
- net E.SMS: now also J4.8 (Pin_8), J5.6
- net E.TX+: now also T1.4 (PRI_3)
- net E.TX+<>: now also J4.6 (Pin_6), J5.3, T1.13 (SEC_4)
- net E.TX-: now also T1.5 (PRI_4)
- net E.TX-<>: now also J4.7 (Pin_7), J5.10, T1.12 (SEC_3)
- net GND: now also J4.9 (Pin_9), J5.1, J5.MH1, J5.MH2, X10.2, X11.2, X12.2, X24.2, X25.2, X26.2, X43.2, X44.2, X45.2, X9.2
- net VCC: now also X10.1, X11.1, X12.1, X24.1, X25.1, X26.1, X43.1, X44.1, X45.1, X9.1
- no-connect marks 13 -> 19
Other:
- note added: "Matching slider is 5745583-5"

Commit message: ongoing ethernet pld
Parts:
- added C61, C62, C63, C64, C65, C66, C67, C68: 100nF 0402, Capacitor_SMD:C_0402_1005Metric, symbol Device:C
- added IC8: ATF1504AS-10AU100, sun3_60:QFP50P1600X1600X120-100N, symbol ATF1504AS-10AU100:ATF1504AS-10AU100
- U518, U519, U520, X43, X44, X45: now not fitted; now left out of the parts list
Connections:
- net BERR-: now also IC8.30 (I/O_15)
- net CLK-: now also IC8.87 (INPUT/GCLK1)
- net DS-: now also IC8.67 (I/O_38)
- net DSACK1-: now also IC8.60 (I/O_33)
- net E.ACK-: now also IC8.36 (I/O_20)
- net E.ALE: now also IC8.42 (I/O/PD2)
- net E.BM0-: now also IC8.46 (I/O_25)
- net E.BM1-: now also IC8.45 (I/O_24)
- net E.CBA: now also IC8.57 (I/O_31)
- net E.CREQ-: now also IC8.12 (I/O/PD1)
- net E.CS-: now also IC8.40 (I/O_22)
- net E.DAS-: now also IC8.47 (I/O_26)
- net E.GAB: now also IC8.52 (I/O_28)
- net E.GBA0-: now also IC8.54 (I/O_29)
- net E.GBA1-: now also IC8.56 (I/O_30)
- net E.HLDA-: now also IC8.41 (I/0)
- net E.HOLD-: now also IC8.44 (I/O_23)
- net E.HREQ-: now also IC8.13 (I/O_5)
- net E.RDY-: now also IC8.37 (I/O_21)
- net E.REQ-: now also IC8.94 (I/O_51)
- net E.WE-: now also IC8.48 (I/O_27)
- net EN.E-: now also IC8.6 (I/O_1)
- net GND: now also C61.2, C62.2, C63.2, C64.2, C65.2, C66.2, C67.2, C68.2, IC8.11 (GND_1), IC8.26 (GND_2), IC8.38 (GND_3), IC8.43 (GND_4), IC8.59 (GND_5), IC8.74 (GND_6), IC8.86 (GND_7), IC8.95 (GND_8)
- net RERUN-: now also IC8.93 (I/O_50)
- net R/W-: now also IC8.61 (I/O_34)
- net SIZ0: now also IC8.64 (I/O_36)
- net SIZ1: now also IC8.63 (I/O_35)
- net VCC: now also C61.1, C62.1, C63.1, C64.1, C65.1, C66.1, C67.1, C68.1, IC8.18 (VCCIO_2), IC8.3 (VCCIO_1), IC8.34 (VCCIO_3), IC8.39 (VCCINT_1), IC8.51 (VCCIO_4), IC8.66 (VCCIO_5), IC8.82 (VCCIO_6), IC8.91 (VCCINT_2)
- net XACK-: now also IC8.29 (I/O_14)
- new net INIT-: IC8.71 (I/O_41)
- new net JTAG_TCK8: IC8.62 (I/O/TCK)
- new net JTAG_TDI8: IC8.4 (I/O/TDI)
- new net JTAG_TDO8: IC8.73 (I/O/TDO)
- new net JTAG_TMS8: IC8.15 (I/O/TMS)
- no-connect marks 19 -> 35
Other:
- note added: "CPLD ETHERNET"

Commit message: ongoing
Parts:
- added U16: 20 MHz, Oscillator:Oscillator_SMD_SeikoEpson_SG8002LB-4Pin_5.0x3.2mm, symbol Oscillator:SG-5032CAN
- added X55: 100nF 0402, Capacitor_SMD:C_0402_1005Metric, symbol Device:C
- added X56: 10nF 0402, Capacitor_SMD:C_0402_1005Metric, symbol Device:C
- C500, C501, U502: now not fitted; now left out of the parts list
- C502: footprint Capacitor_THT:C_Rect_L7.0mm_W2.0mm_P5.00mm -> Capacitor_SMD:C_0402_1005Metric; MPN (none) -> 0402B681K500NT
- C505: footprint Capacitor_THT:C_Rect_L7.0mm_W2.0mm_P5.00mm -> Capacitor_SMD:C_0402_1005Metric; MPN (none) -> 0402B562K500NT
- R501: footprint Resistor_THT:R_Axial_DIN0207_L6.3mm_D2.5mm_P7.62mm_Horizontal -> Resistor_SMD:R_0402_1005Metric; MPN (none) -> 0402WGF5100TCE
- R502: footprint Resistor_THT:R_Axial_DIN0207_L6.3mm_D2.5mm_P7.62mm_Horizontal -> Resistor_SMD:R_0402_1005Metric; MPN (none) -> 0402WGF3001TCE
Connections:
- net E.REQ-: now also IC8.35 (I/O_19); no longer IC8.94 (I/O_51)
- net GND: now also U16.2 (GND), X55.2, X56.2
- net VCC: now also U16.4 (VCC), X55.1, X56.1
- net at C500.2, U502.2: no longer U501.8 (X1)
- net at C501.1, U502.1: no longer U501.9 (X2)
- new net CLK_20MHZ_ETH: U16.3 (OUT), U501.8 (X1)
- no-connect marks 35 -> 37

Commit message: update (lost cause?)
Connections:
- net DSACK1-: now also IC8.16 (I/O_7); no longer IC8.60 (I/O_33)
- net EN.E-: now also IC8.58 (I/O_32); no longer IC8.6 (I/O_1)
- net R/W-: now also IC8.17 (I/O_8); no longer IC8.61 (I/O_34)
- net SIZ0: now also IC8.20 (I/O_10); no longer IC8.64 (I/O_36)
- net SIZ1: now also IC8.19 (I/O_9); no longer IC8.63 (I/O_35)
Changed lines of the file:
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@@
 	(hierarchical_label "R{slash}W-"
 		(shape output)
-		(at -39.37 176.53 0)
-		(effects
-			(font
-				(size 1.27 1.27)
-			)
-			(justify left)
+		(at -115.57 181.61 180)
+		(effects
+			(font
+				(size 1.27 1.27)
+			)
+			(justify right)
 		)
 	)
@@
 	(hierarchical_label "SIZ0"
 		(shape output)
-		(at -39.37 168.91 0)
-		(effects
-			(font
-				(size 1.27 1.27)
-			)
-			(justify left)
+		(at -115.57 189.23 180)
+		(effects
+			(font
+				(size 1.27 1.27)
+			)
+			(justify right)
 		)
 	)
@@
 	(hierarchical_label "EN.E-"
 		(shape input)
-		(at -115.57 153.67 180)
-		(effects
-			(font
-				(size 1.27 1.27)
-			)
-			(justify right)
+		(at -39.37 184.15 0)
+		(effects
+			(font
+				(size 1.27 1.27)
+			)
+			(justify left)
 		)
 	)
@@
 	(hierarchical_label "SIZ1"
 		(shape output)
-		(at -39.37 171.45 0)
-		(effects
-			(font
-				(size 1.27 1.27)
-			)
-			(justify left)
+		(at -115.57 186.69 180)
+		(effects
+			(font
+				(size 1.27 1.27)
+			)
+			(justify right)
 		)
 	)
 	(hierarchical_label "DSACK1-"
 		(shape output)
-		(at -39.37 179.07 0)
-		(effects
-			(font
-				(size 1.27 1.27)
-			)
-			(justify left)
-		)
-	)
+		(at -115.57 179.07 180)
+		(effects
+			(font
+				(size 1.27 1.27)
+			)
+			(justify right)
+		)
+	)
