File: schematics/kicad/sun3_60_memory.kicad_sch (KiCad schematic)
At the start: 10 parts, among them U104 74F04, U108 74F00, U600 74F04, U800 PAL16L8, U801 74AS257, U802 PAL20L8, U803 74F64, U804 74F64, U805 PAL16L8

Commit message: draft, ugly and WiP
Parts:
- removed U801: 74AS257, Package_DIP:DIP-16_W7.62mm, symbol custom:74AS257
- added X110, X15, X16, X2: 100nF 0402, Capacitor_SMD:C_0402_1005Metric, symbol Device:C
- S800: MPN (none) -> 4611X-101-472LF; now not fitted; now left out of the parts list
- U104: footprint Package_DIP:DIP-14_W7.62mm -> Package_SO:SOIC-14_3.9x8.7mm_P1.27mm; MPN (none) -> SN74F04DR
- U108: footprint Package_DIP:DIP-14_W7.62mm -> Package_SO:SOIC-14_3.9x8.7mm_P1.27mm; MPN (none) -> SN74F00DR
- U600: footprint Package_DIP:DIP-14_W7.62mm -> Package_SO:SOIC-14_3.9x8.7mm_P1.27mm; MPN (none) -> SN74F04DR; now not fitted; now left out of the parts list
Connections:
- net PA02/22 is gone; now on net PA22: U802.7 (I7)
- net SEL0- is gone; now on net GND: U800.5 (I5)
- net SEL1 is gone; now on net VCC: U800.6 (I6)
- net GND: now also X110.2, X15.2, X16.2, X2.2
- net VCC: now also X110.1, X15.1, X16.1, X2.1
- net TWOWAY-: no longer names the net of U802.16 (IO16)
- no-connect marks 16 -> 30

Commit message: update (lost cause?)
Parts:
- added R70, R71, R72: 4.7k, Resistor_SMD:R_0402_1005Metric, symbol Device:R
Connections:
- net GND: now also R70.1, R71.1, R72.1
- net M.PD-: no longer U800.11 (I10), U802.23 (I23), U805.5 (I5)
- new net M.PDa-: R70.2, U800.11 (I10)
- new net M.PDb-: R71.2, U802.23 (I23)
- new net M.PDc-: R72.2, U805.5 (I5)
