File: schematics/kicad/sun3_60_simm1.kicad_sch (KiCad schematic)
At the start: 10 parts, among them U900 SIMM, U901 SIMM, U902 SIMM, U903 SIMM, U904 74AS258, U905 74AS258, U906 74AS258, U907 AS1032, U908 AS1032, U909 22 Ohm

Commit message: First draft for an expanded MMU
This version uses vintage parts except for the SRAM, which are IS61C5128AS-25HLI (they could be QLI instead)
Unfortunately, this requires:
* 2 more 74ALS245 to buffer the second byte of PMAP indices in the SMAP
* one more LS2518 (!) to extend the context register
* a couple of 74CBTLV3257 to be able to stay in "normal" Sun3 mode with minimal delays on the signals
* a couple of switches to enabled/disable the new features
* some extra passives
* U231, a PAL16L8, needs another input and another two outputs, or can be split in two PALs (or GAL, CPLDs, ...)

Also this does not include tne necessary decoupling on the new components
Changed lines of the file:
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@@
 (kicad_sch
-	(version 20231120)
+	(version 20250114)
 	(generator "eeschema")
-	(generator_version "8.0")
+	(generator_version "9.0")
 	(paper "A4")
 	(title_block

Commit message: draft, ugly and WiP
Parts:
- removed U909: 22 Ohm, Package_DIP:DIP-16_W7.62mm, symbol Device:R_Pack08
- added C1, C3: 10uF 1206, Capacitor_SMD:C_1206_3216Metric, symbol Device:C
- added R12, R13, R18, R19, R20, R21, R7, R9: 22, Resistor_SMD:R_0402_1005Metric, symbol Device:R
- added X86, X87, X88, X89, X90: 100nF 0402, Capacitor_SMD:C_0402_1005Metric, symbol Device:C
- U900, U901, U902, U903: footprint Connector_PinHeader_2.54mm:PinHeader_1x30_P2.54mm_Vertical -> sun3_60:SIMM
- U904, U905, U906: footprint Package_DIP:DIP-16_W7.62mm -> Package_SO:SOIC-16_3.9x9.9mm_P1.27mm; MPN (none) -> SN74F258D
- U907, U908: footprint Package_DIP:DIP-14_W7.62mm -> Package_SO:SOIC-14_3.9x8.7mm_P1.27mm; MPN (none) -> SN74AS1032AD
Connections:
- net CAS-: now also U908.12, U908.2; no longer U908.1, U908.13
- net CAS0-: now also U908.1, U908.13; no longer U908.12, U908.2
- net CE00-: now also R9.1
- net CE01-: now also R13.1
- net CE02-: now also R19.1
- net CE03-: now also R21.1
- net GND: now also C1.2, C3.2, X86.2, X87.2, X88.2, X89.2, X90.2; no longer U906.13 (4B), U906.14 (4A)
- net M.A9.0: now also U906.12 (4Y); no longer U906.7 (2Y)
- net M.CE00-: now also R9.2
- net M.CE01-: now also R13.2
- net M.CE02-: now also R19.2
- net M.CE03-: now also R21.2
- net M.RE00-: now also R7.2
- net M.RE01-: now also R12.2
- net M.RE02-: now also R18.2
- net M.RE03-: now also R20.2
- net PA18: now also U905.14 (4A); no longer U905.5 (2A)
- net PA19: now also U905.5 (2A); no longer U905.11 (3A)
- net PA20: now also U905.11 (3A); no longer U905.14 (4A)
- net RAS-: now also U907.12, U907.2; no longer U907.1, U907.13
- net RE00-: now also U907.5; no longer U907.2
- net RE01-: now also U907.9; no longer U907.5
- net RE02-: now also U907.1; no longer U907.9
- net RE03-: now also U907.13; no longer U907.12
- net VCC: now also C1.1, C3.1, X86.1, X87.1, X88.1, X89.1, X90.1
- net XE00-: now also U907.6, R7.1; no longer U907.3
- net XE01-: now also U907.8, R12.1; no longer U907.6
- net XE02-: now also U907.3, R18.1; no longer U907.8
- net XE03-: now also R20.1
- net M.A10.0: now reaches U902.19 (A10)
- net M.A10.0: now also U900.19 (A10), U901.19 (A10), U903.19 (A10), U906.7 (2Y)
- net PA22/02 renamed PA22
- new net A2: U906.13 (4B)
- new net PA23: U906.14 (4A)
- no-connect marks 5 -> 0
Other:
- note added: "bulk"
- moved on the sheet: U907A, U907B, U907C

Commit message: update (lost cause?)
Connections:
- net M.PD- is gone; now on net GND: U904.15 (G-), U905.15 (G-), U906.15 (G-)
Changed lines of the file:
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@@
 	)
 	(junction
-		(at 57.15 92.71)
-		(diameter 0)
-		(color 0 0 0 0)
-	)
-	(junction
 		(at 76.2 175.26)
 		(diameter 0)
@@
 	)
 	(junction
-		(at 57.15 133.35)
-		(diameter 0)
-		(color 0 0 0 0)
-	)
-	(junction
 		(at 184.15 33.02)
 		(diameter 0)
@@
 	(wire
 		(pts
-			(xy 57.15 52.07) (xy 57.15 92.71)
-		)
-		(stroke
-			(width 0)
-			(type default)
-		)
-	)
-	(wire
-		(pts
 			(xy 100.33 50.8) (xy 144.78 50.8)
 		)
@@
 	(wire
 		(pts
-			(xy 57.15 92.71) (xy 57.15 133.35)
-		)
-		(stroke
-			(width 0)
-			(type default)
-		)
-	)
-	(wire
-		(pts
 			(xy 71.12 147.32) (xy 78.74 147.32)
 		)
@@
 	(wire
 		(pts
-			(xy 57.15 133.35) (xy 57.15 135.89)
-		)
-		(stroke
-			(width 0)
-			(type default)
-		)
-	)
-	(wire
-		(pts
 			(xy 137.16 83.82) (xy 144.78 83.82)
 		)
@@
 		)
 	)
+	(label "GND"
+		(at 57.15 92.71 0)
+		(effects
+			(font
+				(size 1.27 1.27)
+			)
+			(justify left bottom)
+		)
+	)
 	(label "M.CE01-"
 		(at 162.56 149.86 0)
@@
 		)
 	)
+	(label "GND"
+		(at 57.15 133.35 0)
+		(effects
+			(font
+				(size 1.27 1.27)
+			)
+			(justify left bottom)
+		)
+	)
 	(label "M.A10.0"
 		(at 86.36 48.26 0)
@@
 		)
 	)
+	(label "GND"
+		(at 57.15 52.07 0)
+		(effects
+			(font
+				(size 1.27 1.27)
+			)
+			(justify left bottom)
+		)
+	)
 	(label "M.A9.0"
 		(at 86.36 45.72 0)
@@
 		)
 	)
-	(hierarchical_label "M.PD-"
-		(shape input)
-		(at 57.15 135.89 270)
-		(effects
-			(font
-				(size 1.27 1.27)
-			)
-			(justify right)
-		)
-	)
